File: hardware/schematic/v1.0/XWatch_Rev1.0/Connectivity.kicad_sch (KiCad schematic)
At the start: 1 part, among them U5 NT3H1101W0FHKH

Commit message: sch and pcb update
Parts:
- added IC4: nRF52833-QDAA-R, XWatch_Rev1.0:QFN40P500X500X90-41N, symbol XWatch_Rev1.0:nRF52833-QDAA-R
