File: hardware/schematic/v1.0/XWatch_Rev1.0/Sensors.kicad_sch (KiCad schematic)
At the start: 4 parts, among them U2 LSM6DSOXTR, U3 AK09918C, U4 BMI270, U6 LIS2MDLTR

Commit message: doc and sch update
Parts:
- removed U3: AK09918C, XWatch_Rev1.0:AK09918C, symbol XWatch_Rev1.0:AK09918C
- removed U4: BMI270, XWatch_Rev1.0:BMI270, symbol XWatch_Rev1.0:BMI270
- added IC2: MAX86141ENP+, XWatch_Rev1.0:BGA20C40P5X4_205X185X50, symbol XWatch_Rev1.0:MAX86141ENP+
- added U7: OPT3001DNPR, XWatch_Rev1.0:OPT3001DNPR, symbol XWatch_Rev1.0:OPT3001DNPR
- added U8: LPS27HHWTR, XWatch_Rev1.0:LPS27HHWTR, symbol XWatch_Rev1.0:LPS27HHWTR

Commit message: doc and sch update
Connections:
- net +1V8: now reaches U7.1 (VDD)
- net I2C_SCL: now reaches U7.4 (SCL)
- net I2C_SDA: now reaches U7.6 (SDA)
Other:
- moved on the sheet: U2
Changed lines of the file:
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@@
 	(generator_version "10.0")
 	(paper "A4")
+	(wire
+		(pts
+			(xy 53.34 62.23) (xy 57.15 62.23)
+		)
+		(stroke
+			(width 0)
+			(type default)
+		)
+	)
+	(wire
+		(pts
+			(xy 77.47 62.23) (xy 86.36 62.23)
+		)
+		(stroke
+			(width 0)
+			(type default)
+		)
+	)
+	(wire
+		(pts
+			(xy 77.47 67.31) (xy 86.36 67.31)
+		)
+		(stroke
+			(width 0)
+			(type default)
+		)
+	)
+	(label "I2C_SDA"
+		(at 78.74 62.23 0)
+		(effects
+			(font
+				(size 1.27 1.27)
+			)
+			(justify left bottom)
+		)
+	)
+	(label "I2C_SCL"
+		(at 78.74 67.31 0)
+		(effects
+			(font
+				(size 1.27 1.27)
+			)
+			(justify left bottom)
+		)
+	)
 	(symbol
 		(lib_id "XWatch_Rev1.0:OPT3001DNPR")
@@
 	)
 	(symbol
+		(lib_id "power:+1V8")
+		(at 53.34 62.23 0)
+		(unit 1)
+		(body_style 1)
+		(exclude_from_sim no)
+		(in_bom yes)
+		(on_board yes)
+		(in_pos_files yes)
+		(dnp no)
+		(fields_autoplaced yes)
+		(property "Reference" "#PWR033"
+			(at 53.34 66.04 0)
+			(hide yes)
+			(show_name no)
+			(do_not_autoplace no)
+			(effects
+				(font
+					(size 1.27 1.27)
+				)
+			)
+		)
+		(property "Value" "+1V8"
+			(at 53.34 57.15 0)
+			(show_name no)
+			(do_not_autoplace no)
+			(effects
+				(font
+					(size 1.27 1.27)
+				)
+			)
+		)
+		(property "Footprint" ""
+			(at 53.34 62.23 0)
+			(hide yes)
+			(show_name no)
+			(do_not_autoplace no)
+			(effects
+				(font
+					(size 1.27 1.27)
+				)
+			)
+		)
+		(property "Datasheet" ""
+			(at 53.34 62.23 0)
+			(hide yes)
+			(show_name no)
+			(do_not_autoplace no)
+			(effects
+				(font
+					(size 1.27 1.27)
+				)
+			)
+		)
+		(property "Description" "Power symbol creates a global label with name \"+1V8\""
+			(at 53.34 62.23 0)
+			(hide yes)
+			(show_name no)
+			(do_not_autoplace no)
+			(effects
+				(font
+					(size 1.27 1.27)
+				)
+			)
+		)
+		(pin "1"
+		)
+		(instances
+			(project "XWatch_Rev1.0"
+				(path "/2e5e9480-7d2e-4148-a9bf-0ac7d46b20bc/60582904-f38c-47af-bf5b-266849badec8"
+					(reference "#PWR033")
+					(unit 1)
+				)
+			)
+		)
+	)
+	(symbol
 		(lib_id "XWatch_Rev1.0:LPS27HHWTR")
 		(at 57.15 106.68 0)
@@
 	(symbol
 		(lib_id "XWatch_Rev1.0:LSM6DSOXTR")
-		(at 110.49 97.79 0)
+		(at 152.4 95.25 0)
 		(unit 1)
 		(body_style 1)
@@
 		(fields_autoplaced yes)
 		(property "Reference" "U2"
-			(at 110.49 82.55 0)
+			(at 152.4 80.01 0)
 			(show_name no)
 			(do_not_autoplace no)
@@
 		)
 		(property "Value" "LSM6DSOXTR"
-			(at 110.49 85.09 0)
+			(at 152.4 82.55 0)
 			(show_name no)
 			(do_not_autoplace no)
@@
 		)
 		(property "Footprint" "XWatch_Rev1.0:LSM6DSOXTR"
-			(at 110.49 97.79 0)
+			(at 152.4 95.25 0)
 			(hide yes)
 			(show_name no)
@@
 		)
 		(property "Datasheet" "https://www.lcsc.com/datasheet/lcsc_datasheet_2003181935_STMicroelectronics-LSM6DSOXTR_C481766.pdf"
-			(at 110.49 97.79 0)
+			(at 152.4 95.25 0)
 			(hide yes)
 			(show_name no)
@@
 		)
 		(property "Description" "-40℃~+85℃ 1.71V~3.6V 3uA 9KB IMU (accelerometer + gyroscope) Motion event detection、Synchronization and timestamp SPI、I2C X,Y,Z X,Y,Z ±16g ±2000dps LGA-14 Accelerometers ROHS"
-			(at 110.49 97.79 0)
+			(at 152.4 95.25 0)
 			(hide yes)
 			(show_name no)
@@
 		)
 		(property "LCSC" "C481766"
-			(at 110.49 97.79 0)
+			(at 152.4 95.25 0)
 			(hide yes)
 			(show_name no)
@@
 		)
 		(property "Manufacturer" "STMicroelectronics"
-			(at 110.49 97.79 0)
+			(at 152.4 95.25 0)
 			(hide yes)
 			(show_name no)
@@
 		)
 		(property "Manufacturer Part" "LSM6DSOXTR"
-			(at 110.49 97.79 0)
-			(hide yes)
-			(show_name no)
+			(at 152.4 95.25 0)
+			(hide yes)
+			(show_name no)
