File: hardware/schematic/v1.0/XWatch_Rev1.0/Display.kicad_sch (KiCad schematic)
At the start: 3 parts, among them CN1 FH19C-8S-0.5SH, CN2 504208-2410, IC3 SGM38046YG_TR

Commit message: doc and sch update
Parts:
- added C1, C2, C3, C4: 100nF, XWatch_Rev1.0:GEN_C_0201, symbol XWatch_Rev1.0:C
- added R1: 4K7, XWatch_Rev1.0:GEN_R_0201, symbol XWatch_Rev1.0:R
- added R2, R3: R, XWatch_Rev1.0:GEN_R_0201, symbol XWatch_Rev1.0:R
Connections:
- net GND: now reaches CN1.1 (GND)
- net GND: now also CN1.10, CN1.6 (GND), CN1.9, CN2.1 (GND), CN2.10 (GND), CN2.12 (GND), CN2.13 (GND), CN2.14 (GND), CN2.17 (GND), CN2.18 (GND), CN2.25 (PAD), CN2.26 (PAD), CN2.27 (PAD), CN2.28 (PAD), CN2.7 (GND), C1.2, C2.2, C3.2, C4.2
- net DSI_INT: now reaches CN1.2 (INT)
- net DSI_INT: now also R1.2
- net DSI_RST: now reaches CN1.3 (RESET)
- net DSI_RST: now also CN2.2 (XRES)
- net I2C1_SCL: now reaches CN1.4 (SCL)
- net I2C1_SCL: now also R3.2
- net I2C1_SDA: now reaches CN1.5 (SDA)
- net I2C1_SDA: now also R2.2
- net VDD: now reaches CN1.7 (IOVCC)
- net VDD: now also CN2.15 (VDDIO), C1.1, C3.1, R1.1, R2.1, R3.1
- net +3V3: now reaches CN1.8 (VCC)
- net +3V3: now also CN2.16 (VCI), C2.1, C4.1
- net HSSI_CLK_P: now reaches CN2.11 (DSI_CLKP)
- net ELVSS: now reaches CN2.19 (ELVSS)
- net ELVSS: now also CN2.21 (ELVSS), CN2.23 (ELVSS)
- net ELVDD: now reaches CN2.20 (ELVDD)
- net ELVDD: now also CN2.22 (ELVDD), CN2.24 (ELVDD)
- net HSSI_D0_N: now reaches CN2.3 (DSI_D0N)
- net SWIRE: now reaches CN2.4 (SWIRE)
- net HSSI_D0_P: now reaches CN2.5 (DSI_D0P)
- net DSI_TE: now reaches CN2.8 (TE)
- net HSSI_CLK_N: now reaches CN2.9 (DSI_CLKN)
- no-connect marks 0 -> 1
Other:
- note added: "390x390 pixels DSI LCD ZZ1"
- moved on the sheet: CN1, CN2, IC3

Commit message: doc and sch update
Connections:
- net ELVDD: now also IC3.D3 (OVDD)
- net ELVSS: now also IC3.D4 (OVSS)
- net SWIRE: now also IC3.C3 (SWIRE)
- net HSSI_CLK_N renamed DSI_CK_N
- net HSSI_CLK_P renamed DSI_CK_P
- net HSSI_D0_N renamed DSI_D0_N
- net HSSI_D0_P renamed DSI_D0_P
Other:
- note added: "DSI_LANES"
- note added: "I2C"

Commit message: sch and doc update
Parts:
- removed IC3: SGM38046YG_TR, XWatch_Rev1.0:BGA16C50P4X4_200X200X61, symbol XWatch_Rev1.0:SGM38046YG_TR
- added C10, C15, C16, C17, C9: 10uF, XWatch_Rev1.0:GEN_C_0402, symbol XWatch_Rev1.0:C
- added C11, C12: 4.7uF, XWatch_Rev1.0:GEN_C_0402, symbol XWatch_Rev1.0:C
- added C14: 1uF, XWatch_Rev1.0:GEN_C_0402, symbol XWatch_Rev1.0:C
- added IC5: SGM38046YG_TR, XWatch_Rev1.0:BGA16C50P4X4_200X200X61, symbol XWatch_Rev1.0:SGM38046YG_TR
- added L1: 1uH, XWatch_Rev1.0:L_0402_1005Metric, symbol XWatch_Rev1.0:L
Connections:
- net +3V3: no longer C2.1, CN2.16 (VCI)
- net DSI_BL_CTRL: now also IC5.C2 (AVDDEN)
- net ELVDD: now also C15.1, IC5.D3 (OVDD)
- net ELVSS: now also C9.1, IC5.D4 (OVSS)
- net GND: now also C10.1, C11.2, C12.1, C15.2, C16.1, C17.1, C9.2, IC5.A3 (AGND), IC5.B2 (PGND), IC5.B3 (CPGND)
- net SWIRE: now also IC5.C3 (SWIRE)
- net DSI_INT renamed DS_INT
- net DSI_RST renamed DS_RST
- new net: C11.1, IC5.C4 (VON)
- new net: C17.2, IC5.D1 (VOUT)
- new net: C14.1, IC5.A4 (C1P)
- new net: IC5.B1 (SW1), L1.1
- new net: C14.2, IC5.B4 (C1N)
- new net: IC5.C1 (SW2), L1.2
- new net VCI: C16.2, C2.1, CN2.16 (VCI), IC5.D2 (AVDD)
- new net VSYS: C10.2, C12.2, IC5.A1 (PVIN), IC5.A2 (AVIN)

Commit message: doc and sch update
Connections:
- net DSI_BL_CTRL renamed DSI_AVDDEN
Changed lines of the file:
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@@
 		)
 	)
-	(hierarchical_label "DSI_BL_CTRL"
+	(hierarchical_label "DSI_AVDDEN"
 		(shape bidirectional)
 		(at 40.64 172.72 180)

Commit message: sch update
Parts:
- R2, R3: value R -> 1K5; now fitted
Connections:
- net DSI_AVDDEN renamed DSI.AVDDEN
- net DSI_CK_N renamed DSI.CK_N
- net DSI_CK_P renamed DSI.CK_P
- net DSI_D0_N renamed DSI.D0_N
- net DSI_D0_P renamed DSI.D0_P
- net DSI_TE renamed DSI.TE
- net DS_INT renamed TP.INT
- net DS_RST renamed DSI_RST
- net DSI_RST: no longer CN1.3 (RESET)
- net I2C1_SCL renamed TP.SCL
- net I2C1_SDA renamed TP.SDA
- new net TP.RST: CN1.3 (RESET)
Other:
- note added: "Touch Panel"
- note removed: "I2C"
- moved on the sheet: R1
