File: hardware/schematic/v1.0/XWatch_Rev1.0/MCU.kicad_sch (KiCad schematic)
At the start: 1 part, among them U1 STM32L4R9AII6U

Commit message: doc and sch update
Parts:
- added R4, R5: 1K5, XWatch_Rev1.0:GEN_R_0201, symbol XWatch_Rev1.0:R
Connections:
- net GND: now reaches U1.A7 (VSS_1/IO_2)
- net GND: now also U1.B3 (VSS_3/13), U1.C12 (VSS_2), U1.C2 (VSS_10), U1.F13 (VSSIO_1), U1.F2 (VSS_5), U1.H12 (VSS_8/9_0/11), U1.H2 (VSS_4/6), U1.J13 (DSI_VSS_0), U1.K13 (DSI_VSS_1), U1.K2 (VSSA/VREF-), U1.M11 (VSS_12), U1.M3 (VSS_9), U1.M7 (VSS_7)
- net DSI_VCAP: now reaches U1.L13 (DSI_VCAP_0)
- net DSI_SPI_CS: now reaches U1.A13 (PH14)
- net MFX_IRQ_OUT: now reaches U1.B11 (PI1)
- net I2C1_SDA: now reaches U1.G6 (PG13)
- net I2C1_SDA: now also R5.2
- net DSI_D1_P: now reaches U1.J11 (DSI_D1_P)
- net DSI_D1_N: now reaches U1.J12 (DSI_D1_N)
- net DSI_CK_P: now reaches U1.K11 (DSI_CK_P)
- net DSI_CK_N: now reaches U1.K12 (DSI_CK_N)
- net DSI_D0_P: now reaches U1.L11 (DSI_D0_P)
- net DSI_D0_N: now reaches U1.L12 (DSI_D0_N)
- net SWCLK: now reaches U1.A10 (PA14)
- net SWDIO: now reaches U1.A11 (PA13)
- net SWO: now reaches U1.A6 (PB3)
- net I2C1_SCL: now reaches U1.C5 (PB6)
- net I2C1_SCL: now also R4.2
- net DSI_SWIRE: now reaches U1.E11 (PA8)
- net DSI_SPI_MOSI: now reaches U1.L10 (PB15)
- net DSI_BL_CTRL: now reaches U1.L5 (PB1)
- net DSI_SPI_DCX: now reaches U1.M12 (PB14)
- net USART_RX: now reaches U1.M2 (PA3)
- net DSI_TE: now reaches U1.M5 (PF11)
- net USART_TX: now reaches U1.N1 (PA2-WKUP)
- net DSI_SPI_CK: now reaches U1.N13 (PB13)
- net DSI_USART_CK: now reaches U1.N4 (PB0)
- net MFX_WAKEUP: now reaches U1.N5 (PB2)
- net DSI_USART_TX: now reaches U1.N9 (PB10)
- new net VDD: R4.1, R5.1
Other:
- note added: "DSI LCD"
- note added: "DSI_LANES"
- note added: "DSI_SPI"
- note added: "DSI_USART"
- note added: "MFX"
- note added: "ST LINK"
- moved on the sheet: U1A, U1B, U1C

Commit message: sch and doc update
Parts:
- added C5, C6: 5.6pF, XWatch_Rev1.0:GEN_C_0402, symbol XWatch_Rev1.0:C
- added C7, C8: 10pF, XWatch_Rev1.0:GEN_C_0201, symbol XWatch_Rev1.0:C
- added X1: NX3215SA_32_768KHZ_EXS00A-MU00525, XWatch_Rev1.0:NX3215SA_32_768KHZ_EXS00A-MU00525, symbol XWatch_Rev1.0:NX3215SA_32_768KHZ_EXS00A-MU00525
- added X2: TXM16M0004252CBCEO00T, XWatch_Rev1.0:TXM16M0004252CBCEO00T, symbol XWatch_Rev1.0:TXM16M0004252CBCEO00T
Connections:
- net GND: now also C5.1, C6.1, C7.2, C8.1, X2.4
- net OSC32_IN: now reaches U1.F1 (PC14-OSC32_IN)
- net OSC32_IN: now also C6.2, X1.2
- net OSC32_OUT: now reaches U1.G1 (PC15-OSC32_OUT)
- net OSC32_OUT: now also C5.2, X1.1
- net at U1.H1 (PH0-OSC_IN): now also X2.3 (OSC2)
- net at U1.J1 (PH1-OSC_OUT): now also C7.1, X2.1 (OSC1)
- net DS_RST: now reaches U1.K10 (PD8)
- net DS_INT: now reaches U1.K9 (PD9)
- new net: C8.2, X2.2

Commit message: doc and sch update
Parts:
- added C13, C18, C19, C20, C21, C22, C23, C24, C25, C26, C27, C28, C29, C30: 100nF, XWatch_Rev1.0:GEN_C_0201, symbol XWatch_Rev1.0:C
- added R6: 0, XWatch_Rev1.0:GEN_R_0201, symbol XWatch_Rev1.0:R
Connections:
- net GND: now also C13.2, C18.2, C19.2, C20.2, C21.2, C22.2, C23.2, C24.2, C25.2, C26.2, C27.2, C28.2, C29.2, C30.2
- net +1V8: now reaches U1.A3 (VDD_3/13)
- net +1V8: now also U1.A8 (VDD_9), U1.B6 (VDDIO_2), U1.C1 (VDD_12), U1.C13 (VDD_2), U1.D12 (VDDUSB), U1.F12 (VDDIO_1), U1.G2 (VDD_5), U1.H13 (VDD_8/11), U1.N11 (VDD_1/9_0/10), U1.N3 (VDD_4), U1.N7 (VDD_6/7), C13.1, C18.1, C19.1, C20.1, C21.1, C22.1, C23.1, C24.1, C25.1, C26.1, C27.1, C28.1, C29.1, C30.1, R6.1
- net at U1.E2 (VBAT): now also R6.2
- net DSI_BL_CTRL renamed DSI_AVDDEN
Other:
- moved on the sheet: U1C

Commit message: sch update
Parts:
- removed R4, R5: 1K5, XWatch_Rev1.0:GEN_R_0201, symbol XWatch_Rev1.0:R
Connections:
- net DSI_AVDDEN renamed DSI.AVDDEN
- net DSI_CK_N renamed DSI.CK_N
- net DSI_CK_P renamed DSI.CK_P
- net DSI_D0_N renamed DSI.D0_N
- net DSI_D0_P renamed DSI.D0_P
- net DSI_SPI_CK: no longer names the net of U1.N13 (PB13)
- net DSI_SPI_CS: no longer names the net of U1.A13 (PH14)
- net DSI_SPI_DCX: no longer names the net of U1.M12 (PB14)
- net DSI_SPI_MOSI: no longer names the net of U1.L10 (PB15)
- net DSI_SWIRE renamed DSI.SWIRE
- net DSI_TE renamed DSI.TE
- net DSI_USART_CK: no longer names the net of U1.N4 (PB0)
- net DSI_USART_TX: no longer names the net of U1.N9 (PB10)
- net DS_INT renamed TP.INT
- net DS_RST renamed DSI.RST
- net I2C1_SCL renamed TP.SCL
- net I2C1_SDA renamed TP.SDA
Other:
- note removed: "DSI_SPI"
- note removed: "DSI_USART"
