File: hardware/schematic/v1.0/XWatch_Rev2.0/MCU_PWR.kicad_sch (KiCad schematic)
At the start: 1 part, among them U11 STM32U5G9NJH6Q

Commit message: add rev2.0
Parts:
- U1: renamed from U11; footprint XWatch_Rev1.0:STM32U5G9NJH6Q -> XWatch_Rev2.0:STM32U5G9NJH6Q
Connections:
- net GND: now reaches U1.A1 (VSS)
- net GND: now also U1.A15 (VSS), U1.E10 (VSS), U1.F10 (VSS), U1.F6 (VSS), U1.F7 (VSS), U1.F9 (VSS), U1.G10 (VSS), U1.G6 (VSSDSI), U1.H10 (VSS), U1.H15 (VSS), U1.H2 (VSSDSI), U1.H6 (VSSDSI), U1.J10 (VSS), U1.J15 (VSS), U1.J2 (VSSDSI), U1.J6 (VSS), U1.K10 (VSS), U1.K5 (VREFM), U1.K6 (VSSA), U1.K7 (VSS), U1.K8 (VSS), U1.K9 (VSS), U1.L10 (VSS), U1.P12 (VSSSMPS), U1.R1 (VSS), U1.R15 (VSS)

Commit message: sch update
Parts:
- added C20, C21, C22, C23, C24, C25, C26, C27, C28, C29, C31, C32, C35, C37, C38, C39, C40, C43, C44, C45, C47: 100nF, XWatch_Rev2.0:GEN_C_0201, symbol XWatch_Rev2.0:C
- added C30, C46: 10uF, XWatch_Rev2.0:GEN_C_0402, symbol XWatch_Rev2.0:C
- added C33: 4.7uF, XWatch_Rev2.0:GEN_C_0402, symbol XWatch_Rev2.0:C
- added C34, C36: 1uF, XWatch_Rev2.0:GEN_C_0402, symbol XWatch_Rev2.0:C
- added C41, C42: 2.2uF, XWatch_Rev2.0:GEN_C_0402, symbol XWatch_Rev2.0:C
- added FB1: 0, symbol XWatch_Rev2.0:FerriteBead_Small
- added L3: 2.2uH, XWatch_Rev2.0:L_0402_1005Metric, symbol XWatch_Rev2.0:L
Connections:
- net +1V8: now also U1.C2 (VBAT), U1.E8 (VDDIO2), U1.E9 (VDDUSB), U1.F5 (VDD), U1.F8 (VDD), U1.G11 (VDDIO2), U1.G5 (VDDDSI), U1.H11 (VDD), U1.J11 (VDD), U1.J5 (VDD), U1.K11 (VDD), U1.L11 (VDD), U1.L7 (VDD), U1.L8 (VDD), U1.L9 (VDD), U1.R12 (VDDSMPS), C20.1, C21.1, C22.1, C23.1, C24.1, C25.1, C26.1, C27.1, C28.1, C29.1, C30.1, C31.1, C32.1, C33.1, C38.1, C39.1, C40.1, C46.1, C47.1, FB1.1
- net GND: now also C20.2, C21.2, C22.2, C23.2, C24.2, C25.2, C26.2, C27.2, C28.2, C29.2, C30.2, C31.2, C32.2, C33.2, C34.2, C35.2, C36.2, C37.2, C38.2, C39.2, C40.2, C41.2, C42.2, C43.2, C44.2, C45.2, C46.2, C47.2
- net VDD11: now reaches U1.E11 (VDD11)
- net VDD11: now also U1.E6 (VDD11), U1.F11 (VDD11USB), U1.H5 (VDD11DSI), U1.R13 (VDD11), C41.1, C42.1, C43.1, C44.1, C45.1, L3.1
- net at U1.L5 (VREFP): now also U1.L6 (VDDA), C34.1, C35.1, C36.1, C37.1, FB1.2
- net at U1.R11 (VLXSMPS): now also L3.2
Other:
- note added: "10uF靠近BGA"
- note added: "CIN"
- note added: "USB不用，接VDD"
- note added: "VDDA"
- note added: "VREF+"
- note added: "全部直接 打孔到 整层 GND （不分割 AGND）"
- note added: "可选"
- note added: "无备份电池，接VDD"
- note added: "每个 VDD 球 1 颗100nF"
- note added: "每球 1 颗100nF"
- note added: "靠近G5"
- note added: "靠近L5"
- note added: "靠近L6"
- note added: "靠近R13"
- note added: "须接VDD11"
