File: hardware/schematic/v1.0/XWatch_Rev2.0/SENSOR.kicad_sch (KiCad schematic)
At the start: 2 parts, among them U6 LSM6DSOXTR, U7 LIS2MDLTR

Commit message: doc and sch update
Parts:
- added R11, R12: 4.7K, XWatch_Rev2.0:GEN_R_0201, symbol XWatch_Rev2.0:R
- added U10: OPT3001DNPR, XWatch_Rev2.0:OPT3001DNPR, symbol XWatch_Rev2.0:OPT3001DNPR
- added U11: MAX30101EFD_T, XWatch_Rev2.0:MAX30101EFD_T, symbol XWatch_Rev2.0:MAX30101EFD_T
- added U9: LPS27HHWTR, XWatch_Rev2.0:LPS27HHWTR, symbol XWatch_Rev2.0:LPS27HHWTR
Connections:
- new net +1V8: R11.1, R12.1
- new net SENSOR_SCL: R12.2
- new net SENSOR_SDA: R11.2
Other:
- note added: "3D磁传感器"
- note added: "IMU"
- note added: "气压传感器"
- note added: "环境光传感器"

Commit message: sch update
Parts:
- added U12: DRV2605LDGSR, XWatch_Rev2.0:DRV2605LDGSR, symbol XWatch_Rev2.0:DRV2605LDGSR
Other:
- note added: "触觉驱动芯片"
- moved on the sheet: U7
Changed lines of the file:
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@@
 	(text "\n3D磁传感器"
 		(exclude_from_sim no)
-		(at 87.884 146.304 0)
+		(at 94.234 124.714 0)
+		(effects
+			(font
+				(size 1.27 1.27)
+			)
+		)
+	)
+	(text "触觉驱动芯片"
+		(exclude_from_sim no)
+		(at 102.108 168.656 0)
 		(effects
 			(font
@@
 	(symbol
 		(lib_id "XWatch_Rev2.0:LIS2MDLTR")
-		(at 87.63 135.89 0)
+		(at 93.98 114.3 0)
 		(unit 1)
 		(body_style 1)
@@
 		(fields_autoplaced yes)
 		(property "Reference" "U7"
-			(at 87.63 121.92 0)
+			(at 93.98 100.33 0)
 			(show_name no)
 			(do_not_autoplace no)
@@
 		)
 		(property "Value" "LIS2MDLTR"
-			(at 87.63 124.46 0)
+			(at 93.98 102.87 0)
 			(show_name no)
 			(do_not_autoplace no)
@@
 		)
 		(property "Footprint" "XWatch_Rev2.0:LIS2MDLTR"
-			(at 87.63 135.89 0)
+			(at 93.98 114.3 0)
 			(hide yes)
 			(show_name no)
@@
 		)
 		(property "Datasheet" "https://www.lcsc.com/datasheet/lcsc_datasheet_2111191730_STMicroelectronics-LIS2MDLTR_C919695.pdf"
-			(at 87.63 135.89 0)
+			(at 93.98 114.3 0)
 			(hide yes)
 			(show_name no)
@@
 		)
 		(property "Description" "-40℃~+85℃ 1.71V~3.6V 16bit 200uA I2C、SPI ±5mT ±5mT LGA-12(2x2) 3D Magnetic Sensors ROHS"
-			(at 87.63 135.89 0)
+			(at 93.98 114.3 0)
 			(hide yes)
 			(show_name no)
@@
 		)
 		(property "LCSC" "C919695"
-			(at 87.63 135.89 0)
+			(at 93.98 114.3 0)
 			(hide yes)
 			(show_name no)
@@
 		)
 		(property "Manufacturer" "STMicroelectronics"
-			(at 87.63 135.89 0)
+			(at 93.98 114.3 0)
 			(hide yes)
 			(show_name no)
@@
 		)
 		(property "Manufacturer Part" "LIS2MDLTR"
-			(at 87.63 135.89 0)
+			(at 93.98 114.3 0)
 			(hide yes)
 			(show_name no)
@@
 					(unit 1)
 				)
+			)
+		)
+	)
+	(symbol
+		(lib_id "XWatch_Rev2.0:DRV2605LDGSR")
+		(at 102.87 157.48 0)
+		(unit 1)
+		(body_style 1)
+		(exclude_from_sim no)
+		(in_bom yes)
+		(on_board yes)
+		(in_pos_files yes)
+		(dnp no)
+		(fields_autoplaced yes)
+		(property "Reference" "U12"
+			(at 102.87 144.78 0)
+			(show_name no)
+			(do_not_autoplace no)
+			(effects
+				(font
+					(size 1.27 1.27)
+				)
+			)
+		)
+		(property "Value" "DRV2605LDGSR"
+			(at 102.87 147.32 0)
+			(show_name no)
+			(do_not_autoplace no)
+			(effects
+				(font
+					(size 1.27 1.27)
+				)
+			)
+		)
+		(property "Footprint" "XWatch_Rev2.0:DRV2605LDGSR"
+			(at 102.87 157.48 0)
+			(hide yes)
+			(show_name no)
+			(do_not_autoplace no)
+			(effects
+				(font
+					(size 1.27 1.27)
+				)
+			)
+		)
+		(property "Datasheet" "https://www.lcsc.com/datasheet/lcsc_datasheet_2005142220_Texas-Instruments-DRV2605LDGSR_C527464.pdf"
+			(at 102.87 157.48 0)
+			(hide yes)
+			(show_name no)
+			(do_not_autoplace no)
+			(effects
+				(font
+					(size 1.27 1.27)
+				)
+			)
+		)
+		(property "Description" "-40℃~+85℃ 1 2V~5.2V 500uA I2C Yes VSSOP-10-0.5mm Brushed DC Motor Drivers ROHS"
+			(at 102.87 157.48 0)
+			(hide yes)
+			(show_name no)
+			(do_not_autoplace no)
+			(effects
+				(font
+					(size 1.27 1.27)
+				)
+			)
+		)
+		(property "LCSC" "C527464"
+			(at 102.87 157.48 0)
+			(hide yes)
+			(show_name no)
+			(do_not_autoplace no)
+			(effects
+				(font
+					(size 1.27 1.27)
+				)
+			)
+		)
+		(property "Manufacturer" "Texas Instruments"
+			(at 102.87 157.48 0)
+			(hide yes)
+			(show_name no)
+			(do_not_autoplace no)
+			(effects
+				(font
+					(size 1.27 1.27)
+				)
+			)
+		)
+		(property "Manufacturer Part" "DRV2605LDGSR"
+			(at 102.87 157.48 0)
+			(hide yes)
+			(show_name no)
+			(do_not_autoplace no)
+			(effects
+				(font
+					(size 1.27 1.27)
+				)
+			)
+		)
+		(pin "6"
+		)
+		(pin "2"
+		)
+		(pin "8"
+		)
+		(pin "7"
+		)
+		(pin "1"
+		)
+		(pin "4"
+		)
+		(pin "5"
+		)
+		(pin "10"
+		)
+		(pin "3"
+		)
+		(pin "9"
+		)
+		(instances
+			(project "XWatch_Rev2.0"
+				(path "/64425c00-526a-4829-b8a6-ed1dc1b19578/0fbd71dc-4ace-4821-a549-b0309b8febde"
+					(reference "U12")
+					(unit 1)
+				)

Commit message: sch update
Connections:
- net VBAT: now reaches U12.10 (VDD)
Changed lines of the file:
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@@
 	(generator_version "10.0")
 	(paper "A4")
+	(text "触觉驱动芯片"
+		(exclude_from_sim no)
+		(at 121.158 177.546 0)
+		(effects
+			(font
+				(size 1.27 1.27)
+			)
+		)
+	)
 	(text "IMU"
 		(exclude_from_sim no)
@@
 		)
 	)
-	(text "触觉驱动芯片"
-		(exclude_from_sim no)
-		(at 102.108 168.656 0)
-		(effects
-			(font
-				(size 1.27 1.27)
-			)
-		)
-	)
 	(junction
 		(at 223.52 128.27)
@@
 	(wire
 		(pts
+			(xy 140.97 160.02) (xy 140.97 161.29)
+		)
+		(stroke
+			(width 0)
+			(type default)
+		)
+	)
+	(wire
+		(pts
 			(xy 223.52 128.27) (xy 223.52 130.81)
+		)
+		(stroke
+			(width 0)
+			(type default)
+		)
+	)
+	(wire
+		(pts
+			(xy 137.16 161.29) (xy 140.97 161.29)
 		)
 		(stroke
@@
 				(path "/64425c00-526a-4829-b8a6-ed1dc1b19578/0fbd71dc-4ace-4821-a549-b0309b8febde"
 					(reference "R11")
+					(unit 1)
+				)
+			)
+		)
+	)
+	(symbol
+		(lib_id "XWatch_Rev2.0:VBAT")
+		(at 140.97 160.02 0)
+		(unit 1)
+		(body_style 1)
+		(exclude_from_sim no)
+		(in_bom yes)
+		(on_board yes)
+		(in_pos_files yes)
+		(dnp no)
+		(fields_autoplaced yes)
+		(property "Reference" "#PWR09"
+			(at 140.97 163.83 0)
+			(hide yes)
+			(show_name no)
+			(do_not_autoplace no)
+			(effects
+				(font
+					(size 1.27 1.27)
+				)
+			)
+		)
+		(property "Value" "VBAT"
+			(at 140.97 154.94 0)
+			(show_name no)
+			(do_not_autoplace no)
+			(effects
+				(font
+					(size 1.27 1.27)
+				)
+			)
+		)
+		(property "Footprint" ""
+			(at 140.97 160.02 0)
+			(hide yes)
+			(show_name no)
+			(do_not_autoplace no)
+			(effects
+				(font
+					(size 1.27 1.27)
+				)
+			)
+		)
+		(property "Datasheet" ""
+			(at 140.97 160.02 0)
+			(hide yes)
+			(show_name no)
+			(do_not_autoplace no)
+			(effects
+				(font
+					(size 1.27 1.27)
+				)
+			)
+		)
+		(property "Description" "Power symbol creates a global label with name \"VBAT\""
+			(at 140.97 160.02 0)
+			(hide yes)
+			(show_name no)
+			(do_not_autoplace no)
+			(effects
+				(font
+					(size 1.27 1.27)
+				)
+			)
+		)
+		(pin "1"
+		)
+		(instances
+			(project "XWatch_Rev2.0"
+				(path "/64425c00-526a-4829-b8a6-ed1dc1b19578/0fbd71dc-4ace-4821-a549-b0309b8febde"
+					(reference "#PWR09")
 					(unit 1)
 				)
@@
 	)
 	(symbol
-		(lib_id "XWatch_Rev2.0:DRV2605LDGSR")
-		(at 102.87 157.48 0)
-		(unit 1)
-		(body_style 1)
-		(exclude_from_sim no)
-		(in_bom yes)
-		(on_board yes)
-		(in_pos_files yes)
-		(dnp no)
-		(fields_autoplaced yes)
-		(property "Reference" "U12"
-			(at 102.87 144.78 0)
-			(show_name no)
-			(do_not_autoplace no)
-			(effects
-				(font
-					(size 1.27 1.27)
-				)
-			)
-		)
-		(property "Value" "DRV2605LDGSR"
-			(at 102.87 147.32 0)
-			(show_name no)
-			(do_not_autoplace no)
-			(effects
-				(font
-					(size 1.27 1.27)
-				)
-			)
-		)
-		(property "Footprint" "XWatch_Rev2.0:DRV2605LDGSR"
-			(at 102.87 157.48 0)
-			(hide yes)
-			(show_name no)
-			(do_not_autoplace no)
-			(effects
-				(font
-					(size 1.27 1.27)
-				)
-			)
-		)
-		(property "Datasheet" "https://www.lcsc.com/datasheet/lcsc_datasheet_2005142220_Texas-Instruments-DRV2605LDGSR_C527464.pdf"
-			(at 102.87 157.48 0)
-			(hide yes)
-			(show_name no)
-			(do_not_autoplace no)
-			(effects
-				(font
-					(size 1.27 1.27)
-				)
-			)
-		)
-		(property "Description" "-40℃~+85℃ 1 2V~5.2V 500uA I2C Yes VSSOP-10-0.5mm Brushed DC Motor Drivers ROHS"
-			(at 102.87 157.48 0)
-			(hide yes)
-			(show_name no)
-			(do_not_autoplace no)
-			(effects
-				(font
-					(size 1.27 1.27)
-				)
-			)
-		)
-		(property "LCSC" "C527464"
-			(at 102.87 157.48 0)
-			(hide yes)
-			(show_name no)
-			(do_not_autoplace no)
-			(effects
-				(font
-					(size 1.27 1.27)
-				)
-			)
-		)
-		(property "Manufacturer" "Texas Instruments"
-			(at 102.87 157.48 0)
-			(hide yes)
-			(show_name no)
-			(do_not_autoplace no)
-			(effects
-				(font
-					(size 1.27 1.27)
-				)
-			)
-		)
-		(property "Manufacturer Part" "DRV2605LDGSR"
-			(at 102.87 157.48 0)
-			(hide yes)
-			(show_name no)
-			(do_not_autoplace no)
-			(effects
-				(font
-					(size 1.27 1.27)
-				)
-			)
-		)
-		(pin "6"
-		)
-		(pin "2"
-		)
-		(pin "8"
-		)
-		(pin "7"
-		)
-		(pin "1"
-		)
-		(pin "4"
-		)
-		(pin "5"
-		)
-		(pin "10"
-		)
-		(pin "3"
-		)
-		(pin "9"
-		)
-		(instances
-			(project "XWatch_Rev2.0"
-				(path "/64425c00-526a-4829-b8a6-ed1dc1b19578/0fbd71dc-4ace-4821-a549-b0309b8febde"
-					(reference "U12")
-					(unit 1)
-				)
-			)
-		)
-	)
-	(symbol
 		(lib_id "XWatch_Rev2.0:MAX30101EFD_T")
 		(at 224.79 87.63 0)
@@
 					(unit 1)
 				)
+			)
+		)
+	)
+	(symbol
+		(lib_id "XWatch_Rev2.0:DRV2605LDGSR")
+		(at 121.92 166.37 0)
+		(unit 1)
+		(body_style 1)
+		(exclude_from_sim no)
+		(in_bom yes)
+		(on_board yes)
+		(in_pos_files yes)
+		(dnp no)
+		(fields_autoplaced yes)
+		(property "Reference" "U12"
+			(at 121.92 153.67 0)
+			(show_name no)
+			(do_not_autoplace no)
+			(effects
+				(font
+					(size 1.27 1.27)
+				)
+			)
+		)
+		(property "Value" "DRV2605LDGSR"
+			(at 121.92 156.21 0)
+			(show_name no)
+			(do_not_autoplace no)
+			(effects
+				(font
+					(size 1.27 1.27)
+				)
+			)
+		)
+		(property "Footprint" "XWatch_Rev2.0:DRV2605LDGSR"
+			(at 121.92 166.37 0)
+			(hide yes)
+			(show_name no)
+			(do_not_autoplace no)
+			(effects
+				(font
+					(size 1.27 1.27)
+				)
+			)
+		)
+		(property "Datasheet" "https://www.lcsc.com/datasheet/lcsc_datasheet_2005142220_Texas-Instruments-DRV2605LDGSR_C527464.pdf"
+			(at 121.92 166.37 0)
+			(hide yes)
+			(show_name no)
+			(do_not_autoplace no)
+			(effects
+				(font
+					(size 1.27 1.27)
+				)
+			)
+		)
+		(property "Description" "-40℃~+85℃ 1 2V~5.2V 500uA I2C Yes VSSOP-10-0.5mm Brushed DC Motor Drivers ROHS"
+			(at 121.92 166.37 0)
+			(hide yes)
+			(show_name no)
+			(do_not_autoplace no)
+			(effects
+				(font
+					(size 1.27 1.27)
+				)
+			)
+		)
+		(property "LCSC" "C527464"
+			(at 121.92 166.37 0)
+			(hide yes)
+			(show_name no)
+			(do_not_autoplace no)
+			(effects
+				(font
+					(size 1.27 1.27)
+				)
+			)
+		)
+		(property "Manufacturer" "Texas Instruments"
+			(at 121.92 166.37 0)
+			(hide yes)
+			(show_name no)
+			(do_not_autoplace no)
+			(effects
+				(font
+					(size 1.27 1.27)
+				)
+			)
+		)
+		(property "Manufacturer Part" "DRV2605LDGSR"
+			(at 121.92 166.37 0)
+			(hide yes)
+			(show_name no)
+			(do_not_autoplace no)
+			(effects
+				(font
+					(size 1.27 1.27)
+				)
+			)
+		)
+		(pin "6"
+		)
+		(pin "2"
+		)
+		(pin "8"
+		)
+		(pin "7"
+		)
+		(pin "1"
+		)
+		(pin "4"
+		)
+		(pin "5"
+		)
+		(pin "10"
+		)
+		(pin "3"
+		)
+		(pin "9"
+		)
+		(instances
+			(project "XWatch_Rev2.0"
+				(path "/64425c00-526a-4829-b8a6-ed1dc1b19578/0fbd71dc-4ace-4821-a549-b0309b8febde"
+					(reference "U12")
+					(unit 1)
+				)

Commit message: sch update
Parts:
- added C50, C51: 100nF, XWatch_Rev2.0:GEN_C_0201, symbol XWatch_Rev2.0:C
- R11, R12: value 4.7K -> 2.2K
Connections:
- net +1V8: now also U6.12 (CS), U6.5 (VDDIO), U6.8 (VDD), C50.1, C51.1
- net SENSOR_SCL: now also U6.13 (SCL)
- net SENSOR_SDA: now also U6.14 (SDA)
- net GND: now reaches U6.1 (SDO/SA0)
- net GND: now also U6.2 (SDX), U6.3 (SCX), U6.6 (GND), U6.7 (GND), C50.2, C51.2
- net IMU_INT1: now reaches U6.4 (INT1)
- net IMU_INT2: now reaches U6.9 (INT2)
- no-connect marks 0 -> 2
Other:
- note added: "0x6A"
- note added: "2.2 kΩ（建议）"
- note added: "3 轴磁力计"
- note added: "400 kHz 有充足余量"
- note added: "6 轴 IMU"
- note added: "说明 INT1/INT2 默认推挽、高有效，不加外部上拉； INT1 上电期间不要被外部拉高（手册引脚说明）； SDX/SCX 接 GND，OSC_AUX/SDO_AUX 悬空。"
- note removed: "3D磁传感器"
- note removed: "IMU"
- moved on the sheet: U6

Commit message: sch update
Parts:
- added C52: 220nF, XWatch_Rev2.0:GEN_C_0201, symbol XWatch_Rev2.0:C
- added C53, C54, C55, C56: 100nF, XWatch_Rev2.0:GEN_C_0201, symbol XWatch_Rev2.0:C
Connections:
- net +1V8: now also U7.10 (Vdd_IO), U7.3 (CS), U7.9 (Vdd), U9.1 (Vdd_IO), U9.10 (VDD), U9.6 (CS), C53.1, C54.1, C55.1, C56.2
- net GND: now also U7.6 (GND), U7.8 (GND), U9.11 (GND), U9.3 (Reserved), U9.5 (SDO/SA0), U9.8 (GND), U9.9 (GND), C52.2, C53.2, C54.2, C55.2, C56.1
- net SENSOR_SCL: now also U7.1 (SCL/SPC), U9.2 (SCL/SPC)
- net SENSOR_SDA: now also U7.4 (SDA/SDI/SDO), U9.4 (SDA/SDI/SDO)
- net MAG_C1: now reaches U7.5 (C1)
- net MAG_C1: now also C52.1
- net MAG_DRDY: now reaches U7.7 (INT/DRDY/SDO)
- net BARO_INT: now reaches U9.7 (INT_DRDY)
- no-connect marks 2 -> 5
Other:
- note added: "0x5C"
- note added: "INT_DRDY 默认推挽、高有效"
- note added: "地址固定 0x1E"
- note added: "防水气压计"
- note removed: "气压传感器"
- moved on the sheet: U7, U9

Commit message: sch update
Parts:
- added C57: 100nF, XWatch_Rev2.0:GEN_C_0201, symbol XWatch_Rev2.0:C
- added R15: 10K, XWatch_Rev2.0:GEN_R_0201, symbol XWatch_Rev2.0:R
Connections:
- net +1V8: now also U10.1 (VDD), C57.1, R15.1
- net GND: now also U10.2 (ADDR), U10.3 (GND), U10.7 (EP), C57.2
- net SENSOR_SCL: now also U10.4 (SCL)
- net SENSOR_SDA: now also U10.6 (SDA)
- net ALS_INT_N: now reaches U10.5 (INT)
- net ALS_INT_N: now also R15.2
Other:
- note added: "0x44"
- note added: "INT 为开漏，需上拉"
- note added: "说明 ADDR 可选 GND/VDD/SDA/SCL → 0x44/0x45/0x46/0x47； INT 低有效，可设窗口阈值中断； 感光面朝上，对准表壳透光窗。"
- moved on the sheet: C55, C56, U10, U9

Commit message: sch update
Parts:
- added C58, C60: 100nF, XWatch_Rev2.0:GEN_C_0201, symbol XWatch_Rev2.0:C
- added C59: 10uF, XWatch_Rev2.0:GEN_C_0402, symbol XWatch_Rev2.0:C
- added C61: 1uF, XWatch_Rev2.0:GEN_C_0402, symbol XWatch_Rev2.0:C
- added R16: 10K, XWatch_Rev2.0:GEN_R_0201, symbol XWatch_Rev2.0:R
Connections:
- net +1V8: now also U11.11 (VDD), C60.1, C61.1, R16.1
- net GND: now also U11.12 (GND), U11.4 (PGND), C58.2, C59.2, C60.2, C61.2
- net SENSOR_SCL: now also U11.2 (SCL)
- net SENSOR_SDA: now also U11.3 (SDA)
- net VSYS: now reaches U11.10 (VLED+)
- net VSYS: now also U11.9 (VLED+), C58.1, C59.1
- net PPG_INT_N: now reaches U11.13 (INT#)
- net PPG_INT_N: now also R16.2
- no-connect marks 5 -> 11
Other:
- note added: "INT# 开漏，低有效"
- note added: "贴 9/10 脚 VLED+，承受 LED 脉冲"
- moved on the sheet: U11

Commit message: sch update
Parts:
- added C62, C64: 1uF, XWatch_Rev2.0:GEN_C_0402, symbol XWatch_Rev2.0:C
- added C63: 10uF, XWatch_Rev2.0:GEN_C_0402, symbol XWatch_Rev2.0:C
- added R17: 100K, XWatch_Rev2.0:GEN_R_0201, symbol XWatch_Rev2.0:R
Connections:
- net GND: now also U12.4 (IN/TRIG), U12.8 (GND), C62.2, C63.2, C64.1, R17.2
- net SENSOR_SCL: now also U12.2 (SCL)
- net SENSOR_SDA: now also U12.3 (SDA)
- net VBAT: now also U12.6 (VDD/NC), C62.1, C63.1
- net DRV_REG: now reaches U12.1 (REG)
- net DRV_REG: now also C64.2
- net HAPTIC_EN: now reaches U12.5 (EN)
- net HAPTIC_EN: now also R17.1
Other:
- note added: "内部 LDO 输出，只接电容"
- note added: "贴 10 脚 VDD；VBAT 走线 ≥0.3mm"
