File: hardware/schematic/v1.0/XWatch_Rev2.0/SENSOR.kicad_sch (KiCad schematic)
At the start: 26 parts, among them U10 OPT3001DNPR, U11 MAX30101EFD_T, U12 DRV2605LDGSR, U6 LSM6DSOXTR, U7 LIS2MDLTR, U9 LPS27HHWTR

Commit message: sch update
Connections:
- net LRA_P: now reaches U12.7 (OUT+)
- net LRA_N: now reaches U12.9 (OUT-)
Other:
- note added: "I²C 地址 0x1E"
- note added: "I²C 地址 0x44"
- note added: "I²C 地址 0x57"
- note added: "I²C 地址 0x5A"
- note added: "I²C 地址 0x5C"
- note added: "I²C 地址 0x6A"
- note added: "LRA 触觉驱动"
- note added: "PPG 心率/血氧"
- note removed: "0x44"
- note removed: "0x5C"
- note removed: "0x6A"
- note removed: "地址固定 0x1E"
- note removed: "触觉驱动芯片"
Changed lines of the file:
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@@
 	(generator_version "10.0")
 	(paper "A4")
+	(text "I²C 地址 0x5A"
+		(exclude_from_sim no)
+		(at 121.158 181.356 0)
+		(effects
+			(font
+				(size 1.27 1.27)
+			)
+		)
+	)
 	(text "说明\nINT1/INT2 默认推挽、高有效，不加外部上拉；\nINT1 上电期间不要被外部拉高（手册引脚说明）；\nSDX/SCX 接 GND，OSC_AUX/SDO_AUX 悬空。"
 		(exclude_from_sim no)
@@
 		)
 	)
+	(text "I²C 地址 0x57"
+		(exclude_from_sim no)
+		(at 223.52 91.694 0)
+		(effects
+			(font
+				(size 1.27 1.27)
+			)
+		)
+	)
 	(text "内部 LDO 输出，只接电容"
 		(exclude_from_sim no)
@@
 		)
 	)
-	(text "触觉驱动芯片"
-		(exclude_from_sim no)
-		(at 121.158 177.546 0)
+	(text "I²C 地址 0x5C"
+		(exclude_from_sim no)
+		(at 162.56 69.088 0)
 		(effects
 			(font
@@
 		)
 	)
-	(text "0x6A"
-		(exclude_from_sim no)
-		(at 74.168 70.104 0)
+	(text "I²C 地址 0x6A"
+		(exclude_from_sim no)
+		(at 74.422 70.104 0)
 		(effects
 			(font
@@
 		)
 	)
+	(text "I²C 地址 0x1E"
+		(exclude_from_sim no)
+		(at 75.692 120.904 0)
+		(effects
+			(font
+				(size 1.27 1.27)
+			)
+		)
+	)
 	(text "INT# 开漏，低有效"
 		(exclude_from_sim no)
@@
 		)
 	)
-	(text "0x44"
-		(exclude_from_sim no)
-		(at 164.846 119.634 0)
+	(text "PPG 心率/血氧"
+		(exclude_from_sim no)
+		(at 223.774 88.9 0)
 		(effects
 			(font
@@
 		)
 	)
-	(text "0x5C"
-		(exclude_from_sim no)
-		(at 162.814 68.834 0)
-		(effects
-			(font
-				(size 1.27 1.27)
-			)
-		)
-	)
 	(text "说明\nADDR 可选 GND/VDD/SDA/SCL\n→ 0x44/0x45/0x46/0x47；\nINT 低有效，可设窗口阈值中断；\n感光面朝上，对准表壳透光窗。"
 		(exclude_from_sim no)
@@
 		)
 	)
-	(text "地址固定 0x1E"
-		(exclude_from_sim no)
-		(at 75.946 121.412 0)
+	(text "I²C 地址 0x44"
+		(exclude_from_sim no)
+		(at 164.338 119.634 0)
 		(effects
 			(font
@@
 		(exclude_from_sim no)
 		(at 75.946 117.348 0)
+		(effects
+			(font
+				(size 1.27 1.27)
+			)
+		)
+	)
+	(text "LRA 触觉驱动"
+		(exclude_from_sim no)
+		(at 121.158 177.292 0)
 		(effects
 			(font
@@
 		)
 	)
+	(hierarchical_label "LRA_P"
+		(shape output)
+		(at 137.16 168.91 0)
+		(effects
+			(font
+				(size 1.27 1.27)
+			)
+			(justify left)
+		)
+	)
 	(hierarchical_label "SENSOR_SCL"
 		(shape input)
@@
 		(effects
 			(font
+				(size 1.27 1.27)
+			)
+			(justify left)
+		)
+	)
+	(hierarchical_label "LRA_N"
+		(shape output)
+		(at 137.16 163.83 0)
+		(effects
+			(font

Commit message: sch update
Connections:
- net DRV_REG: no longer names the net of C64.2, U12.1 (REG)
- net MAG_C1: no longer names the net of C52.1, U7.5 (C1)
Changed lines of the file:
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@@
-	)
-	(junction
-		(at 45.72 109.22)
-		(diameter 0)
-		(color 0 0 0 0)
-	)
-	(junction
-		(at 104.14 161.29)
-		(diameter 0)
-		(color 0 0 0 0)
 	)
 	(junction
@@
 	(wire
 		(pts
-			(xy 43.18 109.22) (xy 45.72 109.22)
-		)
-		(stroke
-			(width 0)
-			(type default)
-		)
-	)
-	(wire
-		(pts
 			(xy 232.41 128.27) (xy 232.41 130.81)
 		)
@@
 		(pts
 			(xy 140.97 171.45) (xy 140.97 172.72)
-		)
-		(stroke
-			(width 0)
-			(type default)
-		)
-	)
-	(wire
-		(pts
-			(xy 99.06 161.29) (xy 104.14 161.29)
 		)
 		(stroke
@@
 		)
 	)
-	(hierarchical_label "MAG_C1"
-		(shape output)
-		(at 43.18 109.22 180)
-		(effects
-			(font
-				(size 1.27 1.27)
-			)
-			(justify right)
-		)
-	)
 	(hierarchical_label "LRA_P"
 		(shape output)
@@
 		(effects
 			(font
-				(size 1.27 1.27)
-			)
-			(justify right)
-		)
-	)
-	(hierarchical_label "DRV_REG"
-		(shape input)
-		(at 99.06 161.29 180)
-		(effects
-			(font
