File: hardware/schematic/v1.0/XWatch_Rev2.0/BUTTONS.kicad_sch (KiCad schematic)
At the start: 1 part, among them SW1 EVPAEDB2A

Commit message: sch update
Parts:
- added SW2, SW3, SW4, SW5: EVPAEDB2A, XWatch_Rev2.0:EVPAEDB2A, symbol XWatch_Rev2.0:EVPAEDB2A
Connections:
- net GND: now also SW2.1, SW2.3, SW2.4, SW2.5, SW3.1, SW3.3, SW3.4, SW3.5, SW4.1, SW4.3, SW4.4, SW4.5, SW5.1, SW5.3, SW5.4, SW5.5
- new net SW2: SW2.2
- new net SW3: SW3.2
- new net SW4: SW4.2
- new net SW5: SW5.2

Commit message: sch update
Changed lines of the file:
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@@
 	)
 	(hierarchical_label "SW5"
-		(shape input)
+		(shape output)
 		(at 218.44 121.92 90)
 		(effects
@@
 	)
 	(hierarchical_label "SW2"
-		(shape input)
+		(shape output)
 		(at 88.9 121.92 90)
 		(effects
@@
 	)
 	(hierarchical_label "SW4"
-		(shape input)
+		(shape output)
 		(at 185.42 121.92 90)
 		(effects
@@
 	)
 	(hierarchical_label "SW3"
-		(shape input)
+		(shape output)
 		(at 142.24 121.92 90)
 		(effects

Commit message: sch update
Other:
- note added: "BACK"
- note added: "DOWN"
- note added: "PWR·LIGHT"
- note added: "START·OK"
- note added: "UP·MENU"
- note added: "右上 2 点"
- note added: "右下 4 点"
- note added: "左上 10 点"
- note added: "左下 8 点"
- note added: "左中 9 点"
- note added: "网络 建议引脚 EXTI WKUP 备选引脚（同一 WKUP 编号） KEY_MCU（SW1） PA0 EXTI0 WKUP1 PB2、PE4 SW2 PA1 EXTI1 WKUP3 PB6、PE6 SW3 PA2 EXTI2 WKUP4 PB1、PB7 SW4 PA3 EXTI3 WKUP5 PB8、PC5 SW5 PA4 EXTI4 WKUP2 PC13、PE5"
- moved on the sheet: SW1, SW2, SW3, SW4, SW5

Commit message: sch update
Other:
- moved on the sheet: SW3, SW5
