File: hardware/schematic/v1.0/XWatch_Rev2.0/PWR.kicad_sch (KiCad schematic)
At the start: 3 parts, among them U3 DA9168, U4 TPS62840DLCR, U5 MAX17048G_T10

Commit message: sch update
Parts:
- added C10, C6, C9: 10uF, XWatch_Rev2.0:GEN_C_0402, symbol XWatch_Rev2.0:C
- added C11, C12, C13: 2.2uF, XWatch_Rev2.0:GEN_C_0402, symbol XWatch_Rev2.0:C
- added C14, C7: 100nF, XWatch_Rev2.0:GEN_C_0402, symbol XWatch_Rev2.0:C
- added C5: 4.7uF, XWatch_Rev2.0:GEN_C_0402, symbol XWatch_Rev2.0:C
- added C8: 47nF, XWatch_Rev2.0:GEN_C_0402, symbol XWatch_Rev2.0:C
- added L1, L2: 2.2uH, XWatch_Rev2.0:L_0402_1005Metric, symbol XWatch_Rev2.0:L
Connections:
- net GND: now reaches U5.1 (CTG)
- net GND: now also U3.A1 (GND), U3.B1 (AGND), U3.E5 (EN), U4.1 (GND), U4.3 (MODE), U4.5 (VSET), U4.6 (STOP), U5.4 (GND), U5.6 (QSTRT), U5.9 (EP), C10.2, C11.2, C12.2, C13.2, C14.2, C5.2, C6.2, C7.2, C9.2
- net VBAT: now reaches U5.2 (CELL)
- net VBAT: now also U5.3 (VDD), C7.1
- net FG_ALRT_N: now reaches U5.5 (ALRT#)
- net PWR_SCL: now reaches U5.7 (SCL)
- net PWR_SCL: now also U3.F5 (SCL)
- net PWR_SDA: now reaches U5.8 (SDA)
- net PWR_SDA: now also U3.E4 (SDA)
- net VSYS: now reaches U4.2 (VIN)
- net VSYS: now also U3.C2,D2,E2,F2 (VSYS), U4.4 (EN), C10.1, C5.1, C9.1, L2.2
- net at U4.7 (SW): now also L1.1
- net +1V8: now reaches U4.8 (VOS)
- net +1V8: now also C6.1, L1.2
- net at U3.A2,B2 (CHG_LX): now also C8.1, L2.1
- net at U3.B5 (VOUT1): now also C12.1
- net at U3.C1,D1,E1,F1 (VBAT): now also C11.1
- net at U3.C3 (VBTS): now also C8.2
- net at U3.D5 (VOUT2): now also C13.1
- net at U3.F3 (VBAT__SNS): now also C14.1

Commit message: sch update
Parts:
- added C15: 4.7uF, XWatch_Rev2.0:GEN_C_0402, symbol XWatch_Rev2.0:C
- added C16, C17: 10uF, XWatch_Rev2.0:GEN_C_0402, symbol XWatch_Rev2.0:C
- added C18, C19: 1uF, XWatch_Rev2.0:GEN_C_0402, symbol XWatch_Rev2.0:C
- added R3: 100K, XWatch_Rev2.0:GEN_R_0201, symbol XWatch_Rev2.0:R
- added R4, R5: 4.7K, XWatch_Rev2.0:GEN_R_0201, symbol XWatch_Rev2.0:R
- added R6, R7: 10K, XWatch_Rev2.0:GEN_R_0201, symbol XWatch_Rev2.0:R
- U3: footprint (none) -> XWatch_Rev2.0:BGA30C40P5X6_214X254X56
Connections:
- net +1V8: now also R4.1, R5.1, R6.1, R7.1
- net FG_ALRT_N: now also R7.2
- net GND: now also C15.2, C16.2, C17.2, C18.2, C19.2, R3.2
- net PWR_SCL: now also R4.2
- net PWR_SDA: now also R5.2
- net VBAT: now also C11.1, C14.1, U3.C1,D1,E1,F1 (VBAT), U3.F3 (VBAT__SNS)
- net at U3.A3,B3 (VMID): now also C16.1, C17.1
- net VBUS: now reaches U3.A4,B4 (VBUS)
- net VBUS: now also U3.A5 (VBUS__SNS), C18.1, C19.1
- net at U3.C4 (REF): now also C15.1
- net PWR_CHG_EN_N: now reaches U3.E3 (CHG__EN_N)
- net PWR_CHG_EN_N: now also R3.1
- net PWR_INT_N: now reaches U3.F4 (INT_N)
- net PWR_INT_N: now also R6.2
Other:
- moved on the sheet: C11, C13

Commit message: sch update
Other:
- note added: "Open-Drain, Active-Low Alert Output."
Changed lines of the file:
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@@
 	(generator_version "10.0")
 	(paper "A4")
+	(text "Open-Drain, Active-Low Alert Output. "
+		(exclude_from_sim no)
+		(at 221.488 106.426 0)
+		(effects
+			(font
+				(size 1.27 1.27)
+			)
+		)
+	)
 	(junction
 		(at 140.97 60.96)
@@
 	)
 	(hierarchical_label "FG_ALRT_N"
-		(shape input)
+		(shape output)
 		(at 241.3 149.86 180)
 		(effects
@@
 	)
 	(hierarchical_label "FG_ALRT_N"
-		(shape input)
+		(shape output)
 		(at 217.17 100.33 0)
 		(effects

Commit message: sch update
Parts:
- C12, C13: now not fitted
Other:
- note added: "VOUT1/VOUT2 不用： 只留电容焊盘，不接负载"
Changed lines of the file:
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@@
 	(generator_version "10.0")
 	(paper "A4")
+	(text "VOUT1/VOUT2 不用：\n只留电容焊盘，不接负载"
+		(exclude_from_sim no)
+		(at 147.32 87.884 0)
+		(effects
+			(font
+				(size 1.27 1.27)
+			)
+		)
+	)
 	(text "Open-Drain, Active-Low Alert Output. "
 		(exclude_from_sim no)
@@
 		(shape input)
 		(at 241.3 138.43 180)
+		(effects
+			(font
+				(size 1.27 1.27)
+			)
+			(justify right)
+		)
+	)
+	(hierarchical_label "PWR_INT_N"
+		(shape output)
+		(at 241.3 153.67 180)
 		(effects
 			(font
@@
 		(on_board yes)
 		(in_pos_files yes)
-		(dnp no)
+		(dnp yes)
 		(property "Reference" "C13"
 			(at 123.952 90.424 0)
@@
 		(on_board yes)
 		(in_pos_files yes)
-		(dnp no)
+		(dnp yes)
 		(property "Reference" "C12"
 			(at 123.952 78.994 0)

Commit message: sch update
Parts:
- added R10: 38.3 k 1%, XWatch_Rev2.0:GEN_R_0201, symbol XWatch_Rev2.0:R
- added R9: 24.9 k 1%, XWatch_Rev2.0:GEN_R_0201, symbol XWatch_Rev2.0:R
- added U8: SM03B-SRSS-TB_LF_SN_P, XWatch_Rev2.0:SM03B-SRSS-TB_LF_SN_P, symbol XWatch_Rev2.0:SM03B-SRSS-TB_LF_SN_P
Connections:
- net GND: now also R10.2, U8.3 (BAT-), U8.4, U8.5
- net VBAT: now also U8.1 (BAT+)
- net at U3.C5 (ILIMIT): now also R9.1
- net BAT_NTC: now reaches U3.D3 (TMP__SNS)
- net BAT_NTC: now also R10.1, R9.2, U8.2 (NTC)
Other:
- note added: "ILIMIT=NTC 分压供电端"
- note added: "不加滤波电容(≤10 nF)"

Commit message: sch update
Parts:
- added C49: 100nF, XWatch_Rev2.0:GEN_C_0402, symbol XWatch_Rev2.0:C
Connections:
- net GND: now also C49.2
- net PWR_RIN_N: now reaches U3.D4 (RIN_N)
- net PWR_RIN_N: now also C49.1
Changed lines of the file:
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@@
 	)
 	(junction
+		(at 128.27 115.57)
+		(diameter 0)
+		(color 0 0 0 0)
+	)
+	(junction
 		(at 132.08 41.91)
 		(diameter 0)
@@
 	)
 	(junction
-		(at 128.27 66.04)
+		(at 120.65 119.38)
 		(diameter 0)
 		(color 0 0 0 0)
 	)
 	(junction
-		(at 158.75 139.7)
+		(at 128.27 66.04)
 		(diameter 0)
 		(color 0 0 0 0)
 	)
 	(junction
-		(at 120.65 119.38)
+		(at 158.75 139.7)
 		(diameter 0)
 		(color 0 0 0 0)
@@
 	(wire
 		(pts
+			(xy 128.27 128.27) (xy 128.27 129.54)
+		)
+		(stroke
+			(width 0)
+			(type default)
+		)
+	)
+	(wire
+		(pts
 			(xy 54.61 149.86) (xy 57.15 149.86)
 		)
@@
 	(wire
 		(pts
+			(xy 128.27 115.57) (xy 128.27 120.65)
+		)
+		(stroke
+			(width 0)
+			(type default)
+		)
+	)
+	(wire
+		(pts
 			(xy 118.11 104.14) (xy 120.65 104.14)
 		)
@@
 	(wire
 		(pts
+			(xy 120.65 119.38) (xy 132.08 119.38)
+		)
+		(stroke
+			(width 0)
+			(type default)
+		)
+	)
+	(wire
+		(pts
 			(xy 209.55 139.7) (xy 213.36 139.7)
 		)
@@
 	(wire
 		(pts
+			(xy 118.11 115.57) (xy 128.27 115.57)
+		)
+		(stroke
+			(width 0)
+			(type default)
+		)
+	)
+	(wire
+		(pts
 			(xy 62.23 41.91) (xy 62.23 43.18)
 		)
@@
 	(wire
 		(pts
-			(xy 120.65 119.38) (xy 123.19 119.38)
+			(xy 133.35 72.39) (xy 146.05 72.39)
 		)
 		(stroke
@@
 	(wire
 		(pts
-			(xy 133.35 72.39) (xy 146.05 72.39)
+			(xy 262.89 124.46) (xy 262.89 127)
 		)
 		(stroke
@@
 	(wire
 		(pts
-			(xy 262.89 124.46) (xy 262.89 127)
+			(xy 62.23 100.33) (xy 67.31 100.33)
 		)
 		(stroke
@@
 	(wire
 		(pts
-			(xy 62.23 100.33) (xy 67.31 100.33)
+			(xy 128.27 66.04) (xy 133.35 66.04)
 		)
 		(stroke
@@
 	(wire
 		(pts
-			(xy 128.27 66.04) (xy 133.35 66.04)
+			(xy 67.31 58.42) (xy 67.31 62.23)
 		)
 		(stroke
@@
 	(wire
 		(pts
-			(xy 67.31 58.42) (xy 67.31 62.23)
+			(xy 185.42 95.25) (xy 189.23 95.25)
 		)
 		(stroke
@@
 	(wire
 		(pts
-			(xy 185.42 95.25) (xy 189.23 95.25)
+			(xy 128.27 115.57) (xy 132.08 115.57)
 		)
 		(stroke
@@
 		)
 	)
+	(hierarchical_label "PWR_RIN_N"
+		(shape output)
+		(at 132.08 115.57 0)
+		(effects
+			(font
+				(size 1.27 1.27)
+			)
+			(justify left)
+		)
+	)
 	(hierarchical_label "PWR_CHG_EN_N"
 		(shape input)
-		(at 123.19 119.38 0)
+		(at 132.08 119.38 0)
 		(effects
 			(font
@@
 	)
 	(symbol
+		(lib_id "XWatch_Rev2.0:C")
+		(at 128.27 124.46 0)
+		(unit 1)
+		(body_style 1)
+		(exclude_from_sim no)
+		(in_bom yes)
+		(on_board yes)
+		(in_pos_files yes)
+		(dnp no)
+		(property "Reference" "C49"
+			(at 123.698 122.174 0)
+			(show_name no)
+			(do_not_autoplace no)
+			(effects
+				(font
+					(size 1.27 1.27)
+				)
+				(justify left)
+			)
+		)
+		(property "Value" "100nF"
+			(at 121.92 127 0)
+			(show_name no)
+			(do_not_autoplace no)
+			(effects
+				(font
+					(size 1.27 1.27)
+				)
+				(justify left)
+			)
+		)
+		(property "Footprint" "XWatch_Rev2.0:GEN_C_0402"
+			(at 129.2352 128.27 0)
+			(hide yes)
+			(show_name no)
+			(do_not_autoplace no)
+			(effects
+				(font
+					(size 1.27 1.27)
+				)
+			)
+		)
+		(property "Datasheet" ""
+			(at 128.27 124.46 0)
+			(hide yes)
+			(show_name no)
+			(do_not_autoplace no)
+			(effects
+				(font
+					(size 1.27 1.27)
+				)
+			)
+		)
+		(property "Description" "Unpolarized capacitor"
+			(at 128.27 124.46 0)
+			(hide yes)
+			(show_name no)
+			(do_not_autoplace no)
+			(effects
+				(font
+					(size 1.27 1.27)
+				)
+			)
+		)
+		(pin "1"
+		)
+		(pin "2"
+		)
+		(instances
+			(project "XWatch_Rev2.0"
+				(path "/64425c00-526a-4829-b8a6-ed1dc1b19578/e10fc6fe-cee5-4ccf-ade7-f348522d306a"
+					(reference "C49")
+					(unit 1)
+				)
+			)
+		)
+	)
+	(symbol
 		(lib_id "power:GND")
 		(at 120.65 128.27 0)
@@
 		(in_pos_files yes)
 		(dnp no)
-		(fields_autoplaced yes)
 		(property "Reference" "R3"
-			(at 123.19 121.9199 0)
+			(at 116.332 121.412 0)
 			(show_name no)
 			(do_not_autoplace no)
@@
 		)
 		(property "Value" "100K"
-			(at 123.19 124.4599 0)
+			(at 114.554 123.952 0)
 			(show_name no)
 			(do_not_autoplace no)
@@
 					(unit 1)
 				)
+			)
+		)
+	)
+	(symbol
+		(lib_id "power:GND")
+		(at 128.27 129.54 0)
+		(unit 1)
+		(body_style 1)
+		(exclude_from_sim no)
+		(in_bom yes)
+		(on_board yes)
+		(in_pos_files yes)
+		(dnp no)
+		(fields_autoplaced yes)
+		(property "Reference" "#PWR0129"
+			(at 128.27 135.89 0)
+			(hide yes)
+			(show_name no)
+			(do_not_autoplace no)
+			(effects
+				(font
+					(size 1.27 1.27)
+				)
+			)
+		)
+		(property "Value" "GND"
+			(at 128.2699 133.35 90)
+			(hide yes)
+			(show_name no)
+			(do_not_autoplace no)
+			(effects
+				(font
+					(size 1.27 1.27)
+				)
+				(justify right)
+			)
+		)
+		(property "Footprint" ""
+			(at 128.27 129.54 0)
+			(hide yes)
+			(show_name no)
+			(do_not_autoplace no)
+			(effects
+				(font
+					(size 1.27 1.27)
+				)
+			)
+		)
+		(property "Datasheet" ""
+			(at 128.27 129.54 0)
+			(hide yes)
+			(show_name no)
+			(do_not_autoplace no)
+			(effects
+				(font
+					(size 1.27 1.27)
+				)
+			)
+		)
+		(property "Description" "Power symbol creates a global label with name \"GND\" , ground"
+			(at 128.27 129.54 0)
+			(hide yes)
+			(show_name no)
+			(do_not_autoplace no)
+			(effects
+				(font
+					(size 1.27 1.27)
+				)
+			)
+		)
+		(pin "1"
+		)
+		(instances
+			(project "XWatch_Rev2.0"
+				(path "/64425c00-526a-4829-b8a6-ed1dc1b19578/e10fc6fe-cee5-4ccf-ade7-f348522d306a"
+					(reference "#PWR0129")
+					(unit 1)
+				)

Commit message: sch update
Parts:
- added C65, C66: 1uF, XWatch_Rev2.0:GEN_C_0402, symbol XWatch_Rev2.0:C
- added R19: 100K, XWatch_Rev2.0:GEN_R_0201, symbol XWatch_Rev2.0:R
- added U13: SK6018D4-33, XWatch_Rev2.0:SK6018D4-33, symbol XWatch_Rev2.0:SK6018D4-33
Connections:
- net GND: now also C65.2, C66.2, R19.2, U13.2 (GND), U13.5 (GND)
- net VSYS: now also C65.1, U13.4 (VIN)
- new net +3V3: C66.1, U13.1 (VOUT)
- new net EN_3V3: R19.1, U13.3 (EN)
Other:
- note added: "1.8V"
- note added: "3.3V"
