File: hardware/schematic/v1.0/XWatch_Rev2.0/PWR.kicad_sch (KiCad schematic)
At the start: 33 parts, among them U13 SK6018D4-33, U3 DA9168, U4 TPS62840DLCR, U5 MAX17048G_T10, U8 SM03B-SRSS-TB_LF_SN_P

Commit message: sch update
Changed lines of the file:
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@@
-		)
-	)
-	(hierarchical_label "PWR_INT_N"
-		(shape output)
-		(at 241.3 153.67 180)
-		(effects
-			(font
-				(size 1.27 1.27)
-			)
-			(justify right)
 		)
 	)
