File: hardware/schematic/v1.0/XWatch_Rev2.0/DSI_LCD.kicad_sch (KiCad schematic)
At the start: 1 part, among them U12 AXE530127

Commit message: add rev2.0
Parts:
- added R1: 0, XWatch_Rev2.0:GEN_R_0201, symbol XWatch_Rev2.0:R
- added R2: 10K, XWatch_Rev2.0:GEN_R_0201, symbol XWatch_Rev2.0:R
- U2: renamed from U12; footprint XWatch_Rev1.0:AXE530127 -> XWatch_Rev2.0:AXE530127
Connections:
- net +1V8: now also R2.1
- net GND: now also R1.1
- net at U2.12: now also R1.2
- net at U2.6: now also R2.2
Other:
- note added: "1.43" 466x466 pixels DSI LCD ZZ1"
- moved on the sheet: U2

Commit message: sch update
Connections:
- net TE renamed DSI_TE
Changed lines of the file:
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@@
+	(wire
+		(pts
+			(xy 74.93 121.92) (xy 91.44 121.92)
+		)
+		(stroke
+			(width 0)
+			(type default)
+		)
+	)
 	(wire
 		(pts
@@
 			(width 0)
 			(type default)
+		)
+	)
+	(label "TE"
+		(at 80.01 121.92 0)
+		(effects
+			(font
+				(size 1.27 1.27)
+			)
+			(justify left bottom)
 		)
 	)
@@
 		)
 	)
+	(hierarchical_label "DSI_TE"
+		(shape output)
+		(at 74.93 121.92 180)
+		(effects
+			(font
+				(size 1.27 1.27)
+			)
+			(justify right)
+		)
+	)

Commit message: sch update
Connections:
- net VBAT renamed VSYS
Changed lines of the file:
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@@
+	)
+	(symbol
+		(lib_id "XWatch_Rev2.0:VSYS")
+		(at 151.13 63.5 0)
+		(unit 1)
+		(body_style 1)
+		(exclude_from_sim no)
+		(in_bom yes)
+		(on_board yes)
+		(in_pos_files yes)
+		(dnp no)
+		(fields_autoplaced yes)
+		(property "Reference" "#PWR03"
+			(at 151.13 67.31 0)
+			(hide yes)
+			(show_name no)
+			(do_not_autoplace no)
+			(effects
+				(font
+					(size 1.27 1.27)
+				)
+			)
+		)
+		(property "Value" "VSYS"
+			(at 151.13 58.42 0)
+			(show_name no)
+			(do_not_autoplace no)
+			(effects
+				(font
+					(size 1.27 1.27)
+				)
+			)
+		)
+		(property "Footprint" ""
+			(at 151.13 63.5 0)
+			(hide yes)
+			(show_name no)
+			(do_not_autoplace no)
+			(effects
+				(font
+					(size 1.27 1.27)
+				)
+			)
+		)
+		(property "Datasheet" ""
+			(at 151.13 63.5 0)
+			(hide yes)
+			(show_name no)
+			(do_not_autoplace no)
+			(effects
+				(font
+					(size 1.27 1.27)
+				)
+			)
+		)
+		(property "Description" "Power symbol creates a global label with name \"VSYS\""
+			(at 151.13 63.5 0)
+			(hide yes)
+			(show_name no)
+			(do_not_autoplace no)
+			(effects
+				(font
+					(size 1.27 1.27)
+				)
+			)
+		)
+		(pin "1"
+		)
+		(instances
+			(project "XWatch_Rev2.0"
+				(path "/64425c00-526a-4829-b8a6-ed1dc1b19578/086d63d7-25af-47fa-acc4-e3e995b262f4"
+					(reference "#PWR03")
+					(unit 1)
+				)
+			)
+		)
 	)
 	(symbol
@@
 					(unit 1)
 				)
-			)
-		)
-	)
-	(symbol
-		(lib_id "power:VBUS")
-		(at 151.13 63.5 0)
-		(unit 1)
-		(body_style 1)
-		(exclude_from_sim no)
-		(in_bom yes)
-		(on_board yes)
-		(in_pos_files yes)
-		(dnp no)
-		(property "Reference" "#PWR055"
-			(at 151.13 67.31 0)
-			(hide yes)
-			(show_name no)
-			(do_not_autoplace no)
-			(effects
-				(font
-					(size 1.27 1.27)
-				)
-			)
-		)
-		(property "Value" "VBAT"
-			(at 151.13 59.436 0)
-			(show_name no)
-			(do_not_autoplace no)
-			(effects
-				(font
-					(size 1.27 1.27)
-				)
-			)
-		)
-		(property "Footprint" ""
-			(at 151.13 63.5 0)
-			(hide yes)
-			(show_name no)
-			(do_not_autoplace no)
-			(effects
-				(font
-					(size 1.27 1.27)
-				)
-			)
-		)
-		(property "Datasheet" ""
-			(at 151.13 63.5 0)
-			(hide yes)
-			(show_name no)
-			(do_not_autoplace no)
-			(effects
-				(font
-					(size 1.27 1.27)
-				)
-			)
-		)
-		(property "Description" "Power symbol creates a global label with name \"VBUS\""
-			(at 151.13 63.5 0)
-			(hide yes)
-			(show_name no)
-			(do_not_autoplace no)
-			(effects
-				(font
-					(size 1.27 1.27)
-				)
-			)
-		)
-		(pin "1"
-		)
-		(instances
-			(project "XWatch_Rev1.0"
-				(path "/2e5e9480-7d2e-4148-a9bf-0ac7d46b20bc/2a0147b1-cbac-4b10-9f04-ad00024f07aa"
-					(reference "#PWR055")
-					(unit 1)
-				)
-			)
-			(project "XWatch_Rev2.0"
-				(path "/64425c00-526a-4829-b8a6-ed1dc1b19578/086d63d7-25af-47fa-acc4-e3e995b262f4"
-					(reference "#PWR055")
-					(unit 1)
-				)

Commit message: sch update
Connections:
- net MIPI_CLKN renamed DSI_CK_N
- net MIPI_CLKP renamed DSI_CK_P
- net MIPI_D0N renamed DSI_D0_N
- net MIPI_D0P renamed DSI_D0_P
- net PWR_EN renamed DSI_PWR_EN
- net RESET renamed DSI_RESET
Other:
- moved on the sheet: R2

Commit message: sch update
Parts:
- added R13, R14: 4.7K, XWatch_Rev2.0:GEN_R_0201, symbol XWatch_Rev2.0:R
Connections:
- net +1V8: now also R13.1, R14.1
- net TP_SCL: now also R14.2
- net TP_SDA: now also R13.2

Commit message: sch update
Parts:
- added R20: 10K, XWatch_Rev2.0:GEN_R_0201, symbol XWatch_Rev2.0:R
Connections:
- net +1V8: now also R20.1
- net TP_INT: now also R20.2
Other:
- moved on the sheet: R14
Changed lines of the file:
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@@
+	)
+	(junction
+		(at 238.76 104.14)
+		(diameter 0)
+		(color 0 0 0 0)
 	)
 	(junction
@@
 	(wire
 		(pts
+			(xy 238.76 104.14) (xy 246.38 104.14)
+		)
+		(stroke
+			(width 0)
+			(type default)
+		)
+	)
+	(wire
+		(pts
 			(xy 110.49 91.44) (xy 110.49 95.25)
 		)
@@
 	(wire
 		(pts
-			(xy 224.79 121.92) (xy 240.03 121.92)
-		)
-		(stroke
-			(width 0)
-			(type default)
-		)
-	)
-	(wire
-		(pts
-			(xy 240.03 114.3) (xy 240.03 121.92)
+			(xy 224.79 121.92) (xy 238.76 121.92)
+		)
+		(stroke
+			(width 0)
+			(type default)
+		)
+	)
+	(wire
+		(pts
+			(xy 238.76 114.3) (xy 238.76 121.92)
 		)
 		(stroke
@@
 	(wire
 		(pts
+			(xy 224.79 124.46) (xy 246.38 124.46)
+		)
+		(stroke
+			(width 0)
+			(type default)
+		)
+	)
+	(wire
+		(pts
 			(xy 119.38 91.44) (xy 127 91.44)
 		)
@@
 	(wire
 		(pts
-			(xy 231.14 104.14) (xy 240.03 104.14)
+			(xy 231.14 104.14) (xy 238.76 104.14)
 		)
 		(stroke
@@
 	(wire
 		(pts
+			(xy 246.38 104.14) (xy 246.38 106.68)
+		)
+		(stroke
+			(width 0)
+			(type default)
+		)
+	)
+	(wire
+		(pts
+			(xy 246.38 114.3) (xy 246.38 124.46)
+		)
+		(stroke
+			(width 0)
+			(type default)
+		)
+	)
+	(wire
+		(pts
 			(xy 147.32 88.9) (xy 153.67 88.9)
 		)
@@
 	(wire
 		(pts
-			(xy 240.03 104.14) (xy 240.03 106.68)
+			(xy 238.76 104.14) (xy 238.76 106.68)
 		)
 		(stroke
@@
 		(shape input)
 		(at 120.65 68.58 180)
+		(effects
+			(font
+				(size 1.27 1.27)
+			)
+			(justify right)
+		)
+	)
+	(hierarchical_label "TP_INT"
+		(shape output)
+		(at 224.79 124.46 180)
 		(effects
 			(font
@@
 	(symbol
 		(lib_id "XWatch_Rev2.0:R")
-		(at 240.03 110.49 0)
+		(at 238.76 110.49 0)
 		(unit 1)
 		(body_style 1)
@@
 		(dnp no)
 		(property "Reference" "R14"
-			(at 235.204 107.95 0)
+			(at 233.934 107.95 0)
 			(show_name no)
 			(do_not_autoplace no)
@@
 		)
 		(property "Value" "4.7K"
-			(at 234.188 112.522 0)
+			(at 232.918 112.522 0)
 			(show_name no)
 			(do_not_autoplace no)
@@
 		)
 		(property "Footprint" "XWatch_Rev2.0:GEN_R_0201"
-			(at 238.252 110.49 90)
+			(at 236.982 110.49 90)
 			(hide yes)
 			(show_name no)
@@
 		)
 		(property "Datasheet" ""
-			(at 240.03 110.49 0)
+			(at 238.76 110.49 0)
 			(hide yes)
 			(show_name no)
@@
 		)
 		(property "Description" "Resistor"
-			(at 240.03 110.49 0)
+			(at 238.76 110.49 0)
 			(hide yes)
 			(show_name no)
@@
 					(unit 1)
 				)
+			)
+		)
+	)
+	(symbol
+		(lib_id "XWatch_Rev2.0:R")
+		(at 246.38 110.49 0)
+		(unit 1)
+		(body_style 1)
+		(exclude_from_sim no)
+		(in_bom yes)
+		(on_board yes)
+		(in_pos_files yes)
+		(dnp no)
+		(property "Reference" "R20"
+			(at 241.554 107.95 0)
+			(show_name no)
+			(do_not_autoplace no)
+			(effects
+				(font
+					(size 1.27 1.27)
+				)
+				(justify left)
+			)
+		)
+		(property "Value" "10K"
+			(at 240.538 112.522 0)
+			(show_name no)
+			(do_not_autoplace no)
+			(effects
+				(font
+					(size 1.27 1.27)
+				)
+				(justify left)
+			)
+		)
+		(property "Footprint" "XWatch_Rev2.0:GEN_R_0201"
+			(at 244.602 110.49 90)
+			(hide yes)
+			(show_name no)
+			(do_not_autoplace no)
+			(effects
+				(font
+					(size 1.27 1.27)
+				)
+			)
+		)
+		(property "Datasheet" ""
+			(at 246.38 110.49 0)
+			(hide yes)
+			(show_name no)
+			(do_not_autoplace no)
+			(effects
+				(font
+					(size 1.27 1.27)
+				)
+			)
+		)
+		(property "Description" "Resistor"
+			(at 246.38 110.49 0)
+			(hide yes)
+			(show_name no)
+			(do_not_autoplace no)
+			(effects
+				(font
+					(size 1.27 1.27)
+				)
+			)
+		)
+		(pin "1"
+		)
+		(pin "2"
+		)
+		(instances
+			(project "XWatch_Rev2.0"
+				(path "/64425c00-526a-4829-b8a6-ed1dc1b19578/086d63d7-25af-47fa-acc4-e3e995b262f4"
+					(reference "R20")
+					(unit 1)
+				)

Commit message: sch update
Parts:
- added C67, C71: 1uF, XWatch_Rev2.0:GEN_C_0402, symbol XWatch_Rev2.0:C
- added C68, C70, C72: 100nF, XWatch_Rev2.0:GEN_C_0402, symbol XWatch_Rev2.0:C
- added C69: 10uF, XWatch_Rev2.0:GEN_C_0402, symbol XWatch_Rev2.0:C
- R1: now fitted
Connections:
- net +1V8: now also C71.2, C72.2
- net +3V3: now also C67.1, C68.1
- net GND: now also C67.2, C68.2, C69.1, C70.1, C71.1, C72.1
- net VSYS: now also C69.2, C70.2
Other:
- note added: "IM0 = 0"
- note added: "IM1 = 0"

Commit message: sch update
Parts:
- removed C67, C71: 1uF, XWatch_Rev2.0:GEN_C_0402, symbol XWatch_Rev2.0:C
- removed C68, C70, C72: 100nF, XWatch_Rev2.0:GEN_C_0402, symbol XWatch_Rev2.0:C
- removed C69: 10uF, XWatch_Rev2.0:GEN_C_0402, symbol XWatch_Rev2.0:C
- removed R1: 0, XWatch_Rev2.0:GEN_R_0201, symbol XWatch_Rev2.0:R
- removed R2: 10K, XWatch_Rev2.0:GEN_R_0201, symbol XWatch_Rev2.0:R
- removed U2: AXE530127, XWatch_Rev2.0:AXE530127, symbol XWatch_Rev1.0:AXE530127
- added C73, C75, C77: 100nF, XWatch_Rev2.0:GEN_C_0402, symbol XWatch_Rev2.0:C
- added C74, C76: 1uF, XWatch_Rev2.0:GEN_C_0402, symbol XWatch_Rev2.0:C
- added C78: 10uF, XWatch_Rev2.0:GEN_C_0402, symbol XWatch_Rev2.0:C
- added R21: 10K, XWatch_Rev2.0:GEN_R_0201, symbol XWatch_Rev2.0:R
- added R22: 0, XWatch_Rev2.0:GEN_R_0201, symbol XWatch_Rev2.0:R
- added U14: AXE530127-DO0143FMST02, XWatch_Rev2.0:AXE530127, symbol XWatch_Rev2.0:AXE530127-DO0143FMST02
Connections:
- net +1V8: now also C75.2, C76.2, R21.1, U14.25 (VDDIO)
- net +3V3: now also C73.1, C74.1, U14.11 (TP_VCC), U14.23 (VCI_IN)
- net DSI_CK_N: now also U14.20 (MIPI_CLKN)
- net DSI_CK_P: now also U14.18 (MIPI_CLKP)
- net DSI_D0_N: now also U14.26 (MIPI_D0N)
- net DSI_D0_P: now also U14.24 (MIPI_D0P)
- net DSI_PWR_EN: now also U14.21 (PWR_EN)
- net DSI_RESET: now also U14.19 (RESET)
- net DSI_TE: now also U14.27 (TE)
- net GND: now also C73.2, C74.2, C77.1, C78.1, R22.1, U14.1 (GND), U14.10 (SDI2), U14.14 (RDX_SDIO0), U14.15 (IM1), U14.16 (GND), U14.17 (IM0), U14.2 (DCX_RS), U14.22 (GND), U14.28 (GND), U14.4 (WRX_SCL), U14.8 (SDI3), U14.Y1, U14.Y2, U14.Z1, U14.Z2
- net TP_INT: now also U14.7 (TP_INT)
- net TP_RESET: now also U14.9 (TP_RESET)
- net TP_SCL: now also U14.3 (TP_SCL)
- net TP_SDA: now also U14.5 (TP_SDA)
- net VSYS: now also C77.2, C78.2, U14.29 (VBAT), U14.30 (VBAT)
- new net: R21.2, U14.6 (CS)
- new net: R22.2, U14.12 (SDO_SDI1)
