File: hardware/schematic/v1.0/XWatch_Rev2.0/MCU_IO.kicad_sch (KiCad schematic)
At the start: 1 part, among them U11 STM32U5G9NJH6Q

Commit message: add rev2.0
Parts:
- added C1, C2: 5.6pF, XWatch_Rev2.0:GEN_C_0201, symbol XWatch_Rev2.0:C
- added C3, C4: 10pF, XWatch_Rev2.0:GEN_C_0201, symbol XWatch_Rev2.0:C
- added X1: 32.768KHZ, XWatch_Rev2.0:NX3215SA_32_768KHZ_EXS00A-MU00525, symbol XWatch_Rev2.0:NX3215SA_32_768KHZ_EXS00A-MU00525
- added X2: 16MHZ, XWatch_Rev2.0:TXM16M0004252CBCEO00T, symbol XWatch_Rev2.0:TXM16M0004252CBCEO00T
- U1: renamed from U11; footprint XWatch_Rev1.0:STM32U5G9NJH6Q -> XWatch_Rev2.0:STM32U5G9NJH6Q
Connections:
- net at U1.B1 (PC14-OSC32_IN): now also C2.2, X1.2
- net at U1.C1 (PC15-OSC32_OUT): now also C1.2, X1.1
- net at U1.N1 (PH0-OSC_IN): now also X2.3 (OSC2)
- net at U1.N2 (PH1-OSC_OUT): now also C4.1, X2.1 (OSC1)
- net DSI_PWR_ON: now reaches U1.C4 (PI5)
- net DSI_TP_RESET: now reaches U1.D5 (PI6)
- net DSI_TP_INT: now reaches U1.M8 (PE8-WKUP7)
- new net: C3.2, X2.2
- new net GND: C1.1, C2.1, C3.1, C4.2, X2.4
Other:
- note added: "PE8"
- note added: "PI5"
- note added: "PI6"

Commit message: sch update
Connections:
- net DSI.CK_N renamed DSI_CK_N
- net DSI.CK_P renamed DSI_CK_P
- net DSI.D0_N renamed DSI_D0_N
- net DSI.D0_P renamed DSI_D0_P
- net DSI.D1_N renamed DSI_D1_N
- net DSI.D1_P renamed DSI_D1_P
- net DSI_PWR_ON renamed DSI_PWR_EN
- net DSI_RESETn renamed DSI_RESET
- net DSI_TP_INT renamed TP_INT
- net DSI_TP_RESET renamed TP_RESET
- net I2C5.SCL renamed TP_SCL
- net I2C5.SDA renamed TP_SDA
Changed lines of the file:
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@@
 		(color 0 0 0 0)
 	)
-	(bus_entry
-		(at 325.12 212.09)
-		(size 2.54 -2.54)
-		(stroke
-			(width 0)
-			(type default)
-		)
-	)
-	(bus_entry
-		(at 325.12 224.79)
-		(size 2.54 -2.54)
-		(stroke
-			(width 0)
-			(type default)
-		)
-	)
-	(bus_entry
-		(at 325.12 203.2)
-		(size 2.54 -2.54)
-		(stroke
-			(width 0)
-			(type default)
-		)
-	)
-	(bus_entry
-		(at 325.12 222.25)
-		(size 2.54 -2.54)
-		(stroke
-			(width 0)
-			(type default)
-		)
-	)
-	(bus_entry
-		(at 325.12 205.74)
-		(size 2.54 -2.54)
-		(stroke
-			(width 0)
-			(type default)
-		)
-	)
-	(bus_entry
-		(at 325.12 209.55)
-		(size 2.54 -2.54)
-		(stroke
-			(width 0)
-			(type default)
-		)
-	)
-	(bus_entry
-		(at 325.12 199.39)
-		(size 2.54 -2.54)
-		(stroke
-			(width 0)
-			(type default)
-		)
-	)
-	(bus_entry
-		(at 325.12 196.85)
-		(size 2.54 -2.54)
-		(stroke
-			(width 0)
-			(type default)
-		)
-	)
 	(wire
 		(pts
@@
 	(wire
 		(pts
-			(xy 311.15 205.74) (xy 325.12 205.74)
+			(xy 311.15 200.66) (xy 325.12 200.66)
 		)
 		(stroke
@@
 	(wire
 		(pts
-			(xy 311.15 199.39) (xy 325.12 199.39)
-		)
-		(stroke
-			(width 0)
-			(type default)
-		)
-	)
-	(bus
-		(pts
-			(xy 327.66 219.71) (xy 327.66 222.25)
+			(xy 311.15 213.36) (xy 325.12 213.36)
 		)
 		(stroke
@@
 	(wire
 		(pts
-			(xy 311.15 209.55) (xy 325.12 209.55)
+			(xy 311.15 204.47) (xy 325.12 204.47)
 		)
 		(stroke
@@
 		)
 	)
-	(bus
-		(pts
-			(xy 327.66 219.71) (xy 330.2 219.71)
-		)
-		(stroke
-			(width 0)
-			(type default)
-		)
-	)
 	(wire
 		(pts
@@
 		)
 	)
-	(bus
-		(pts
-			(xy 327.66 194.31) (xy 327.66 209.55)
-		)
-		(stroke
-			(width 0)
-			(type default)
-		)
-	)
 	(wire
 		(pts
@@
 	(wire
 		(pts
-			(xy 311.15 212.09) (xy 325.12 212.09)
+			(xy 311.15 207.01) (xy 325.12 207.01)
 		)
 		(stroke
@@
 	(wire
 		(pts
-			(xy 311.15 203.2) (xy 325.12 203.2)
+			(xy 311.15 198.12) (xy 325.12 198.12)
 		)
 		(stroke
@@
 		)
 	)
-	(bus
-		(pts
-			(xy 327.66 194.31) (xy 330.2 194.31)
-		)
-		(stroke
-			(width 0)
-			(type default)
-		)
-	)
 	(wire
 		(pts
@@
 	(wire
 		(pts
-			(xy 311.15 196.85) (xy 325.12 196.85)
+			(xy 311.15 210.82) (xy 325.12 210.82)
 		)
 		(stroke
@@
 		)
 	)
-	(label "DSI_RESETn"
+	(label "DSI.RESET"
 		(at 158.75 55.88 0)
 		(effects
@@
 	)
 	(label "DSI.CK_N"
-		(at 311.15 199.39 0)
+		(at 311.15 213.36 0)
 		(effects
 			(font
@@
 		)
 	)
-	(label "DSI_TE"
+	(label "DSI.TE"
 		(at 311.15 232.41 0)
 		(effects
@@
 		)
 	)
-	(label "DSI_PWR_ON"
+	(label "DSI_PWR_EN"
 		(at 367.03 238.76 0)
 		(effects
@@
 	)
 	(label "DSI.D0_N"
-		(at 311.15 205.74 0)
+		(at 311.15 200.66 0)
 		(effects
 			(font
@@
 	)
 	(label "DSI.D1_P"
-		(at 311.15 209.55 0)
+		(at 311.15 204.47 0)
 		(effects
 			(font
@@
 		)
 	)
-	(label "DSI_TE"
+	(label "DSI.TE"
 		(at 158.75 162.56 0)
 		(effects
@@
 	)
 	(label "DSI.CK_P"
-		(at 311.15 196.85 0)
+		(at 311.15 210.82 0)
 		(effects
 			(font
@@
 	)
 	(label "DSI.D0_P"
-		(at 311.15 203.2 0)
-		(effects
-			(font
-				(size 1.27 1.27)
-			)
-			(justify left bottom)
-		)
-	)
-	(label "DSI_RESETn"
+		(at 311.15 198.12 0)
+		(effects
+			(font
+				(size 1.27 1.27)
+			)
+			(justify left bottom)
+		)
+	)
+	(label "DSI.RESET"
 		(at 311.15 238.76 0)
 		(effects
@@
 	)
 	(label "DSI.D1_N"
-		(at 311.15 212.09 0)
-		(effects
-			(font
-				(size 1.27 1.27)
-			)
-			(justify left bottom)
-		)
-	)
-	(label "DSI_PWR_ON"
+		(at 311.15 207.01 0)
+		(effects
+			(font
+				(size 1.27 1.27)
+			)
+			(justify left bottom)
+		)
+	)
+	(label "DSI_PWR_EN"
 		(at 330.2 54.61 0)
 		(effects
@@
 		)
 	)
-	(hierarchical_label "DSI_PWR_ON"
+	(hierarchical_label "TP_SCL"
+		(shape output)
+		(at 325.12 224.79 0)
+		(effects
+			(font
+				(size 1.27 1.27)
+			)
+			(justify left)
+		)
+	)
+	(hierarchical_label "DSI_PWR_EN"
+		(shape output)
+		(at 382.27 238.76 0)
+		(effects
+			(font
+				(size 1.27 1.27)
+			)
+			(justify left)
+		)
+	)
+	(hierarchical_label "TP_INT"
 		(shape input)
-		(at 382.27 238.76 0)
-		(effects
-			(font
-				(size 1.27 1.27)
-			)
-			(justify left)
-		)
-	)
-	(hierarchical_label "DSI_TP_INT"
-		(shape output)
 		(at 382.27 234.95 0)
 		(effects
@@
 		)
 	)
-	(hierarchical_label "DSI"
+	(hierarchical_label "DSI_CK_P"
 		(shape bidirectional)
-		(at 330.2 194.31 0)
-		(effects
-			(font
-				(size 1.27 1.27)
-			)
-			(justify left)
-		)
-	)
-	(hierarchical_label "I2C5"
+		(at 325.12 210.82 0)
+		(effects
+			(font
+				(size 1.27 1.27)
+			)
+			(justify left)
+		)
+	)
+	(hierarchical_label "DSI_D0_N"
 		(shape bidirectional)
-		(at 330.2 219.71 0)
-		(effects
-			(font
-				(size 1.27 1.27)
-			)
-			(justify left)
-		)
-	)
-	(hierarchical_label "DSI_RESETn"
+		(at 325.12 200.66 0)
+		(effects
+			(font
+				(size 1.27 1.27)
+			)
+			(justify left)
+		)
+	)
+	(hierarchical_label "DSI_CK_N"
+		(shape bidirectional)
+		(at 325.12 213.36 0)
+		(effects
+			(font
+				(size 1.27 1.27)
+			)
+			(justify left)
+		)
+	)
+	(hierarchical_label "DSI_D1_P"
+		(shape bidirectional)
+		(at 325.12 204.47 0)
+		(effects
+			(font
+				(size 1.27 1.27)
+			)
+			(justify left)
+		)
+	)
+	(hierarchical_label "TP_SDA"
+		(shape bidirectional)
+		(at 325.12 222.25 0)
+		(effects
+			(font
+				(size 1.27 1.27)
+			)
+			(justify left)
+		)
+	)
+	(hierarchical_label "DSI_D1_N"
+		(shape bidirectional)
+		(at 325.12 207.01 0)
+		(effects
+			(font
+				(size 1.27 1.27)
+			)
+			(justify left)
+		)
+	)
+	(hierarchical_label "DSI_RESET"
 		(shape output)
 		(at 325.12 238.76 0)
@@
 		)
 	)
-	(hierarchical_label "DSI_TP_RESET"
+	(hierarchical_label "TP_RESET"
 		(shape output)
 		(at 382.27 231.14 0)
 		(effects
 			(font
+				(size 1.27 1.27)
+			)
+			(justify left)
+		)
+	)
+	(hierarchical_label "DSI_D0_P"
+		(shape bidirectional)
+		(at 325.12 198.12 0)
+		(effects
+			(font

Commit message: sch update
Connections:
- net I2C1.SCL renamed PWR_SCL
- net I2C1.SDA renamed PWR_SDA
- net I2C3.SCL renamed SENSOR_SCL
- net I2C3.SDA renamed SENSOR_SDA
Other:
- note added: "PWR"
- note added: "SENSOR"
Changed lines of the file:
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@@
 	(paper "A3")
+	(rectangle
+		(start 71.12 205.74)
+		(end 177.8 278.13)
+		(stroke
+			(width 0.1524)
+			(type solid)
+		)
+		(fill
+			(type none)
+		)
+	)
 	(rectangle
 		(start 299.72 176.53)
@@
 		)
 	)
+	(rectangle
+		(start 185.42 205.74)
+		(end 292.1 278.13)
+		(stroke
+			(width 0.1524)
+			(type solid)
+		)
+		(fill
+			(type none)
+		)
+	)
 	(text "PF11"
 		(exclude_from_sim no)
@@
 		)
 	)
-	(text "PE8"
-		(exclude_from_sim no)
-		(at 174.244 108.458 0)
-		(effects
-			(font
-				(size 1.27 1.27)
-			)
-		)
-	)
-	(text "PH8"
-		(exclude_from_sim no)
-		(at 250.698 99.822 0)
-		(effects
-			(font
-				(size 1.27 1.27)
-			)
-		)
-	)
-	(text "PE8"
-		(exclude_from_sim no)
-		(at 363.728 234.442 0)
-		(effects
-			(font
-				(size 1.27 1.27)
-			)
-		)
-	)
-	(text "PI6"
-		(exclude_from_sim no)
-		(at 346.456 56.388 0)
-		(effects
-			(font
-				(size 1.27 1.27)
-			)
-		)
-	)
-	(text "PH5"
-		(exclude_from_sim no)
-		(at 250.698 92.202 0)
-		(effects
-			(font
-				(size 1.27 1.27)
-			)
-		)
-	)
-	(text "PG14"
-		(exclude_from_sim no)
-		(at 250.698 76.962 0)
-		(effects
-			(font
-				(size 1.27 1.27)
-			)
-		)
-	)
-	(text "PD5"
-		(exclude_from_sim no)
-		(at 307.848 238.252 0)
-		(effects
-			(font
-				(size 1.27 1.27)
-			)
-		)
-	)
-	(text "DSI LCD"
-		(exclude_from_sim no)
-		(at 303.022 183.642 0)
+	(text "PWR"
+		(exclude_from_sim no)
+		(at 77.216 213.614 0)
 		(effects
 			(font
@@
 		)
 	)
+	(text "PE8"
+		(exclude_from_sim no)
+		(at 174.244 108.458 0)
+		(effects
+			(font
+				(size 1.27 1.27)
+			)
+		)
+	)
+	(text "PH8"
+		(exclude_from_sim no)
+		(at 250.698 99.822 0)
+		(effects
+			(font
+				(size 1.27 1.27)
+			)
+		)
+	)
+	(text "PE8"
+		(exclude_from_sim no)
+		(at 363.728 234.442 0)
+		(effects
+			(font
+				(size 1.27 1.27)
+			)
+		)
+	)
+	(text "PG13"
+		(exclude_from_sim no)
+		(at 80.264 225.298 0)
+		(effects
+			(font
+				(size 1.27 1.27)
+			)
+		)
+	)
+	(text "PI6"
+		(exclude_from_sim no)
+		(at 346.456 56.388 0)
+		(effects
+			(font
+				(size 1.27 1.27)
+			)
+		)
+	)
+	(text "SENSOR"
+		(exclude_from_sim no)
+		(at 191.516 213.614 0)
+		(effects
+			(font
+				(size 2.54 2.54)
+				(bold yes)
+			)
+			(justify left bottom)
+		)
+	)
+	(text "PH8"
+		(exclude_from_sim no)
+		(at 194.564 225.298 0)
+		(effects
+			(font
+				(size 1.27 1.27)
+			)
+		)
+	)
+	(text "PG14"
+		(exclude_from_sim no)
+		(at 80.264 228.092 0)
+		(effects
+			(font
+				(size 1.27 1.27)
+			)
+		)
+	)
+	(text "PH5"
+		(exclude_from_sim no)
+		(at 250.698 92.202 0)
+		(effects
+			(font
+				(size 1.27 1.27)
+			)
+		)
+	)
+	(text "PG14"
+		(exclude_from_sim no)
+		(at 250.698 76.962 0)
+		(effects
+			(font
+				(size 1.27 1.27)
+			)
+		)
+	)
+	(text "PD5"
+		(exclude_from_sim no)
+		(at 307.848 238.252 0)
+		(effects
+			(font
+				(size 1.27 1.27)
+			)
+		)
+	)
+	(text "DSI LCD"
+		(exclude_from_sim no)
+		(at 303.022 183.642 0)
+		(effects
+			(font
+				(size 2.54 2.54)
+				(bold yes)
+			)
+			(justify left bottom)
+		)
+	)
 	(text "PH7"
 		(exclude_from_sim no)
@@
 		(exclude_from_sim no)
 		(at 307.594 221.488 0)
+		(effects
+			(font
+				(size 1.27 1.27)
+			)
+		)
+	)
+	(text "PH7"
+		(exclude_from_sim no)
+		(at 194.564 228.092 0)
 		(effects
 			(font
@@
 	(wire
 		(pts
+			(xy 83.82 228.6) (xy 97.79 228.6)
+		)
+		(stroke
+			(width 0)
+			(type default)
+		)
+	)
+	(wire
+		(pts
 			(xy 237.49 125.73) (xy 271.78 125.73)
 		)
@@
 	(wire
 		(pts
+			(xy 198.12 228.6) (xy 212.09 228.6)
+		)
+		(stroke
+			(width 0)
+			(type default)
+		)
+	)
+	(wire
+		(pts
 			(xy 245.11 148.59) (xy 245.11 157.48)
 		)
@@
 	(wire
 		(pts
+			(xy 83.82 226.06) (xy 97.79 226.06)
+		)
+		(stroke
+			(width 0)
+			(type default)
+		)
+	)
+	(wire
+		(pts
 			(xy 250.19 140.97) (xy 271.78 140.97)
 		)
@@
 		(pts
 			(xy 237.49 115.57) (xy 237.49 118.11)
+		)
+		(stroke
+			(width 0)
+			(type default)
+		)
+	)
+	(wire
+		(pts
+			(xy 198.12 226.06) (xy 212.09 226.06)
 		)
 		(stroke
@@
 		)
 	)
+	(label "I2C1.SCL"
+		(at 83.82 228.6 0)
+		(effects
+			(font
+				(size 1.27 1.27)
+			)
+			(justify left bottom)
+		)
+	)
 	(label "DSI.TE"
 		(at 311.15 232.41 0)
@@
 		)
 	)
+	(label "I2C3.SCL"
+		(at 198.12 228.6 0)
+		(effects
+			(font
+				(size 1.27 1.27)
+			)
+			(justify left bottom)
+		)
+	)
+	(label "I2C3.SDA"
+		(at 198.12 226.06 0)
+		(effects
+			(font
+				(size 1.27 1.27)
+			)
+			(justify left bottom)
+		)
+	)
 	(label "DSI.D1_P"
 		(at 330.2 146.05 0)
@@
 	(label "DSI_TP_INT"
 		(at 367.03 234.95 0)
+		(effects
+			(font
+				(size 1.27 1.27)
+			)
+			(justify left bottom)
+		)
+	)
+	(label "I2C1.SDA"
+		(at 83.82 226.06 0)
 		(effects
 			(font
@@
 		)
 	)
+	(hierarchical_label "SENSOR_SCL"
+		(shape output)
+		(at 212.09 228.6 0)
+		(effects
+			(font
+				(size 1.27 1.27)
+			)
+			(justify left)
+		)
+	)
 	(hierarchical_label "DSI_CK_P"
 		(shape bidirectional)
@@
 		)
 	)
+	(hierarchical_label "PWR_SDA"
+		(shape bidirectional)
+		(at 97.79 226.06 0)
+		(effects
+			(font
+				(size 1.27 1.27)
+			)
+			(justify left)
+		)
+	)
+	(hierarchical_label "SENSOR_SDA"
+		(shape bidirectional)
+		(at 212.09 226.06 0)
+		(effects
+			(font
+				(size 1.27 1.27)
+			)
+			(justify left)
+		)
+	)
 	(hierarchical_label "DSI_D0_N"
 		(shape bidirectional)
@@
 		(effects
 			(font
+				(size 1.27 1.27)
+			)
+			(justify left)
+		)
+	)
+	(hierarchical_label "PWR_SCL"
+		(shape output)
+		(at 97.79 228.6 0)
+		(effects
+			(font

Commit message: sch update
Parts:
- added C48: 100nF, XWatch_Rev2.0:GEN_C_0201, symbol XWatch_Rev2.0:C
- added R8: 10K, XWatch_Rev2.0:GEN_R_0201, symbol XWatch_Rev2.0:R
Connections:
- net GND: now also C48.2, R8.2
- net at U1.B4 (PH3-BOOT0): now also R8.1
- net at U1.R2 (NRST): now also C48.1
Other:
- note added: "BOOT0 加一个测试点， NRST 引到 SWD 接口， C48 要尽量贴近 R2 球放"

Commit message: sch update
Changed lines of the file:
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@@
 	(paper "A3")
 	(rectangle
-		(start 71.12 205.74)
-		(end 177.8 278.13)
+		(start 124.46 205.74)
+		(end 200.66 278.13)
 		(stroke
 			(width 0.1524)
@@
 	)
 	(rectangle
-		(start 185.42 205.74)
+		(start 205.74 205.74)
 		(end 292.1 278.13)
 		(stroke
@@
 	(text "BOOT0 加一个测试点，\n\nNRST 引到 SWD 接口，\n\nC48 要尽量贴近 R2 球放"
 		(exclude_from_sim no)
-		(at 266.192 173.228 0)
+		(at 266.446 179.07 0)
 		(effects
 			(font
@@
 	(text "PWR"
 		(exclude_from_sim no)
-		(at 77.216 213.614 0)
+		(at 129.286 212.344 0)
 		(effects
 			(font
@@
 	(text "PG13"
 		(exclude_from_sim no)
-		(at 80.264 225.298 0)
+		(at 132.334 224.028 0)
 		(effects
 			(font
@@
 	(text "SENSOR"
 		(exclude_from_sim no)
-		(at 191.516 213.614 0)
+		(at 209.296 212.344 0)
 		(effects
 			(font
@@
 	(text "PH8"
 		(exclude_from_sim no)
-		(at 194.564 225.298 0)
+		(at 212.344 224.028 0)
 		(effects
 			(font
@@
 	(text "PG14"
 		(exclude_from_sim no)
-		(at 80.264 228.092 0)
+		(at 132.334 226.822 0)
 		(effects
 			(font
@@
 	(text "PH7"
 		(exclude_from_sim no)
-		(at 194.564 228.092 0)
+		(at 212.344 226.822 0)
 		(effects
 			(font
@@
 	(wire
 		(pts
-			(xy 83.82 228.6) (xy 97.79 228.6)
+			(xy 135.89 227.33) (xy 149.86 227.33)
 		)
 		(stroke
@@
 	(wire
 		(pts
-			(xy 198.12 228.6) (xy 212.09 228.6)
+			(xy 215.9 227.33) (xy 229.87 227.33)
 		)
 		(stroke
@@
 	(wire
 		(pts
-			(xy 83.82 226.06) (xy 97.79 226.06)
+			(xy 135.89 224.79) (xy 149.86 224.79)
 		)
 		(stroke
@@
 	(wire
 		(pts
-			(xy 198.12 226.06) (xy 212.09 226.06)
+			(xy 215.9 224.79) (xy 229.87 224.79)
 		)
 		(stroke
@@
 	)
 	(label "I2C1.SCL"
-		(at 83.82 228.6 0)
+		(at 135.89 227.33 0)
 		(effects
 			(font
@@
 	)
 	(label "I2C3.SCL"
-		(at 198.12 228.6 0)
+		(at 215.9 227.33 0)
 		(effects
 			(font
@@
 	)
 	(label "I2C3.SDA"
-		(at 198.12 226.06 0)
+		(at 215.9 224.79 0)
 		(effects
 			(font
@@
 	)
 	(label "I2C1.SDA"
-		(at 83.82 226.06 0)
+		(at 135.89 224.79 0)
 		(effects
 			(font
@@
 	(hierarchical_label "SENSOR_SCL"
 		(shape output)
-		(at 212.09 228.6 0)
+		(at 229.87 227.33 0)
 		(effects
 			(font
@@
 	(hierarchical_label "PWR_SDA"
 		(shape bidirectional)
-		(at 97.79 226.06 0)
+		(at 149.86 224.79 0)
 		(effects
 			(font
@@
 	(hierarchical_label "SENSOR_SDA"
 		(shape bidirectional)
-		(at 212.09 226.06 0)
+		(at 229.87 224.79 0)
 		(effects
 			(font
@@
 	(hierarchical_label "PWR_SCL"
 		(shape output)
-		(at 97.79 228.6 0)
-		(effects
-			(font
+		(at 149.86 227.33 0)
+		(effects
+			(font

Commit message: sch update
Connections:
- net SW3: now reaches U1.M4 (PA2-WKUP4)
- net SW5: now reaches U1.M5 (PA4-WKUP2)
- net SW2: now reaches U1.P3 (PA1-WKUP3)
- net SW4: now reaches U1.P4 (PA3-WKUP5)
Changed lines of the file:
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@@
+	(wire
+		(pts
+			(xy 99.06 45.72) (xy 100.33 45.72)
+		)
+		(stroke
+			(width 0)
+			(type default)
+		)
+	)
 	(wire
 		(pts
@@
 	(wire
 		(pts
+			(xy 99.06 53.34) (xy 100.33 53.34)
+		)
+		(stroke
+			(width 0)
+			(type default)
+		)
+	)
+	(wire
+		(pts
 			(xy 325.12 238.76) (xy 311.15 238.76)
 		)
@@
 	(wire
 		(pts
+			(xy 99.06 50.8) (xy 100.33 50.8)
+		)
+		(stroke
+			(width 0)
+			(type default)
+		)
+	)
+	(wire
+		(pts
 			(xy 245.11 166.37) (xy 250.19 166.37)
 		)
@@
 		(pts
 			(xy 229.87 153.67) (xy 229.87 157.48)
+		)
+		(stroke
+			(width 0)
+			(type default)
+		)
+	)
+	(wire
+		(pts
+			(xy 99.06 48.26) (xy 100.33 48.26)
 		)
 		(stroke
@@
 		)
 	)
+	(hierarchical_label "SW5"
+		(shape input)
+		(at 99.06 53.34 180)
+		(effects
+			(font
+				(size 1.27 1.27)
+			)
+			(justify right)
+		)
+	)
 	(hierarchical_label "PWR_SDA"
 		(shape bidirectional)
@@
 		)
 	)
+	(hierarchical_label "SW2"
+		(shape input)
+		(at 99.06 45.72 180)
+		(effects
+			(font
+				(size 1.27 1.27)
+			)
+			(justify right)
+		)
+	)
 	(hierarchical_label "DSI_CK_N"
 		(shape bidirectional)
@@
 		)
 	)
+	(hierarchical_label "SW4"
+		(shape input)
+		(at 99.06 50.8 180)
+		(effects
+			(font
+				(size 1.27 1.27)
+			)
+			(justify right)
+		)
+	)
 	(hierarchical_label "DSI_D1_P"
 		(shape bidirectional)
@@
 		)
 	)
+	(hierarchical_label "SW3"
+		(shape input)
+		(at 99.06 48.26 180)
+		(effects
+			(font
+				(size 1.27 1.27)
+			)
+			(justify right)
+		)
+	)

Commit message: sch update
Parts:
- added R18: 10K, XWatch_Rev2.0:GEN_R_0201, symbol XWatch_Rev2.0:R
Connections:
- net SW1: now reaches U1.N4 (PA0-WKUP1)
- net SW1: now also R18.2
- new net +1V8: R18.1
Changed lines of the file:
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@@
 	)
 	(junction
+		(at 96.52 43.18)
+		(diameter 0)
+		(color 0 0 0 0)
+	)
+	(junction
 		(at 247.65 118.11)
 		(diameter 0)
@@
 	(wire
 		(pts
+			(xy 96.52 43.18) (xy 100.33 43.18)
+		)
+		(stroke
+			(width 0)
+			(type default)
+		)
+	)
+	(wire
+		(pts
+			(xy 96.52 41.91) (xy 96.52 43.18)
+		)
+		(stroke
+			(width 0)
+			(type default)
+		)
+	)
+	(wire
+		(pts
 			(xy 99.06 53.34) (xy 100.33 53.34)
 		)
@@
 	(wire
 		(pts
+			(xy 93.98 43.18) (xy 96.52 43.18)
+		)
+		(stroke
+			(width 0)
+			(type default)
+		)
+	)
+	(wire
+		(pts
 			(xy 311.15 213.36) (xy 325.12 213.36)
 		)
@@
 		)
 	)
+	(wire
+		(pts
+			(xy 96.52 34.29) (xy 96.52 33.02)
+		)
+		(stroke
+			(width 0)
+			(type default)
+		)
+	)
 	(label "DSI.RESET"
 		(at 158.75 55.88 0)
@@
 		)
 	)
+	(hierarchical_label "SW1"
+		(shape input)
+		(at 93.98 43.18 180)
+		(effects
+			(font
+				(size 1.27 1.27)
+			)
+			(justify right)
+		)
+	)
 	(hierarchical_label "SW5"
 		(shape input)
@@
 	)
 	(symbol
+		(lib_id "XWatch_Rev2.0:R")
+		(at 96.52 38.1 0)
+		(unit 1)
+		(body_style 1)
+		(exclude_from_sim no)
+		(in_bom yes)
+		(on_board yes)
+		(in_pos_files yes)
+		(dnp no)
+		(property "Reference" "R18"
+			(at 98.044 37.592 0)
+			(show_name no)
+			(do_not_autoplace no)
+			(effects
+				(font
+					(size 1.27 1.27)
+				)
+				(justify left)
+			)
+		)
+		(property "Value" "10K"
+			(at 98.044 40.132 0)
+			(show_name no)
+			(do_not_autoplace no)
+			(effects
+				(font
+					(size 1.27 1.27)
+				)
+				(justify left)
+			)
+		)
+		(property "Footprint" "XWatch_Rev2.0:GEN_R_0201"
+			(at 94.742 38.1 90)
+			(hide yes)
+			(show_name no)
+			(do_not_autoplace no)
+			(effects
+				(font
+					(size 1.27 1.27)
+				)
+			)
+		)
+		(property "Datasheet" ""
+			(at 96.52 38.1 0)
+			(hide yes)
+			(show_name no)
+			(do_not_autoplace no)
+			(effects
+				(font
+					(size 1.27 1.27)
+				)
+			)
+		)
+		(property "Description" "Resistor"
+			(at 96.52 38.1 0)
+			(hide yes)
+			(show_name no)
+			(do_not_autoplace no)
+			(effects
+				(font
+					(size 1.27 1.27)
+				)
+			)
+		)
+		(pin "1"
+		)
+		(pin "2"
+		)
+		(instances
+			(project "XWatch_Rev2.0"
+				(path "/64425c00-526a-4829-b8a6-ed1dc1b19578/999006d4-9c3b-4798-99ee-23f029574470"
+					(reference "R18")
+					(unit 1)
+				)
+			)
+		)
+	)
+	(symbol
 		(lib_id "XWatch_Rev2.0:C")
 		(at 237.49 111.76 0)
@@
 					(unit 1)
 				)
+			)
+		)
+	)
+	(symbol
+		(lib_id "power:+1V8")
+		(at 96.52 33.02 0)
+		(unit 1)
+		(body_style 1)
+		(exclude_from_sim no)
+		(in_bom yes)
+		(on_board yes)
+		(in_pos_files yes)
+		(dnp no)
+		(property "Reference" "#PWR0192"
+			(at 96.52 36.83 0)
+			(hide yes)
+			(show_name no)
+			(do_not_autoplace no)
+			(effects
+				(font
+					(size 1.27 1.27)
+				)
+			)
+		)
+		(property "Value" "+1V8"
+			(at 96.012 29.21 0)
+			(show_name no)
+			(do_not_autoplace no)
+			(effects
+				(font
+					(size 1.27 1.27)
+				)
+			)
+		)
+		(property "Footprint" ""
+			(at 96.52 33.02 0)
+			(hide yes)
+			(show_name no)
+			(do_not_autoplace no)
+			(effects
+				(font
+					(size 1.27 1.27)
+				)
+			)
+		)
+		(property "Datasheet" ""
+			(at 96.52 33.02 0)
+			(hide yes)
+			(show_name no)
+			(do_not_autoplace no)
+			(effects
+				(font
+					(size 1.27 1.27)
+				)
+			)
+		)
+		(property "Description" "Power symbol creates a global label with name \"+1V8\""
+			(at 96.52 33.02 0)
+			(hide yes)
+			(show_name no)
+			(do_not_autoplace no)
+			(effects
+				(font
+					(size 1.27 1.27)
+				)
+			)
+		)
+		(pin "1"
+		)
+		(instances
+			(project "XWatch_Rev2.0"
+				(path "/64425c00-526a-4829-b8a6-ed1dc1b19578/999006d4-9c3b-4798-99ee-23f029574470"
+					(reference "#PWR0192")
+					(unit 1)
+				)

Commit message: sch update
Parts:
- added D1: RB520S-30, XWatch_Rev2.0:RB520S-30_C7502701, symbol XWatch_Rev2.0:RB520S-30
Connections:
- net SW1: now also D1.1 (K); no longer R18.2, U1.N4 (PA0-WKUP1)
- new net: D1.2 (A), R18.2, U1.N4 (PA0-WKUP1)
Other:
- note added: "BUTTONS"
