File: hardware/schematic/v1.0/XWatch_Rev2.0/MCU_IO.kicad_sch (KiCad schematic)
At the start: 11 parts, among them U1 STM32U5G9NJH6Q, X1 32.768KHZ, X2 16MHZ

Commit message: sch update
Connections:
- net OSPI_IO1: now reaches U1.M9 (PE13)
- net OSPI_IO3: now reaches U1.N10 (PE15)
- net OSPI_IO0: now reaches U1.N11 (PE12)
- net OSPI_CLK: now reaches U1.P10 (PE10)
- net OSPI_NCS: now reaches U1.P11 (PE11)
- net OSPI_IO2: now reaches U1.R10 (PE14)
Other:
- note added: "MEMORY"

Commit message: sch update
Other:
- note added: "PA0"
- note added: "PA1"
- note added: "PA2"
- note added: "PA3"
- note added: "PA4"
- note added: "PE10"
- note added: "PE11"
- note added: "PE12"
- note added: "PE13"
- note added: "PE14"
- note added: "PE15"
Changed lines of the file:
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@@
+		)
+	)
+	(text "PE10"
+		(exclude_from_sim no)
+		(at 174.752 113.538 0)
+		(effects
+			(font
+				(size 1.27 1.27)
+			)
+		)
+	)
+	(text "PE15"
+		(exclude_from_sim no)
+		(at 56.896 276.352 0)
+		(effects
+			(font
+				(size 1.27 1.27)
+			)
+		)
+	)
+	(text "PE13"
+		(exclude_from_sim no)
+		(at 56.896 268.732 0)
+		(effects
+			(font
+				(size 1.27 1.27)
+			)
 		)
 	)
@@
 		)
 	)
+	(text "PE13"
+		(exclude_from_sim no)
+		(at 174.752 121.666 0)
+		(effects
+			(font
+				(size 1.27 1.27)
+			)
+		)
+	)
 	(text "PI6"
 		(exclude_from_sim no)
@@
 		(exclude_from_sim no)
 		(at 250.698 89.408 0)
+		(effects
+			(font
+				(size 1.27 1.27)
+			)
+		)
+	)
+	(text "PA0"
+		(exclude_from_sim no)
+		(at 57.15 223.012 0)
+		(effects
+			(font
+				(size 1.27 1.27)
+			)
+		)
+	)
+	(text "PE12"
+		(exclude_from_sim no)
+		(at 56.896 265.176 0)
 		(effects
 			(font
@@
 		)
 	)
+	(text "PA3"
+		(exclude_from_sim no)
+		(at 57.15 234.442 0)
+		(effects
+			(font
+				(size 1.27 1.27)
+			)
+		)
+	)
 	(text "PWR"
 		(exclude_from_sim no)
@@
 		)
 	)
+	(text "PE10"
+		(exclude_from_sim no)
+		(at 56.896 257.556 0)
+		(effects
+			(font
+				(size 1.27 1.27)
+			)
+		)
+	)
 	(text "PH8"
 		(exclude_from_sim no)
@@
 		(exclude_from_sim no)
 		(at 132.334 224.028 0)
+		(effects
+			(font
+				(size 1.27 1.27)
+			)
+		)
+	)
+	(text "PE14"
+		(exclude_from_sim no)
+		(at 174.752 124.206 0)
 		(effects
 			(font
@@
 		)
 	)
+	(text "PE11"
+		(exclude_from_sim no)
+		(at 174.752 116.332 0)
+		(effects
+			(font
+				(size 1.27 1.27)
+			)
+		)
+	)
 	(text "PH8"
 		(exclude_from_sim no)
@@
 		)
 	)
+	(text "PE11"
+		(exclude_from_sim no)
+		(at 56.896 261.112 0)
+		(effects
+			(font
+				(size 1.27 1.27)
+			)
+		)
+	)
+	(text "PE15"
+		(exclude_from_sim no)
+		(at 174.752 126.746 0)
+		(effects
+			(font
+				(size 1.27 1.27)
+			)
+		)
+	)
+	(text "PA4"
+		(exclude_from_sim no)
+		(at 57.15 238.252 0)
+		(effects
+			(font
+				(size 1.27 1.27)
+			)
+		)
+	)
 	(text "PG14"
 		(exclude_from_sim no)
 		(at 250.698 76.962 0)
+		(effects
+			(font
+				(size 1.27 1.27)
+			)
+		)
+	)
+	(text "PA2"
+		(exclude_from_sim no)
+		(at 57.15 230.632 0)
+		(effects
+			(font
+				(size 1.27 1.27)
+			)
+		)
+	)
+	(text "PA1"
+		(exclude_from_sim no)
+		(at 57.15 226.822 0)
 		(effects
 			(font
@@
 		)
 	)
+	(text "PE14"
+		(exclude_from_sim no)
+		(at 56.896 272.288 0)
+		(effects
+			(font
+				(size 1.27 1.27)
+			)
+		)
+	)
 	(text "PH4"
 		(exclude_from_sim no)
@@
 		(effects
 			(font
+				(size 1.27 1.27)
+			)
+		)
+	)
+	(text "PE12"
+		(exclude_from_sim no)
+		(at 174.752 118.872 0)
+		(effects
+			(font
