File: hardware/schematic/v1.0/XWatch_Rev2.0/XWatch_Rev2.0.kicad_sch (KiCad schematic)
At the start: 0 parts

Commit message: sch update
Other:
- sheet MCU_IO ports: added OSPI_CLK, OSPI_IO0, OSPI_IO1, OSPI_IO2, OSPI_IO3, OSPI_NCS; removed none
Changed lines of the file:
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@@
 	(paper "A4")
 	(sheet
-		(at 114.3 101.6)
+		(at 102.87 19.05)
 		(size 16.51 35.56)
 		(exclude_from_sim no)
@@
 		)
 		(property "Sheetname" "DSI_LCD"
-			(at 114.3 100.8884 0)
+			(at 102.87 18.3384 0)
 			(show_name no)
 			(do_not_autoplace no)
@@
 		)
 		(property "Sheetfile" "DSI_LCD.kicad_sch"
-			(at 114.3 137.7446 0)
+			(at 102.87 55.1946 0)
 			(show_name no)
 			(do_not_autoplace no)
@@
 		)
 		(pin "DSI_D0_N" bidirectional
-			(at 114.3 109.22 180)
+			(at 102.87 26.67 180)
 			(effects
 				(font
@@
 		)
 		(pin "DSI_CK_N" bidirectional
-			(at 114.3 114.3 180)
+			(at 102.87 31.75 180)
 			(effects
 				(font
@@
 		)
 		(pin "DSI_CK_P" bidirectional
-			(at 114.3 111.76 180)
+			(at 102.87 29.21 180)
 			(effects
 				(font
@@
 		)
 		(pin "DSI_RESET" input
-			(at 114.3 119.38 180)
+			(at 102.87 36.83 180)
 			(effects
 				(font
@@
 		)
 		(pin "DSI_TE" input
-			(at 114.3 121.92 180)
+			(at 102.87 39.37 180)
 			(effects
 				(font
@@
 		)
 		(pin "TP_SDA" bidirectional
-			(at 114.3 124.46 180)
+			(at 102.87 41.91 180)
 			(effects
 				(font
@@
 		)
 		(pin "TP_INT" output
-			(at 114.3 129.54 180)
+			(at 102.87 46.99 180)
 			(effects
 				(font
@@
 		)
 		(pin "DSI_PWR_EN" input
-			(at 114.3 116.84 180)
+			(at 102.87 34.29 180)
 			(effects
 				(font
@@
 		)
 		(pin "DSI_D0_P" bidirectional
-			(at 114.3 106.68 180)
+			(at 102.87 24.13 180)
 			(effects
 				(font
@@
 		)
 		(pin "TP_RESET" input
-			(at 114.3 132.08 180)
+			(at 102.87 49.53 180)
 			(effects
 				(font
@@
 		)
 		(pin "TP_SCL" input
-			(at 114.3 127 180)
+			(at 102.87 44.45 180)
 			(effects
 				(font
@@
 	)
 	(sheet
-		(at 182.88 58.42)
+		(at 93.98 80.01)
 		(size 12.7 22.86)
 		(exclude_from_sim no)
@@
 		)
 		(property "Sheetname" "MEMORY"
-			(at 182.88 57.7084 0)
+			(at 93.98 79.2984 0)
 			(show_name no)
 			(do_not_autoplace no)
@@
 		)
 		(property "Sheetfile" "MEMORY.kicad_sch"
-			(at 182.88 81.8646 0)
+			(at 93.98 103.4546 0)
 			(show_name no)
 			(do_not_autoplace no)
@@
 		)
 		(pin "OSPI_IO1" input
-			(at 182.88 66.04 180)
+			(at 93.98 87.63 180)
 			(effects
 				(font
@@
 		)
 		(pin "OSPI_IO2" input
-			(at 182.88 68.58 180)
+			(at 93.98 90.17 180)
 			(effects
 				(font
@@
 		)
 		(pin "OSPI_IO0" input
-			(at 182.88 63.5 180)
+			(at 93.98 85.09 180)
 			(effects
 				(font
@@
 		)
 		(pin "OSPI_IO3" input
-			(at 182.88 71.12 180)
+			(at 93.98 92.71 180)
 			(effects
 				(font
@@
 		)
 		(pin "OSPI_NCS" input
-			(at 182.88 73.66 180)
+			(at 93.98 95.25 180)
 			(effects
 				(font
@@
 		)
 		(pin "OSPI_CLK" input
-			(at 182.88 76.2 180)
+			(at 93.98 97.79 180)
 			(effects
 				(font
@@
 	)
 	(sheet
-		(at 101.6 158.75)
+		(at 95.25 113.03)
 		(size 20.32 20.32)
 		(exclude_from_sim no)
@@
 		)
 		(property "Sheetname" "BLE"
-			(at 101.6 158.0384 0)
+			(at 95.25 112.3184 0)
 			(show_name no)
 			(do_not_autoplace no)
@@
 		)
 		(property "Sheetfile" "BLE.kicad_sch"
-			(at 101.6 179.6546 0)
+			(at 95.25 133.9346 0)
 			(show_name no)
 			(do_not_autoplace no)
@@
 	(sheet
 		(at 57.15 76.2)
-		(size 26.67 35.56)
+		(size 26.67 58.42)
 		(exclude_from_sim no)
 		(in_bom yes)
@@
 		)
 		(property "Sheetfile" "MCU_IO.kicad_sch"
-			(at 57.15 112.3446 0)
+			(at 57.15 135.2046 0)
 			(show_name no)
 			(do_not_autoplace no)
@@
 		(pin "SW5" input
 			(at 66.04 76.2 90)
+			(effects
+				(font
+					(size 1.27 1.27)
+				)
+				(justify right)
+			)
+		)
+		(pin "OSPI_IO1" output
+			(at 83.82 87.63 0)
+			(effects
+				(font
+					(size 1.27 1.27)
+				)
+				(justify right)
+			)
+		)
+		(pin "OSPI_IO3" output
+			(at 83.82 92.71 0)
+			(effects
+				(font
+					(size 1.27 1.27)
+				)
+				(justify right)
+			)
+		)
+		(pin "OSPI_IO0" output
+			(at 83.82 85.09 0)
+			(effects
+				(font
+					(size 1.27 1.27)
+				)
+				(justify right)
+			)
+		)
+		(pin "OSPI_IO2" output
+			(at 83.82 90.17 0)
+			(effects
+				(font
+					(size 1.27 1.27)
+				)
+				(justify right)
+			)
+		)
+		(pin "OSPI_CLK" output
+			(at 83.82 97.79 0)
+			(effects
+				(font
+					(size 1.27 1.27)
+				)
+				(justify right)
+			)
+		)
+		(pin "OSPI_NCS" output
+			(at 83.82 95.25 0)
 			(effects
 				(font
@@
 	)
 	(sheet
-		(at 57.15 119.38)
+		(at 125.73 142.24)
 		(size 26.67 27.94)
 		(exclude_from_sim no)
@@
 		)
 		(property "Sheetname" "PWR"
-			(at 57.15 118.6684 0)
+			(at 125.73 141.5284 0)
 			(show_name no)
 			(do_not_autoplace no)
@@
 		)
 		(property "Sheetfile" "PWR.kicad_sch"
-			(at 57.15 147.9046 0)
-			(show_name no)
-			(do_not_autoplace no)
+			(at 125.73 170.7646 0)
+			(show_name no)
+			(do_not_autoplace no)

Commit message: sch update
Other:
- sheet PWR ports: added EN_3V3, FG_ALRT_N, PWR_CHG_EN_N, PWR_INT_N, PWR_RIN_N, PWR_SCL, PWR_SDA; removed none
Changed lines of the file:
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@@
 	(sheet
 		(at 125.73 142.24)
-		(size 26.67 27.94)
+		(size 26.67 22.86)
 		(exclude_from_sim no)
 		(in_bom yes)
@@
 		)
 		(property "Sheetfile" "PWR.kicad_sch"
-			(at 125.73 170.7646 0)
+			(at 125.73 165.6846 0)
 			(show_name no)
 			(do_not_autoplace no)
@@
 			)
 		)
+		(pin "FG_ALRT_N" output
+			(at 152.4 153.67 0)
+			(effects
+				(font
+					(size 1.27 1.27)
+				)
+				(justify right)
+			)
+		)
+		(pin "PWR_SCL" input
+			(at 152.4 146.05 0)
+			(effects
+				(font
+					(size 1.27 1.27)
+				)
+				(justify right)
+			)
+		)
+		(pin "PWR_RIN_N" output
+			(at 152.4 156.21 0)
+			(effects
+				(font
+					(size 1.27 1.27)
+				)
+				(justify right)
+			)
+		)
+		(pin "PWR_CHG_EN_N" input
+			(at 152.4 158.75 0)
+			(effects
+				(font
+					(size 1.27 1.27)
+				)
+				(justify right)
+			)
+		)
+		(pin "EN_3V3" input
+			(at 152.4 161.29 0)
+			(effects
+				(font
+					(size 1.27 1.27)
+				)
+				(justify right)
+			)
+		)
+		(pin "PWR_SDA" bidirectional
+			(at 152.4 148.59 0)
+			(effects
+				(font
+					(size 1.27 1.27)
+				)
+				(justify right)
+			)
+		)
+		(pin "PWR_INT_N" output
+			(at 152.4 151.13 0)
+			(effects
+				(font
+					(size 1.27 1.27)
+				)
+				(justify right)
+			)
+		)
