File: hardware/schematic/v1.0/XWatch_Rev2.0/XWatch_Rev2.0.kicad_sch (KiCad schematic)
At the start: 0 parts

Commit message: sch update
Other:
- sheet SENSOR ports: added ALS_INT_N, BARO_INT, DRV_REG, HAPTIC_EN, IMU_INT1, IMU_INT2, LRA_N, LRA_P, MAG_C1, MAG_DRDY, PPG_INT_N, SENSOR_SCL, SENSOR_SDA; removed none
Changed lines of the file:
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@@
 	)
 	(sheet
-		(at 135.89 60.96)
-		(size 22.86 26.67)
+		(at 135.89 63.5)
+		(size 22.86 50.8)
 		(exclude_from_sim no)
 		(in_bom yes)
@@
 		)
 		(property "Sheetname" "SENSOR"
-			(at 135.89 60.2484 0)
+			(at 135.89 62.7884 0)
 			(show_name no)
 			(do_not_autoplace no)
@@
 		)
 		(property "Sheetfile" "SENSOR.kicad_sch"
-			(at 135.89 88.2146 0)
+			(at 135.89 114.8846 0)
 			(show_name no)
 			(do_not_autoplace no)
@@
 			)
 		)
+		(pin "ALS_INT_N" output
+			(at 135.89 68.58 180)
+			(effects
+				(font
+					(size 1.27 1.27)
+				)
+				(justify left)
+			)
+		)
+		(pin "IMU_INT2" output
+			(at 135.89 71.12 180)
+			(effects
+				(font
+					(size 1.27 1.27)
+				)
+				(justify left)
+			)
+		)
+		(pin "SENSOR_SCL" input
+			(at 135.89 73.66 180)
+			(effects
+				(font
+					(size 1.27 1.27)
+				)
+				(justify left)
+			)
+		)
+		(pin "MAG_DRDY" output
+			(at 135.89 76.2 180)
+			(effects
+				(font
+					(size 1.27 1.27)
+				)
+				(justify left)
+			)
+		)
+		(pin "MAG_C1" output
+			(at 135.89 78.74 180)
+			(effects
+				(font
+					(size 1.27 1.27)
+				)
+				(justify left)
+			)
+		)
+		(pin "BARO_INT" output
+			(at 135.89 81.28 180)
+			(effects
+				(font
+					(size 1.27 1.27)
+				)
+				(justify left)
+			)
+		)
+		(pin "LRA_N" output
+			(at 135.89 83.82 180)
+			(effects
+				(font
+					(size 1.27 1.27)
+				)
+				(justify left)
+			)
+		)
+		(pin "IMU_INT1" output
+			(at 135.89 86.36 180)
+			(effects
+				(font
+					(size 1.27 1.27)
+				)
+				(justify left)
+			)
+		)
+		(pin "HAPTIC_EN" input
+			(at 135.89 88.9 180)
+			(effects
+				(font
+					(size 1.27 1.27)
+				)
+				(justify left)
+			)
+		)
+		(pin "LRA_P" output
+			(at 135.89 91.44 180)
+			(effects
+				(font
+					(size 1.27 1.27)
+				)
+				(justify left)
+			)
+		)
+		(pin "DRV_REG" input
+			(at 135.89 93.98 180)
+			(effects
+				(font
+					(size 1.27 1.27)
+				)
+				(justify left)
+			)
+		)
+		(pin "PPG_INT_N" output
+			(at 135.89 96.52 180)
+			(effects
+				(font
+					(size 1.27 1.27)
+				)
+				(justify left)
+			)
+		)
+		(pin "SENSOR_SDA" bidirectional
+			(at 135.89 99.06 180)
+			(effects
+				(font
+					(size 1.27 1.27)
+				)
+				(justify left)
+			)
+		)

Commit message: sch update
Other:
- sheet MCU_IO ports: added DSI_CK_N, DSI_CK_P, DSI_D0_N, DSI_D0_P, DSI_PWR_EN, DSI_RESET, DSI_TE, TP_INT, TP_RESET, TP_SCL, TP_SDA; removed none

Commit message: sch update
Other:
- sheet SENSOR ports: added none; removed DRV_REG, MAG_C1
Changed lines of the file:
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@@
 			)
 		)
-		(pin "MAG_C1" output
+		(pin "BARO_INT" output
 			(at 154.94 107.95 180)
 			(effects
@@
 			)
 		)
-		(pin "BARO_INT" output
+		(pin "LRA_N" output
 			(at 154.94 110.49 180)
 			(effects
@@
 			)
 		)
-		(pin "LRA_N" output
+		(pin "IMU_INT1" output
 			(at 154.94 113.03 180)
 			(effects
@@
 			)
 		)
-		(pin "IMU_INT1" output
+		(pin "HAPTIC_EN" input
 			(at 154.94 115.57 180)
 			(effects
@@
 			)
 		)
-		(pin "HAPTIC_EN" input
+		(pin "LRA_P" output
 			(at 154.94 118.11 180)
 			(effects
@@
 			)
 		)
-		(pin "LRA_P" output
+		(pin "PPG_INT_N" output
 			(at 154.94 120.65 180)
 			(effects
@@
 			)
 		)
-		(pin "DRV_REG" input
+		(pin "SENSOR_SDA" bidirectional
 			(at 154.94 123.19 180)
 			(effects
 				(font
-					(size 1.27 1.27)
-				)
-				(justify left)
-			)
-		)
-		(pin "PPG_INT_N" output
-			(at 154.94 125.73 180)
-			(effects
-				(font
-					(size 1.27 1.27)
-				)
-				(justify left)
-			)
-		)
-		(pin "SENSOR_SDA" bidirectional
-			(at 154.94 128.27 180)
-			(effects
-				(font
