File: hardware/schematic/v1.0/XWatch_Rev2.0/MEMORY.kicad_sch (KiCad schematic)
At the start: 1 part, among them U2 GD25LQ128EWIGR

Commit message: sch update
Parts:
- added C67: 100nF, XWatch_Rev2.0:GEN_C_0201, symbol XWatch_Rev2.0:C
- added C68: 1uF, XWatch_Rev2.0:GEN_C_0402, symbol XWatch_Rev2.0:C
- added R23, R24, R25: 10K, XWatch_Rev2.0:GEN_R_0201, symbol XWatch_Rev2.0:R
Connections:
- net OSPI_NCS: now reaches U2.1 (CS#)
- net OSPI_NCS: now also R24.2
- net OSPI_IO1: now reaches U2.2 (SO(IO1))
- net OSPI_IO2: now reaches U2.3 (WP#(IO2))
- net OSPI_IO2: now also R23.2
- net GND: now reaches U2.4 (VSS)
- net GND: now also U2.9 (EP), C67.1, C68.1
- net OSPI_IO0: now reaches U2.5 (SI(IO0))
- net OSPI_CLK: now reaches U2.6 (SCLK)
- net OSPI_IO3: now reaches U2.7 (HOLD#(IO3))
- net OSPI_IO3: now also R25.1
- net +1V8: now reaches U2.8 (VCC)
- net +1V8: now also C67.2, C68.2, R23.1, R24.1, R25.2

Commit message: sch update
Other:
- note added: "128Mbit = 16MB"
Changed lines of the file:
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@@
 	(generator_version "10.0")
 	(paper "A4")
+	(text "128Mbit = 16MB"
+		(exclude_from_sim no)
+		(at 132.334 114.3 0)
+		(effects
+			(font
+				(size 1.27 1.27)
+			)
+		)
+	)
 	(junction
 		(at 99.06 86.36)
