File: hardware/schematic/v1.0/XWatch_Rev2.0/XWatch_Rev2.0.kicad_pcb (KiCad board)
At the start: 2 copper layers, 62.6 x 58 mm, 115 parts, among them SW1 EVPAEDB2A, SW2 EVPAEDB2A, SW3 EVPAEDB2A, SW4 EVPAEDB2A, SW5 EVPAEDB2A, U1 STM32U5G9NJH6Q, U10 OPT3001DNPR, U11 MAX30101EFD_T, U12 DRV2605LDGSR, U13 SK6018D4-33, U14 AXE530127-DO0143FMST02, U3 DA9168, U4 TPS62840DLCR, U5 MAX17048G_T10, U6 LSM6DSOXTR, U7 LIS2MDLTR, U8 SM03B-SRSS-TB_LF_SN_P, U9 LPS27HHWTR, X1 32.768KHZ, X2 16MHZ

Commit message: sch update
Parts:
- added D1: RB520S-30, XWatch_Rev2.0:RB520S-30_C7502701, F.Cu at (105.8, 119.3)
- added U2: GD25LQ128EWIGR, XWatch_Rev2.0:GD25LQ128EWIGR, F.Cu at (114.6, 127.2)
- moved SW4 37.1 mm to (133.7, 118.8), turned to 0 degrees
- moved SW5 34.7 mm to (133.7, 123.3), turned to 0 degrees
- moved SW1 33.6 mm to (133.7, 105.4), turned to 0 degrees
- moved C38 27.7 mm to (122.6, 84.0)
- moved C39 27.7 mm to (122.6, 86.0)
- moved C40 27.7 mm to (122.6, 87.9)
- moved C43 27.7 mm to (122.6, 89.8)
- moved C44 27.7 mm to (122.6, 91.7)
- moved C45 27.7 mm to (122.6, 93.7)
- moved C47 27.7 mm to (122.6, 95.6)
- moved C73 27.7 mm to (130.4, 84.1)
- moved C74 27.7 mm to (130.4, 86.3)
- moved C75 27.7 mm to (130.4, 88.4)
- moved C76 27.7 mm to (130.4, 90.5)
- moved C77 27.7 mm to (130.4, 92.6)
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Connections:
- net /MCU_IO/SW1 renamed Net-(D1-A)
Other:
- board size 62.6 x 58 mm -> 5.6 x 1.4 mm

Commit message: sch update
Parts:
- removed SW1, SW2, SW3, SW4, SW5: EVPAEDB2A, XWatch_Rev2.0:EVPAEDB2A
- added C67: 100nF, XWatch_Rev2.0:GEN_C_0201, F.Cu at (154.8, 88.0)
- added C68: 1uF, XWatch_Rev2.0:GEN_C_0402, F.Cu at (155.0, 85.9)
- added IC1: nRF52833-QDAA-R, XWatch_Rev2.0:QFN40P500X500X90-41N, F.Cu at (154.3, 117.4)
- added R23: 10K, XWatch_Rev2.0:GEN_R_0201, F.Cu at (152.3, 85.8)
- added R24: 10K, XWatch_Rev2.0:GEN_R_0201, F.Cu at (152.3, 87.6)
- added R25: 10K, XWatch_Rev2.0:GEN_R_0201, F.Cu at (152.3, 89.4)
- U11, U14, U8: moved to B.Cu
- moved U4 83.3 mm to (171.5, 130.2)
- moved U5 73.0 mm to (175.6, 125.6)
- moved U1 67.5 mm to (166.9, 117.1)
- moved U2 63.5 mm to (177.4, 117.1)
- moved U9 62.1 mm to (175.7, 109.1)
- moved U3 57.0 mm to (154.1, 124.0)
- moved U8 51.9 mm to (154.1, 109.1), turned to 180 degrees
- moved X1 49.8 mm to (144.3, 98.2)
- moved X2 49.8 mm to (139.7, 98.6)
- moved U11 49.0 mm to (165.7, 130.4), turned to 180 degrees
- moved U12 38.2 mm to (159.1, 129.8)
- moved U14 34.6 mm to (165.2, 105.5), turned to 180 degrees
- moved L1 4.16 mm to (109.2, 94.7)
- moved L2 3.80 mm to (109.2, 98.6)
Connections:
- C75 pad 1: unconnected-(C75-Pad1) -> GND
- C76 pad 1: unconnected-(C76-Pad1) -> GND
- U1 pad M9: unconnected-(U1A-PE13-PadM9) -> /MCU_IO/OSPI.IO1
- U1 pad N10: unconnected-(U1A-PE15-PadN10) -> /MCU_IO/OSPI.IO3
- U1 pad N11: unconnected-(U1A-PE12-PadN11) -> /MCU_IO/OSPI.IO0
- U1 pad P10: unconnected-(U1A-PE10-PadP10) -> /MCU_IO/OSPI.CLK
- U1 pad P11: unconnected-(U1A-PE11-PadP11) -> /MCU_IO/OSPI.NCS
- U1 pad R10: unconnected-(U1A-PE14-PadR10) -> /MCU_IO/OSPI.IO2
- U2 pad 1: unconnected-(U2-CS#-Pad1) -> /MEMORY/OSPI_NCS
- U2 pad 2: unconnected-(U2-SO(IO1)-Pad2) -> /MEMORY/OSPI_IO1
- U2 pad 3: unconnected-(U2-WP#(IO2)-Pad3) -> /MEMORY/OSPI_IO2
- U2 pad 4: unconnected-(U2-VSS-Pad4) -> GND
- U2 pad 5: unconnected-(U2-SI(IO0)-Pad5) -> /MEMORY/OSPI_IO0
- U2 pad 6: unconnected-(U2-SCLK-Pad6) -> /MEMORY/OSPI_CLK
- U2 pad 7: unconnected-(U2-HOLD#(IO3)-Pad7) -> /MEMORY/OSPI_IO3
- U2 pad 8: unconnected-(U2-VCC-Pad8) -> +1V8
- U2 pad 9: unconnected-(U2-EP-Pad9) -> GND
Other:
- board size 5.6 x 1.4 mm -> 36 x 36 mm
