File: hardware/schematic/v1.0/XWatch_Rev2.0/BLE.kicad_sch (KiCad schematic)
At the start: 1 part, among them IC1 nRF52833-QDAA-R

Commit message: sch update
Parts:
- added C69, C70: 100nF, XWatch_Rev2.0:GEN_C_0201, symbol XWatch_Rev2.0:C
Connections:
- net at IC1.1 (DEC1): now also C69.2
- net GND: now reaches IC1.10 (VBUS)
- net GND: now also IC1.25 (VSS_PA), IC1.37 (VSS_1), C69.1, C70.2
- net at IC1.21 (DEC5): now also C70.1
- no-connect marks 0 -> 11
