File: hardware/schematic/v1.0/XWatch_Rev3.0/MEMORY.kicad_sch (KiCad schematic)
At the start: 6 parts, among them U2 GD25LQ128EWIGR

Commit message: sch update
Connections:
- net OSPI_CLK renamed OSPI.CLK
- net OSPI_IO0 renamed OSPI.IO0
- net OSPI_IO1 renamed OSPI.IO1
- net OSPI_IO2 renamed OSPI.IO2
- net OSPI_IO3 renamed OSPI.IO3
- net OSPI_NCS renamed OSPI.NCS
Changed lines of the file:
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@@
 		)
 	)
-	(hierarchical_label "OSPI_CLK"
+	(hierarchical_label "OSPI.CLK"
 		(shape input)
 		(at 182.88 104.14 0)
@@
 		)
 	)
-	(hierarchical_label "OSPI_IO3"
+	(hierarchical_label "OSPI.IO3"
 		(shape input)
 		(at 182.88 101.6 0)
@@
 		)
 	)
-	(hierarchical_label "OSPI_IO0"
+	(hierarchical_label "OSPI.IO0"
 		(shape input)
 		(at 182.88 106.68 0)
@@
 		)
 	)
-	(hierarchical_label "OSPI_IO1"
+	(hierarchical_label "OSPI.IO1"
 		(shape input)
 		(at 92.71 101.6 180)
@@
 		)
 	)
-	(hierarchical_label "OSPI_IO2"
+	(hierarchical_label "OSPI.IO2"
 		(shape input)
 		(at 92.71 104.14 180)
@@
 		)
 	)
-	(hierarchical_label "OSPI_NCS"
+	(hierarchical_label "OSPI.NCS"
 		(shape input)
 		(at 92.71 99.06 180)
