File: hardware/schematic/v1.0/XWatch_Rev3.0/XWatch_Rev3.0.kicad_sch (KiCad schematic)
At the start: 0 parts

Commit message: sch update
Other:
- sheet MCU_IO ports: added ALS_INT_N, BARO_INT, DSI_D1_N, DSI_D1_P, FG_ALRT_N, HAPTIC_EN, IMU_INT1, IMU_INT2, MAG_DRDY, PPG_INT_N, PWR_INT_N, PWR_SCL, PWR_SDA, SENSOR_SCL, SENSOR_SDA; removed none
- sheet SENSOR ports: added none; removed DRV_REG, MAG_C1
Changed lines of the file:
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@@
 	(sheet
 		(at 154.94 92.71)
-		(size 22.86 50.8)
+		(size 22.86 45.72)
 		(exclude_from_sim no)
 		(in_bom yes)
@@
 		)
 		(property "Sheetfile" "SENSOR.kicad_sch"
-			(at 154.94 144.0946 0)
+			(at 154.94 139.0146 0)
 			(show_name no)
 			(do_not_autoplace no)
@@
 		)
 		(pin "ALS_INT_N" output
+			(at 154.94 104.14 180)
+			(effects
+				(font
+					(size 1.27 1.27)
+				)
+				(justify left)
+			)
+		)
+		(pin "IMU_INT2" output
+			(at 154.94 109.22 180)
+			(effects
+				(font
+					(size 1.27 1.27)
+				)
+				(justify left)
+			)
+		)
+		(pin "SENSOR_SCL" input
 			(at 154.94 97.79 180)
 			(effects
@@
 			)
 		)
-		(pin "IMU_INT2" output
+		(pin "MAG_DRDY" output
+			(at 154.94 111.76 180)
+			(effects
+				(font
+					(size 1.27 1.27)
+				)
+				(justify left)
+			)
+		)
+		(pin "BARO_INT" output
+			(at 154.94 114.3 180)
+			(effects
+				(font
+					(size 1.27 1.27)
+				)
+				(justify left)
+			)
+		)
+		(pin "LRA_N" output
+			(at 154.94 127 180)
+			(effects
+				(font
+					(size 1.27 1.27)
+				)
+				(justify left)
+			)
+		)
+		(pin "IMU_INT1" output
+			(at 154.94 106.68 180)
+			(effects
+				(font
+					(size 1.27 1.27)
+				)
+				(justify left)
+			)
+		)
+		(pin "HAPTIC_EN" input
+			(at 154.94 119.38 180)
+			(effects
+				(font
+					(size 1.27 1.27)
+				)
+				(justify left)
+			)
+		)
+		(pin "LRA_P" output
+			(at 154.94 124.46 180)
+			(effects
+				(font
+					(size 1.27 1.27)
+				)
+				(justify left)
+			)
+		)
+		(pin "PPG_INT_N" output
+			(at 154.94 116.84 180)
+			(effects
+				(font
+					(size 1.27 1.27)
+				)
+				(justify left)
+			)
+		)
+		(pin "SENSOR_SDA" bidirectional
 			(at 154.94 100.33 180)
-			(effects
-				(font
-					(size 1.27 1.27)
-				)
-				(justify left)
-			)
-		)
-		(pin "SENSOR_SCL" input
-			(at 154.94 102.87 180)
-			(effects
-				(font
-					(size 1.27 1.27)
-				)
-				(justify left)
-			)
-		)
-		(pin "MAG_DRDY" output
-			(at 154.94 105.41 180)
-			(effects
-				(font
-					(size 1.27 1.27)
-				)
-				(justify left)
-			)
-		)
-		(pin "MAG_C1" output
-			(at 154.94 107.95 180)
-			(effects
-				(font
-					(size 1.27 1.27)
-				)
-				(justify left)
-			)
-		)
-		(pin "BARO_INT" output
-			(at 154.94 110.49 180)
-			(effects
-				(font
-					(size 1.27 1.27)
-				)
-				(justify left)
-			)
-		)
-		(pin "LRA_N" output
-			(at 154.94 113.03 180)
-			(effects
-				(font
-					(size 1.27 1.27)
-				)
-				(justify left)
-			)
-		)
-		(pin "IMU_INT1" output
-			(at 154.94 115.57 180)
-			(effects
-				(font
-					(size 1.27 1.27)
-				)
-				(justify left)
-			)
-		)
-		(pin "HAPTIC_EN" input
-			(at 154.94 118.11 180)
-			(effects
-				(font
-					(size 1.27 1.27)
-				)
-				(justify left)
-			)
-		)
-		(pin "LRA_P" output
-			(at 154.94 120.65 180)
-			(effects
-				(font
-					(size 1.27 1.27)
-				)
-				(justify left)
-			)
-		)
-		(pin "DRV_REG" input
-			(at 154.94 123.19 180)
-			(effects
-				(font
-					(size 1.27 1.27)
-				)
-				(justify left)
-			)
-		)
-		(pin "PPG_INT_N" output
-			(at 154.94 125.73 180)
-			(effects
-				(font
-					(size 1.27 1.27)
-				)
-				(justify left)
-			)
-		)
-		(pin "SENSOR_SDA" bidirectional
-			(at 154.94 128.27 180)
 			(effects
 				(font
@@
 			(effects
 				(font
+					(size 1.27 1.27)
+				)
+				(justify left)
+			)
+		)
+		(pin "ALS_INT_N" input
+			(at 148.59 104.14 0)
+			(effects
+				(font
+					(size 1.27 1.27)
+				)
+				(justify right)
+			)
+		)
+		(pin "DSI_D1_P" bidirectional
+			(at 115.57 99.06 180)
+			(effects
+				(font
+					(size 1.27 1.27)
+				)
+				(justify left)
+			)
+		)
+		(pin "PWR_SCL" output
+			(at 115.57 109.22 180)
+			(effects
+				(font
+					(size 1.27 1.27)
+				)
+				(justify left)
+			)
+		)
+		(pin "FG_ALRT_N" input
+			(at 115.57 116.84 180)
+			(effects
+				(font
+					(size 1.27 1.27)
+				)
+				(justify left)
+			)
+		)
+		(pin "IMU_INT1" input
+			(at 148.59 106.68 0)
+			(effects
+				(font
+					(size 1.27 1.27)
+				)
+				(justify right)
+			)
+		)
+		(pin "DSI_D1_N" bidirectional
+			(at 115.57 101.6 180)
+			(effects
+				(font
+					(size 1.27 1.27)
+				)
+				(justify left)
+			)
+		)
+		(pin "MAG_DRDY" input
+			(at 148.59 111.76 0)
+			(effects
+				(font
+					(size 1.27 1.27)
+				)
+				(justify right)
+			)
+		)
+		(pin "HAPTIC_EN" output
+			(at 148.59 119.38 0)
+			(effects
+				(font
+					(size 1.27 1.27)
+				)
+				(justify right)
+			)
+		)
+		(pin "PWR_INT_N" input
+			(at 115.57 114.3 180)
+			(effects
+				(font
+					(size 1.27 1.27)
+				)
+				(justify left)
+			)
+		)
+		(pin "SENSOR_SDA" bidirectional
+			(at 148.59 100.33 0)
+			(effects
+				(font
+					(size 1.27 1.27)
+				)
+				(justify right)
+			)
+		)
+		(pin "SENSOR_SCL" output
+			(at 148.59 97.79 0)
+			(effects
+				(font
+					(size 1.27 1.27)
+				)
+				(justify right)
+			)
+		)
+		(pin "BARO_INT" input
+			(at 148.59 114.3 0)
+			(effects
+				(font
+					(size 1.27 1.27)
+				)
+				(justify right)
+			)
+		)
+		(pin "IMU_INT2" input
+			(at 148.59 109.22 0)
+			(effects
+				(font
+					(size 1.27 1.27)
+				)
+				(justify right)
+			)
+		)
+		(pin "PPG_INT_N" input
+			(at 148.59 116.84 0)
+			(effects
+				(font
+					(size 1.27 1.27)
+				)
+				(justify right)
+			)
+		)
+		(pin "PWR_SDA" bidirectional
+			(at 115.57 111.76 180)
+			(effects
+				(font

Commit message: sch update
Changed lines of the file:
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@@
 			)
 		)
-		(pin "FG_ALRT_N" input
+		(pin "FG_ALRT_N" bidirectional
 			(at 115.57 116.84 180)
 			(effects
@@
 			)
 		)
-		(pin "PWR_INT_N" input
+		(pin "PWR_INT_N" bidirectional
 			(at 115.57 114.3 180)
 			(effects

Commit message: sch update
Other:
- sheet BLE ports: added BLE.MCU_CTS, BLE.MCU_RTS, BLE.MCU_RX, BLE.MCU_TX, BLE.WAKE_MCU, BLE.WAKE_NRF; removed none
Changed lines of the file:
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@@
 	(sheet
 		(at 207.01 101.6)
-		(size 20.32 20.32)
+		(size 20.32 30.48)
 		(exclude_from_sim no)
 		(in_bom yes)
@@
 		)
 		(property "Sheetfile" "BLE.kicad_sch"
-			(at 207.01 122.5046 0)
+			(at 207.01 132.6646 0)
 			(show_name no)
 			(do_not_autoplace no)
@@
 			)
 		)
+		(pin "BLE.WAKE_MCU" input
+			(at 207.01 110.49 180)
+			(effects
+				(font
+					(size 1.27 1.27)
+				)
+				(justify left)
+			)
+		)
+		(pin "BLE.WAKE_NRF" input
+			(at 207.01 113.03 180)
+			(effects
+				(font
+					(size 1.27 1.27)
+				)
+				(justify left)
+			)
+		)
+		(pin "BLE.MCU_RTS" input
+			(at 207.01 115.57 180)
+			(effects
+				(font
+					(size 1.27 1.27)
+				)
+				(justify left)
+			)
+		)
+		(pin "BLE.MCU_CTS" output
+			(at 207.01 118.11 180)
+			(effects
+				(font
+					(size 1.27 1.27)
+				)
+				(justify left)
+			)
+		)
+		(pin "BLE.MCU_TX" input
+			(at 207.01 120.65 180)
+			(effects
+				(font
+					(size 1.27 1.27)
+				)
+				(justify left)
+			)
+		)
+		(pin "BLE.MCU_RX" output
+			(at 207.01 123.19 180)
+			(effects
+				(font
+					(size 1.27 1.27)
+				)
+				(justify left)
+			)
+		)

Commit message: sch update
Other:
- sheet MEMORY ports: added OSPI.CLK, OSPI.IO0, OSPI.IO1, OSPI.IO2, OSPI.IO3, OSPI.NCS; removed OSPI_CLK, OSPI_IO0, OSPI_IO1, OSPI_IO2, OSPI_IO3, OSPI_NCS
Changed lines of the file:
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@@
 	)
 	(sheet
-		(at 154.94 63.5)
-		(size 13.97 21.59)
+		(at 154.94 64.77)
+		(size 13.97 20.32)
 		(exclude_from_sim no)
 		(in_bom yes)
@@
 		)
 		(property "Sheetname" "MEMORY"
-			(at 154.94 62.7884 0)
+			(at 154.94 64.0584 0)
 			(show_name no)
 			(do_not_autoplace no)
@@
 			)
 		)
-		(pin "OSPI_IO1" input
+		(pin "OSPI.IO0" input
+			(at 154.94 68.58 180)
+			(effects
+				(font
+					(size 1.27 1.27)
+				)
+				(justify left)
+			)
+		)
+		(pin "OSPI.IO2" input
+			(at 154.94 73.66 180)
+			(effects
+				(font
+					(size 1.27 1.27)
+				)
+				(justify left)
+			)
+		)
+		(pin "OSPI.IO1" input
 			(at 154.94 71.12 180)
 			(effects
@@
 			)
 		)
-		(pin "OSPI_IO2" input
-			(at 154.94 73.66 180)
+		(pin "OSPI.CLK" input
+			(at 154.94 81.28 180)
 			(effects
 				(font
@@
 			)
 		)
-		(pin "OSPI_IO0" input
-			(at 154.94 68.58 180)
-			(effects
-				(font
-					(size 1.27 1.27)
-				)
-				(justify left)
-			)
-		)
-		(pin "OSPI_IO3" input
+		(pin "OSPI.IO3" input
 			(at 154.94 76.2 180)
 			(effects
@@
 			)
 		)
-		(pin "OSPI_NCS" input
+		(pin "OSPI.NCS" input
 			(at 154.94 78.74 180)
 			(effects
 				(font
-					(size 1.27 1.27)
-				)
-				(justify left)
-			)
-		)
-		(pin "OSPI_CLK" input
-			(at 154.94 81.28 180)
-			(effects
-				(font

Commit message: sch update
Other:
- sheet MCU_IO ports: added OSPI.CLK, OSPI.IO0, OSPI.IO1, OSPI.IO2, OSPI.IO3, OSPI.NCS; removed OSPI_CLK, OSPI_IO0, OSPI_IO1, OSPI_IO2, OSPI_IO3, OSPI_NCS
Changed lines of the file:
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@@
 	(sheet
 		(at 154.94 92.71)
-		(size 22.86 45.72)
+		(size 22.86 31.75)
 		(exclude_from_sim no)
 		(in_bom yes)
@@
 		)
 		(property "Sheetfile" "SENSOR.kicad_sch"
-			(at 154.94 139.0146 0)
+			(at 154.94 125.0446 0)
 			(show_name no)
 			(do_not_autoplace no)
@@
 		)
 		(pin "LRA_N" output
-			(at 154.94 127 180)
-			(effects
-				(font
-					(size 1.27 1.27)
-				)
-				(justify left)
+			(at 177.8 107.95 0)
+			(effects
+				(font
+					(size 1.27 1.27)
+				)
+				(justify right)
 			)
 		)
@@
 		)
 		(pin "LRA_P" output
-			(at 154.94 124.46 180)
-			(effects
-				(font
-					(size 1.27 1.27)
-				)
-				(justify left)
+			(at 177.8 105.41 0)
+			(effects
+				(font
+					(size 1.27 1.27)
+				)
+				(justify right)
 			)
 		)
@@
 			)
 		)
-		(pin "OSPI_IO1" output
-			(at 148.59 71.12 0)
-			(effects
-				(font
-					(size 1.27 1.27)
-				)
-				(justify right)
-			)
-		)
-		(pin "OSPI_IO3" output
-			(at 148.59 76.2 0)
-			(effects
-				(font
-					(size 1.27 1.27)
-				)
-				(justify right)
-			)
-		)
-		(pin "OSPI_IO0" output
-			(at 148.59 68.58 0)
-			(effects
-				(font
-					(size 1.27 1.27)
-				)
-				(justify right)
-			)
-		)
-		(pin "OSPI_IO2" output
-			(at 148.59 73.66 0)
-			(effects
-				(font
-					(size 1.27 1.27)
-				)
-				(justify right)
-			)
-		)
-		(pin "OSPI_CLK" output
-			(at 148.59 81.28 0)
-			(effects
-				(font
-					(size 1.27 1.27)
-				)
-				(justify right)
-			)
-		)
-		(pin "OSPI_NCS" output
-			(at 148.59 78.74 0)
-			(effects
-				(font
-					(size 1.27 1.27)
-				)
-				(justify right)
-			)
-		)
 		(pin "DSI_CK_N" bidirectional
 			(at 115.57 76.2 180)
@@
 			)
 		)
+		(pin "OSPI.NCS" output
+			(at 148.59 78.74 0)
+			(effects
+				(font
+					(size 1.27 1.27)
+				)
+				(justify right)
+			)
+		)
+		(pin "OSPI.IO2" output
+			(at 148.59 73.66 0)
+			(effects
+				(font
+					(size 1.27 1.27)
+				)
+				(justify right)
+			)
+		)
+		(pin "OSPI.IO1" output
+			(at 148.59 71.12 0)
+			(effects
+				(font
+					(size 1.27 1.27)
+				)
+				(justify right)
+			)
+		)
+		(pin "OSPI.IO3" output
+			(at 148.59 76.2 0)
+			(effects
+				(font
+					(size 1.27 1.27)
+				)
+				(justify right)
+			)
+		)
+		(pin "OSPI.IO0" output
+			(at 148.59 68.58 0)
+			(effects
+				(font
+					(size 1.27 1.27)
+				)
+				(justify right)
+			)
+		)
+		(pin "OSPI.CLK" output
+			(at 148.59 81.28 0)
+			(effects
+				(font
+					(size 1.27 1.27)
+				)
+				(justify right)
+			)
+		)

Commit message: sch update
Other:
- sheet DSI_LCD ports: added DSI.CK_N, DSI.CK_P, DSI.D0_N, DSI.D0_P, DSI.PWR_EN, DSI.RESET, DSI.TE, TP.INT, TP.RESET, TP.SCL, TP.SDA; removed DSI_CK_N, DSI_CK_P, DSI_D0_N, DSI_D0_P, DSI_PWR_EN, DSI_RESET, DSI_TE, TP_INT, TP_RESET, TP_SCL, TP_SDA
- sheet MCU_IO ports: added DSI.CK_N, DSI.CK_P, DSI.D0_N, DSI.D0_P, DSI.D1_N, DSI.D1_P, DSI.PWR_EN, DSI.RESET, DSI.TE, TP.INT, TP.RESET, TP.SCL, TP.SDA; removed DSI_CK_N, DSI_CK_P, DSI_D0_N, DSI_D0_P, DSI_D1_N, DSI_D1_P, DSI_PWR_EN, DSI_RESET, DSI_TE, TP_INT, TP_RESET, TP_SCL, TP_SDA
Changed lines of the file:
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@@
 			)
 		)
-		(pin "DSI_D0_N" bidirectional
+		(pin "TP.SCL" input
+			(at 106.68 88.9 0)
+			(effects
+				(font
+					(size 1.27 1.27)
+				)
+				(justify right)
+			)
+		)
+		(pin "DSI.CK_N" bidirectional
+			(at 106.68 76.2 0)
+			(effects
+				(font
+					(size 1.27 1.27)
+				)
+				(justify right)
+			)
+		)
+		(pin "DSI.TE" input
+			(at 106.68 83.82 0)
+			(effects
+				(font
+					(size 1.27 1.27)
+				)
+				(justify right)
+			)
+		)
+		(pin "DSI.CK_P" bidirectional
+			(at 106.68 73.66 0)
+			(effects
+				(font
+					(size 1.27 1.27)
+				)
+				(justify right)
+			)
+		)
+		(pin "TP.SDA" bidirectional
+			(at 106.68 86.36 0)
+			(effects
+				(font
+					(size 1.27 1.27)
+				)
+				(justify right)
+			)
+		)
+		(pin "DSI.RESET" input
+			(at 106.68 81.28 0)
+			(effects
+				(font
+					(size 1.27 1.27)
+				)
+				(justify right)
+			)
+		)
+		(pin "TP.RESET" input
+			(at 106.68 93.98 0)
+			(effects
+				(font
+					(size 1.27 1.27)
+				)
+				(justify right)
+			)
+		)
+		(pin "DSI.D0_N" bidirectional
 			(at 106.68 71.12 0)
 			(effects
@@
 			)
 		)
-		(pin "DSI_CK_N" bidirectional
-			(at 106.68 76.2 0)
-			(effects
-				(font
-					(size 1.27 1.27)
-				)
-				(justify right)
-			)
-		)
-		(pin "DSI_CK_P" bidirectional
-			(at 106.68 73.66 0)
-			(effects
-				(font
-					(size 1.27 1.27)
-				)
-				(justify right)
-			)
-		)
-		(pin "DSI_RESET" input
-			(at 106.68 81.28 0)
-			(effects
-				(font
-					(size 1.27 1.27)
-				)
-				(justify right)
-			)
-		)
-		(pin "DSI_TE" input
-			(at 106.68 83.82 0)
-			(effects
-				(font
-					(size 1.27 1.27)
-				)
-				(justify right)
-			)
-		)
-		(pin "TP_SDA" bidirectional
-			(at 106.68 86.36 0)
-			(effects
-				(font
-					(size 1.27 1.27)
-				)
-				(justify right)
-			)
-		)
-		(pin "TP_INT" output
+		(pin "DSI.PWR_EN" input
+			(at 106.68 78.74 0)
+			(effects
+				(font
+					(size 1.27 1.27)
+				)
+				(justify right)
+			)
+		)
+		(pin "DSI.D0_P" bidirectional
+			(at 106.68 68.58 0)
+			(effects
+				(font
+					(size 1.27 1.27)
+				)
+				(justify right)
+			)
+		)
+		(pin "TP.INT" output
 			(at 106.68 91.44 0)
-			(effects
-				(font
-					(size 1.27 1.27)
-				)
-				(justify right)
-			)
-		)
-		(pin "DSI_PWR_EN" input
-			(at 106.68 78.74 0)
-			(effects
-				(font
-					(size 1.27 1.27)
-				)
-				(justify right)
-			)
-		)
-		(pin "DSI_D0_P" bidirectional
-			(at 106.68 68.58 0)
-			(effects
-				(font
-					(size 1.27 1.27)
-				)
-				(justify right)
-			)
-		)
-		(pin "TP_RESET" input
-			(at 106.68 93.98 0)
-			(effects
-				(font
-					(size 1.27 1.27)
-				)
-				(justify right)
-			)
-		)
-		(pin "TP_SCL" input
-			(at 106.68 88.9 0)
 			(effects
 				(font
@@
 			)
 		)
-		(pin "DSI_CK_N" bidirectional
-			(at 115.57 76.2 180)
-			(effects
-				(font
-					(size 1.27 1.27)
-				)
-				(justify left)
-			)
-		)
-		(pin "DSI_D0_N" bidirectional
-			(at 115.57 71.12 180)
-			(effects
-				(font
-					(size 1.27 1.27)
-				)
-				(justify left)
-			)
-		)
-		(pin "DSI_CK_P" bidirectional
-			(at 115.57 73.66 180)
-			(effects
-				(font
-					(size 1.27 1.27)
-				)
-				(justify left)
-			)
-		)
-		(pin "TP_SDA" bidirectional
-			(at 115.57 86.36 180)
-			(effects
-				(font
-					(size 1.27 1.27)
-				)
-				(justify left)
-			)
-		)
-		(pin "TP_RESET" output
-			(at 115.57 93.98 180)
-			(effects
-				(font
-					(size 1.27 1.27)
-				)
-				(justify left)
-			)
-		)
-		(pin "DSI_RESET" output
-			(at 115.57 81.28 180)
-			(effects
-				(font
-					(size 1.27 1.27)
-				)
-				(justify left)
-			)
-		)
-		(pin "DSI_D0_P" bidirectional
-			(at 115.57 68.58 180)
-			(effects
-				(font
-					(size 1.27 1.27)
-				)
-				(justify left)
-			)
-		)
-		(pin "DSI_TE" input
-			(at 115.57 83.82 180)
-			(effects
-				(font
-					(size 1.27 1.27)
-				)
-				(justify left)
-			)
-		)
-		(pin "DSI_PWR_EN" output
-			(at 115.57 78.74 180)
-			(effects
-				(font
-					(size 1.27 1.27)
-				)
-				(justify left)
-			)
-		)
-		(pin "TP_INT" input
-			(at 115.57 91.44 180)
-			(effects
-				(font
-					(size 1.27 1.27)
-				)
-				(justify left)
-			)
-		)
-		(pin "TP_SCL" output
-			(at 115.57 88.9 180)
-			(effects
-				(font
-					(size 1.27 1.27)
-				)
-				(justify left)
-			)
-		)
 		(pin "ALS_INT_N" input
 			(at 148.59 104.14 0)
@@
 			)
 		)
-		(pin "DSI_D1_P" bidirectional
-			(at 115.57 99.06 180)
-			(effects
-				(font
-					(size 1.27 1.27)
-				)
-				(justify left)
-			)
-		)
 		(pin "PWR_SCL" output
 			(at 115.57 109.22 180)
@@
 			)
 		)
-		(pin "DSI_D1_N" bidirectional
-			(at 115.57 101.6 180)
-			(effects
-				(font
-					(size 1.27 1.27)
-				)
-				(justify left)
-			)
-		)
 		(pin "MAG_DRDY" input
 			(at 148.59 111.76 0)
@@
 			)
 		)
+		(pin "DSI.PWR_EN" output
+			(at 115.57 78.74 180)
+			(effects
+				(font
+					(size 1.27 1.27)
+				)
+				(justify left)
+			)
+		)
+		(pin "DSI.CK_P" bidirectional
+			(at 115.57 73.66 180)
+			(effects
+				(font
+					(size 1.27 1.27)
+				)
+				(justify left)
+			)
+		)
+		(pin "DSI.D0_N" bidirectional
+			(at 115.57 71.12 180)
+			(effects
+				(font
+					(size 1.27 1.27)
+				)
+				(justify left)
+			)
+		)
+		(pin "TP.INT" input
+			(at 115.57 91.44 180)
+			(effects
+				(font
+					(size 1.27 1.27)
+				)
+				(justify left)
+			)
+		)
+		(pin "TP.SCL" output
+			(at 115.57 88.9 180)
+			(effects
+				(font
+					(size 1.27 1.27)
+				)
+				(justify left)
+			)
+		)
+		(pin "DSI.CK_N" bidirectional
+			(at 115.57 76.2 180)
+			(effects
+				(font
+					(size 1.27 1.27)
+				)
+				(justify left)
+			)
+		)
+		(pin "TP.RESET" output
+			(at 115.57 93.98 180)
+			(effects
+				(font
+					(size 1.27 1.27)
+				)
+				(justify left)
+			)
+		)
+		(pin "DSI.RESET" output
+			(at 115.57 81.28 180)
+			(effects
+				(font
+					(size 1.27 1.27)
+				)
+				(justify left)
+			)
+		)
+		(pin "DSI.D0_P" bidirectional
+			(at 115.57 68.58 180)
+			(effects
+				(font
+					(size 1.27 1.27)
+				)
+				(justify left)
+			)
+		)
+		(pin "DSI.D1_P" bidirectional
+			(at 115.57 100.33 180)
+			(effects
+				(font
+					(size 1.27 1.27)
+				)
+				(justify left)
+			)
+		)
+		(pin "TP.SDA" bidirectional
+			(at 115.57 86.36 180)
+			(effects
+				(font
+					(size 1.27 1.27)
+				)
+				(justify left)
+			)
+		)
+		(pin "DSI.D1_N" bidirectional
+			(at 115.57 102.87 180)
+			(effects
+				(font
+					(size 1.27 1.27)
+				)
+				(justify left)
+			)
+		)
+		(pin "DSI.TE" input
+			(at 115.57 83.82 180)
+			(effects
+				(font
+					(size 1.27 1.27)
+				)
+				(justify left)
+			)
+		)

Commit message: sch update
Other:
- sheet MCU_IO ports: added BLE.MCU_CTS, BLE.MCU_RTS, BLE.MCU_RX, BLE.MCU_TX, BLE.WAKE_MCU, BLE.WAKE_NRF, USB_DM, USB_DP; removed none
- sheet PWR ports: added USB_DM, USB_DP; removed none
Changed lines of the file:
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@@
 	)
 	(sheet
-		(at 207.01 62.23)
+		(at 208.28 46.99)
 		(size 25.4 31.75)
 		(exclude_from_sim no)
@@
 		)
 		(property "Sheetname" "MCU_PWR"
-			(at 207.01 61.5184 0)
+			(at 208.28 46.2784 0)
 			(show_name no)
 			(do_not_autoplace no)
@@
 		)
 		(property "Sheetfile" "MCU_PWR.kicad_sch"
-			(at 207.01 94.5646 0)
+			(at 208.28 79.3246 0)
 			(show_name no)
 			(do_not_autoplace no)
@@
 	)
 	(sheet
-		(at 207.01 101.6)
+		(at 154.94 132.08)
 		(size 20.32 30.48)
 		(exclude_from_sim no)
@@
 		)
 		(property "Sheetname" "BLE"
-			(at 207.01 100.8884 0)
+			(at 154.94 131.3684 0)
 			(show_name no)
 			(do_not_autoplace no)
@@
 		)
 		(property "Sheetfile" "BLE.kicad_sch"
-			(at 207.01 132.6646 0)
+			(at 154.94 163.1446 0)
 			(show_name no)
 			(do_not_autoplace no)
@@
 		)
 		(pin "BLE.WAKE_MCU" input
-			(at 207.01 110.49 180)
+			(at 154.94 140.97 180)
 			(effects
 				(font
@@
 		)
 		(pin "BLE.WAKE_NRF" input
-			(at 207.01 113.03 180)
+			(at 154.94 143.51 180)
 			(effects
 				(font
@@
 		)
 		(pin "BLE.MCU_RTS" input
-			(at 207.01 115.57 180)
+			(at 154.94 146.05 180)
 			(effects
 				(font
@@
 		)
 		(pin "BLE.MCU_CTS" output
-			(at 207.01 118.11 180)
+			(at 154.94 148.59 180)
 			(effects
 				(font
@@
 		)
 		(pin "BLE.MCU_TX" input
-			(at 207.01 120.65 180)
+			(at 154.94 151.13 180)
 			(effects
 				(font
@@
 		)
 		(pin "BLE.MCU_RX" output
-			(at 207.01 123.19 180)
+			(at 154.94 153.67 180)
 			(effects
 				(font
@@
 	(sheet
 		(at 115.57 59.69)
-		(size 33.02 78.74)
+		(size 33.02 110.49)
 		(exclude_from_sim no)
 		(in_bom yes)
@@
 		)
 		(property "Sheetfile" "MCU_IO.kicad_sch"
-			(at 115.57 139.0146 0)
+			(at 115.57 170.7646 0)
 			(show_name no)
 			(do_not_autoplace no)
@@
 				)
 				(justify left)
+			)
+		)
+		(pin "BLE.WAKE_NRF" output
+			(at 148.59 143.51 0)
+			(effects
+				(font
+					(size 1.27 1.27)
+				)
+				(justify right)
+			)
+		)
+		(pin "USB_DP" bidirectional
+			(at 115.57 130.81 180)
+			(effects
+				(font
+					(size 1.27 1.27)
+				)
+				(justify left)
+			)
+		)
+		(pin "USB_DM" bidirectional
+			(at 115.57 133.35 180)
+			(effects
+				(font
+					(size 1.27 1.27)
+				)
+				(justify left)
+			)
+		)
+		(pin "BLE.MCU_RX" input
+			(at 148.59 153.67 0)
+			(effects
+				(font
+					(size 1.27 1.27)
+				)
+				(justify right)
+			)
+		)
+		(pin "BLE.MCU_CTS" input
+			(at 148.59 148.59 0)
+			(effects
+				(font
+					(size 1.27 1.27)
+				)
+				(justify right)
+			)
+		)
+		(pin "BLE.MCU_TX" output
+			(at 148.59 151.13 0)
+			(effects
+				(font
+					(size 1.27 1.27)
+				)
+				(justify right)
+			)
+		)
+		(pin "BLE.WAKE_MCU" output
+			(at 148.59 140.97 0)
+			(effects
+				(font
+					(size 1.27 1.27)
+				)
+				(justify right)
+			)
+		)
+		(pin "BLE.MCU_RTS" output
+			(at 148.59 146.05 0)
+			(effects
+				(font
+					(size 1.27 1.27)
+				)
+				(justify right)
 			)
 		)
@@
 	(sheet
 		(at 83.82 105.41)
-		(size 22.86 22.86)
+		(size 22.86 36.83)
 		(exclude_from_sim no)
 		(in_bom yes)
@@
 		)
 		(property "Sheetfile" "PWR.kicad_sch"
-			(at 83.82 128.8546 0)
+			(at 83.82 142.8246 0)
 			(show_name no)
 			(do_not_autoplace no)
@@
 			(effects
 				(font
+					(size 1.27 1.27)
+				)
+				(justify right)
+			)
+		)
+		(pin "USB_DP" bidirectional
+			(at 106.68 130.81 0)
+			(effects
+				(font
+					(size 1.27 1.27)
+				)
+				(justify right)
+			)
+		)
+		(pin "USB_DM" bidirectional
+			(at 106.68 133.35 0)
+			(effects
+				(font

Commit message: sch update
Changed lines of the file:
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@@
 	(generator_version "10.0")
 	(paper "A4")
+	(wire
+		(pts
+			(xy 148.59 153.67) (xy 154.94 153.67)
+		)
+		(stroke
+			(width 0)
+			(type default)
+		)
+	)
+	(wire
+		(pts
+			(xy 148.59 146.05) (xy 154.94 146.05)
+		)
+		(stroke
+			(width 0)
+			(type default)
+		)
+	)
+	(wire
+		(pts
+			(xy 148.59 148.59) (xy 154.94 148.59)
+		)
+		(stroke
+			(width 0)
+			(type default)
+		)
+	)
+	(wire
+		(pts
+			(xy 148.59 140.97) (xy 154.94 140.97)
+		)
+		(stroke
+			(width 0)
+			(type default)
+		)
+	)
+	(wire
+		(pts
+			(xy 148.59 143.51) (xy 154.94 143.51)
+		)
+		(stroke
+			(width 0)
+			(type default)
+		)
+	)
+	(wire
+		(pts
+			(xy 148.59 151.13) (xy 154.94 151.13)
+		)
+		(stroke
+			(width 0)
+			(type default)
+		)
+	)
 	(sheet
 		(at 90.17 63.5)
