File: hardware/schematic/v1.0/XWatch_Rev3.0/XWatch_Rev3.0.kicad_sch (KiCad schematic)
At the start: 0 parts

Commit message: sch update
Changed lines of the file:
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@@
+	(wire
+		(pts
+			(xy 148.59 73.66) (xy 154.94 73.66)
+		)
+		(stroke
+			(width 0)
+			(type default)
+		)
+	)
 	(wire
 		(pts
 			(xy 148.59 153.67) (xy 154.94 153.67)
+		)
+		(stroke
+			(width 0)
+			(type default)
+		)
+	)
+	(wire
+		(pts
+			(xy 132.08 50.8) (xy 132.08 59.69)
+		)
+		(stroke
+			(width 0)
+			(type default)
+		)
+	)
+	(wire
+		(pts
+			(xy 129.54 50.8) (xy 129.54 59.69)
+		)
+		(stroke
+			(width 0)
+			(type default)
+		)
+	)
+	(wire
+		(pts
+			(xy 148.59 68.58) (xy 154.94 68.58)
+		)
+		(stroke
+			(width 0)
+			(type default)
+		)
+	)
+	(wire
+		(pts
+			(xy 148.59 81.28) (xy 154.94 81.28)
+		)
+		(stroke
+			(width 0)
+			(type default)
+		)
+	)
+	(wire
+		(pts
+			(xy 148.59 71.12) (xy 154.94 71.12)
 		)
 		(stroke
@@
 		(pts
 			(xy 148.59 148.59) (xy 154.94 148.59)
+		)
+		(stroke
+			(width 0)
+			(type default)
+		)
+	)
+	(wire
+		(pts
+			(xy 127 50.8) (xy 127 59.69)
+		)
+		(stroke
+			(width 0)
+			(type default)
+		)
+	)
+	(wire
+		(pts
+			(xy 148.59 76.2) (xy 154.94 76.2)
 		)
 		(stroke
@@
 		)
 		(stroke
+			(width 0)
+			(type default)
+		)
+	)
+	(wire
+		(pts
+			(xy 137.16 50.8) (xy 137.16 59.69)
+		)
+		(stroke
+			(width 0)
+			(type default)
+		)
+	)
+	(wire
+		(pts
+			(xy 148.59 78.74) (xy 154.94 78.74)
+		)
+		(stroke
+			(width 0)
+			(type default)
+		)
+	)
+	(wire
+		(pts
+			(xy 134.62 50.8) (xy 134.62 59.69)
+		)
+		(stroke

Commit message: sch update
Other:
- sheet MCU_IO ports: added PWR.ALRT_N, PWR.CHG_EN_N, PWR.EN_3V3, PWR.INT_N, PWR.RIN_N, PWR.SCL, PWR.SDA, USB.DM, USB.DP; removed FG_ALRT_N, PWR_INT_N, PWR_SCL, PWR_SDA, USB_DM, USB_DP
- sheet PWR ports: added PWR.ALRT_N, PWR.CHG_EN_N, PWR.EN_3V3, PWR.INT_N, PWR.RIN_N, PWR.SCL, PWR.SDA, USB.DM, USB.DP; removed EN_3V3, FG_ALRT_N, PWR_CHG_EN_N, PWR_INT_N, PWR_RIN_N, PWR_SCL, PWR_SDA, USB_DM, USB_DP

Commit message: sch update
Other:
- sheet MCU_IO ports: added ALS.INT_N, BARO.INT, HAPTIC.EN, IMU.INT1, IMU.INT2, MAG.DRDY, PPG.INT_N, SENSOR.SCL, SENSOR.SDA; removed ALS_INT_N, BARO_INT, HAPTIC_EN, IMU_INT1, IMU_INT2, MAG_DRDY, PPG_INT_N, SENSOR_SCL, SENSOR_SDA
- sheet SENSOR ports: added ALS.INT_N, BARO.INT, HAPTIC.EN, IMU.INT1, IMU.INT2, LRA.N, LRA.P, MAG.DRDY, PPG.INT_N, SENSOR.SCL, SENSOR.SDA; removed ALS_INT_N, BARO_INT, HAPTIC_EN, IMU_INT1, IMU_INT2, LRA_N, LRA_P, MAG_DRDY, PPG_INT_N, SENSOR_SCL, SENSOR_SDA
Changed lines of the file:
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@@
 			)
 		)
-		(pin "ALS_INT_N" output
+		(pin "BARO.INT" output
+			(at 154.94 114.3 180)
+			(effects
+				(font
+					(size 1.27 1.27)
+				)
+				(justify left)
+			)
+		)
+		(pin "LRA.N" output
+			(at 177.8 114.3 0)
+			(effects
+				(font
+					(size 1.27 1.27)
+				)
+				(justify right)
+			)
+		)
+		(pin "LRA.P" output
+			(at 177.8 111.76 0)
+			(effects
+				(font
+					(size 1.27 1.27)
+				)
+				(justify right)
+			)
+		)
+		(pin "HAPTIC.EN" input
+			(at 154.94 119.38 180)
+			(effects
+				(font
+					(size 1.27 1.27)
+				)
+				(justify left)
+			)
+		)
+		(pin "SENSOR.SCL" input
+			(at 154.94 97.79 180)
+			(effects
+				(font
+					(size 1.27 1.27)
+				)
+				(justify left)
+			)
+		)
+		(pin "IMU.INT2" output
+			(at 154.94 109.22 180)
+			(effects
+				(font
+					(size 1.27 1.27)
+				)
+				(justify left)
+			)
+		)
+		(pin "SENSOR.SDA" bidirectional
+			(at 154.94 100.33 180)
+			(effects
+				(font
+					(size 1.27 1.27)
+				)
+				(justify left)
+			)
+		)
+		(pin "ALS.INT_N" output
 			(at 154.94 104.14 180)
 			(effects
@@
 			)
 		)
-		(pin "IMU_INT2" output
-			(at 154.94 109.22 180)
-			(effects
-				(font
-					(size 1.27 1.27)
-				)
-				(justify left)
-			)
-		)
-		(pin "SENSOR_SCL" input
-			(at 154.94 97.79 180)
-			(effects
-				(font
-					(size 1.27 1.27)
-				)
-				(justify left)
-			)
-		)
-		(pin "MAG_DRDY" output
+		(pin "MAG.DRDY" output
 			(at 154.94 111.76 180)
 			(effects
@@
 			)
 		)
-		(pin "BARO_INT" output
-			(at 154.94 114.3 180)
-			(effects
-				(font
-					(size 1.27 1.27)
-				)
-				(justify left)
-			)
-		)
-		(pin "LRA_N" output
-			(at 177.8 107.95 0)
-			(effects
-				(font
-					(size 1.27 1.27)
-				)
-				(justify right)
-			)
-		)
-		(pin "IMU_INT1" output
+		(pin "IMU.INT1" output
 			(at 154.94 106.68 180)
 			(effects
@@
 			)
 		)
-		(pin "HAPTIC_EN" input
-			(at 154.94 119.38 180)
-			(effects
-				(font
-					(size 1.27 1.27)
-				)
-				(justify left)
-			)
-		)
-		(pin "LRA_P" output
-			(at 177.8 105.41 0)
-			(effects
-				(font
-					(size 1.27 1.27)
-				)
-				(justify right)
-			)
-		)
-		(pin "PPG_INT_N" output
+		(pin "PPG.INT_N" output
 			(at 154.94 116.84 180)
-			(effects
-				(font
-					(size 1.27 1.27)
-				)
-				(justify left)
-			)
-		)
-		(pin "SENSOR_SDA" bidirectional
-			(at 154.94 100.33 180)
 			(effects
 				(font
@@
 			)
 		)
-		(pin "ALS_INT_N" input
-			(at 148.59 104.14 0)
-			(effects
-				(font
-					(size 1.27 1.27)
-				)
-				(justify right)
-			)
-		)
-		(pin "IMU_INT1" input
-			(at 148.59 106.68 0)
-			(effects
-				(font
-					(size 1.27 1.27)
-				)
-				(justify right)
-			)
-		)
-		(pin "MAG_DRDY" input
-			(at 148.59 111.76 0)
-			(effects
-				(font
-					(size 1.27 1.27)
-				)
-				(justify right)
-			)
-		)
-		(pin "HAPTIC_EN" output
-			(at 148.59 119.38 0)
-			(effects
-				(font
-					(size 1.27 1.27)
-				)
-				(justify right)
-			)
-		)
-		(pin "SENSOR_SDA" bidirectional
-			(at 148.59 100.33 0)
-			(effects
-				(font
-					(size 1.27 1.27)
-				)
-				(justify right)
-			)
-		)
-		(pin "SENSOR_SCL" output
-			(at 148.59 97.79 0)
-			(effects
-				(font
-					(size 1.27 1.27)
-				)
-				(justify right)
-			)
-		)
-		(pin "BARO_INT" input
-			(at 148.59 114.3 0)
-			(effects
-				(font
-					(size 1.27 1.27)
-				)
-				(justify right)
-			)
-		)
-		(pin "IMU_INT2" input
-			(at 148.59 109.22 0)
-			(effects
-				(font
-					(size 1.27 1.27)
-				)
-				(justify right)
-			)
-		)
-		(pin "PPG_INT_N" input
-			(at 148.59 116.84 0)
-			(effects
-				(font
-					(size 1.27 1.27)
-				)
-				(justify right)
-			)
-		)
 		(pin "OSPI.NCS" output
 			(at 148.59 78.74 0)
@@
 			)
 		)
+		(pin "BARO.INT" input
+			(at 148.59 114.3 0)
+			(effects
+				(font
+					(size 1.27 1.27)
+				)
+				(justify right)
+			)
+		)
+		(pin "PPG.INT_N" input
+			(at 148.59 116.84 0)
+			(effects
+				(font
+					(size 1.27 1.27)
+				)
+				(justify right)
+			)
+		)
+		(pin "SENSOR.SDA" bidirectional
+			(at 148.59 100.33 0)
+			(effects
+				(font
+					(size 1.27 1.27)
+				)
+				(justify right)
+			)
+		)
+		(pin "SENSOR.SCL" output
+			(at 148.59 97.79 0)
+			(effects
+				(font
+					(size 1.27 1.27)
+				)
+				(justify right)
+			)
+		)
+		(pin "IMU.INT2" input
+			(at 148.59 109.22 0)
+			(effects
+				(font
+					(size 1.27 1.27)
+				)
+				(justify right)
+			)
+		)
+		(pin "MAG.DRDY" input
+			(at 148.59 111.76 0)
+			(effects
+				(font
+					(size 1.27 1.27)
+				)
+				(justify right)
+			)
+		)
+		(pin "HAPTIC.EN" output
+			(at 148.59 119.38 0)
+			(effects
+				(font
+					(size 1.27 1.27)
+				)
+				(justify right)
+			)
+		)
+		(pin "ALS.INT_N" input
+			(at 148.59 104.14 0)
+			(effects
+				(font
+					(size 1.27 1.27)
+				)
+				(justify right)
+			)
+		)
+		(pin "IMU.INT1" input
+			(at 148.59 106.68 0)
+			(effects
+				(font
+					(size 1.27 1.27)
+				)
+				(justify right)
+			)
+		)

Commit message: add pdf
Other:
- added sheet NFC (NFC.kicad_sch)
Changed lines of the file:
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@@
+	)
+	(sheet
+		(at 90.17 143.51)
+		(size 16.51 16.51)
+		(exclude_from_sim no)
+		(in_bom yes)
+		(on_board yes)
+		(dnp no)
+		(fields_autoplaced yes)
+		(stroke
+			(width 0.1524)
+			(type solid)
+		)
+		(fill
+			(color 0 0 0 0)
+		)
+		(property "Sheetname" "NFC"
+			(at 90.17 142.7984 0)
+			(show_name no)
+			(do_not_autoplace no)
+			(effects
+				(font
+					(size 1.27 1.27)
+				)
+				(justify left bottom)
+			)
+		)
+		(property "Sheetfile" "NFC.kicad_sch"
+			(at 90.17 160.6046 0)
+			(show_name no)
+			(do_not_autoplace no)
+			(effects
+				(font
+					(size 1.27 1.27)
+				)
+				(justify left top)
+			)
+		)
+		(instances
+			(project "XWatch_Rev3.0"
+				(path "/64425c00-526a-4829-b8a6-ed1dc1b19578"
+					(page "10")
+				)
+			)
+		)
 	)
 	(sheet
@@
 	)
 	(sheet
-		(at 83.82 105.41)
-		(size 22.86 36.83)
+		(at 87.63 105.41)
+		(size 19.05 31.75)
 		(exclude_from_sim no)
 		(in_bom yes)
@@
 		)
 		(property "Sheetname" "PWR"
-			(at 83.82 104.6984 0)
+			(at 87.63 104.6984 0)
 			(show_name no)
 			(do_not_autoplace no)
@@
 		)
 		(property "Sheetfile" "PWR.kicad_sch"
-			(at 83.82 142.8246 0)
-			(show_name no)
-			(do_not_autoplace no)
+			(at 87.63 137.7446 0)
+			(show_name no)
+			(do_not_autoplace no)
