File: hardware/schematic/v1.0/XWatch_Rev3.0/MCU_IO.kicad_sch (KiCad schematic)
At the start: 11 parts, among them U1 STM32U5G9NJH6Q, X1 32.768KHZ, X2 16MHZ

Commit message: sch update
Parts:
- added U15: STM32U5A9BJY6QTR, XWatch_Rev3.0:STM32U5A9BJY6QTR, symbol XWatch_Rev3.0:STM32U5A9BJY6QTR
Connections:
- net DSI_CK_N: now also U15.H25 (DSI_CKN); no longer U1.J1 (DSI_CKN)
- net DSI_CK_P: now also U15.G26 (DSI_CKP); no longer U1.H1 (DSI_CKP)
- net DSI_D0_N: now also U15.F25 (DSI_D0N); no longer U1.G2 (DSI_D0N)
- net DSI_D0_P: now also U15.E26 (DSI_D0P); no longer U1.G1 (DSI_D0P)
- net DSI_D1_N: now also U15.K25 (DSI_D1N); no longer U1.K1 (DSI_D1N)
- net DSI_D1_P: now also U15.J26 (DSI_D1P); no longer U1.K2 (DSI_D1P)
- net OSPI_CLK: now also U15.M13 (PE10)
- net OSPI_IO0: now also U15.R14 (PE12)
- net OSPI_IO1: now also U15.N12 (PE13)
- net OSPI_IO2: now also U15.P13 (PE14)
- net OSPI_IO3: now also U15.R12 (PE15)
- net OSPI_NCS: now also U15.P15 (PE11)
- net PWR_SCL: now also U15.C16 (PG14); no longer U1.D7 (PG14)
- net PWR_SDA: now also U15.A14 (PG13); no longer U1.B6 (PG13)
- net SENSOR_SCL: now also U15.E12 (PH7); no longer U1.B11 (PH7)
- net SENSOR_SDA: now also U15.G16 (PH8); no longer U1.D10 (PH8)
- net SW2: now also U15.L16 (PA1); no longer U1.P3 (PA1-WKUP3)
- net SW3: now also U15.M17 (PA2); no longer U1.M4 (PA2-WKUP4)
- net SW4: now also U15.P23 (PA3); no longer U1.P4 (PA3-WKUP5)
- net SW5: now also U15.N20 (PA4); no longer U1.M5 (PA4-WKUP2)
- net TP_SCL: now also U15.H15 (PH6); no longer U1.B12 (PH5)
- net TP_SDA: now also U15.F13 (PH5); no longer U1.C12 (PH4)
- net at C2.2, X1.2: now also U15.D25 (PC15-OSC32_OUT); no longer U1.B1 (PC14-OSC32_IN)
- net at U1.B4 (PH3-BOOT0): no longer R8.1
- net at C1.2, X1.1: now also U15.C26 (PC14-OSC32_IN); no longer U1.C1 (PC15-OSC32_OUT)
- net at D1.2 (A), R18.2: now also U15.N22 (PA0); no longer U1.N4 (PA0-WKUP1)
- new net: R8.1, U15.E20 (PH3-BOOT0)
Other:
- moved on the sheet: C3, C4, C48, U1A, U1B, U1D, X2

Commit message: sch update
Parts:
- removed U1: STM32U5G9NJH6Q, XWatch_Rev3.0:STM32U5G9NJH6Q, symbol XWatch_Rev3.0:STM32U5G9NJH6Q
Connections:
- net DSI_PWR_EN: now also U15.C22 (PI5)
- net DSI_RESET: now also U15.E16 (PD5)
- net DSI_TE: now also U15.N16 (PF11)
- net SENSOR_SCL: now also U15.H15 (PH6); no longer U15.E12 (PH7)
- net SENSOR_SDA: now also U15.E12 (PH7); no longer U15.G16 (PH8)
- net TP_INT: now also U15.N14 (PE8)
- net TP_RESET: now also U15.D21 (PI6)
- net TP_SCL: now also U15.F13 (PH5); no longer U15.H15 (PH6)
- net TP_SDA: now also U15.E10 (PH4); no longer U15.F13 (PH5)
- net at X2.3 (OSC2): now also U15.M25 (PH1-OSC_OUT)
- net at C4.1, X2.1 (OSC1): now also U15.M23 (PH0-OSC_IN)
- net at C48.1: now also U15.M21 (NRST)
- net IMU_INT2: now reaches U15.J14 (PF7)
- net IMU_INT1: now reaches U15.J16 (PF6)
- net ALS_INT_N: now reaches U15.K21 (PF5)
- net MAG_DRDY: now reaches U15.L20 (PF9)
- net BARO_INT: now reaches U15.L22 (PF10)
- net HAPTIC_EN: now reaches U15.P17 (PF13)
- net PPG_INT_N: now reaches U15.T21 (PF12)
Other:
- note added: "PF10"
- note added: "PF12"
- note added: "PF13"
- note added: "PF5"
- note added: "PF6"
- note added: "PF7"
- note added: "PF9"
- moved on the sheet: C1, C2, X1

Commit message: sch update
Connections:
- net USB_DP: now reaches U15.B1 (PA12)
- net USB_DM: now reaches U15.C2 (PA11)
Other:
- note added: "PA11"
- note added: "PA12"
Changed lines of the file:
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@@
+		)
+	)
+	(text "PA11"
+		(exclude_from_sim no)
+		(at 211.582 114.808 0)
+		(effects
+			(font
+				(size 1.27 1.27)
+			)
 		)
 	)
@@
 		)
 	)
+	(text "PA12"
+		(exclude_from_sim no)
+		(at 211.582 117.602 0)
+		(effects
+			(font
+				(size 1.27 1.27)
+			)
+		)
+	)
 	(text "PH7"
 		(exclude_from_sim no)
@@
 		)
 	)
+	(text "PA12"
+		(exclude_from_sim no)
+		(at 132.842 247.142 0)
+		(effects
+			(font
+				(size 1.27 1.27)
+			)
+		)
+	)
 	(text "PG14"
 		(exclude_from_sim no)
@@
 		(exclude_from_sim no)
 		(at 88.646 61.976 0)
+		(effects
+			(font
+				(size 1.27 1.27)
+			)
+		)
+	)
+	(text "PA11"
+		(exclude_from_sim no)
+		(at 132.842 244.348 0)
 		(effects
 			(font
@@
 	(wire
 		(pts
+			(xy 214.63 115.57) (xy 229.87 115.57)
+		)
+		(stroke
+			(width 0)
+			(type default)
+		)
+	)
+	(wire
+		(pts
+			(xy 214.63 118.11) (xy 229.87 118.11)
+		)
+		(stroke
+			(width 0)
+			(type default)
+		)
+	)
+	(wire
+		(pts
 			(xy 176.53 124.46) (xy 176.53 128.27)
 		)
@@
 	(wire
 		(pts
+			(xy 135.89 247.65) (xy 149.86 247.65)
+		)
+		(stroke
+			(width 0)
+			(type default)
+		)
+	)
+	(wire
+		(pts
 			(xy 60.96 238.76) (xy 74.93 238.76)
 		)
@@
 		(pts
 			(xy 60.96 231.14) (xy 74.93 231.14)
+		)
+		(stroke
+			(width 0)
+			(type default)
+		)
+	)
+	(wire
+		(pts
+			(xy 135.89 245.11) (xy 149.86 245.11)
 		)
 		(stroke
@@
 		)
 	)
+	(label "USB_OTG_DP"
+		(at 135.89 247.65 0)
+		(effects
+			(font
+				(size 1.27 1.27)
+			)
+			(justify left bottom)
+		)
+	)
+	(label "USB_OTG_DM"
+		(at 135.89 245.11 0)
+		(effects
+			(font
+				(size 1.27 1.27)
+			)
+			(justify left bottom)
+		)
+	)
 	(label "I2C5.SDA"
 		(at 311.15 222.25 0)
@@
 		)
 	)
+	(label "USB_OTG_DP"
+		(at 214.63 118.11 0)
+		(effects
+			(font
+				(size 1.27 1.27)
+			)
+			(justify left bottom)
+		)
+	)
 	(label "OSPI.IO0"
 		(at 62.23 265.43 0)
@@
 		)
 	)
+	(label "USB_OTG_DM"
+		(at 214.63 115.57 0)
+		(effects
+			(font
+				(size 1.27 1.27)
+			)
+			(justify left bottom)
+		)
+	)
 	(hierarchical_label "PWR_INT_N"
-		(shape input)
+		(shape bidirectional)
 		(at 149.86 236.22 0)
 		(effects
@@
 		)
 	)
+	(hierarchical_label "USB_DP"
+		(shape bidirectional)
+		(at 149.86 247.65 0)
+		(effects
+			(font
+				(size 1.27 1.27)
+			)
+			(justify left)
+		)
+	)
 	(hierarchical_label "HAPTIC_EN"
 		(shape output)
@@
 		)
 	)
+	(hierarchical_label "USB_DM"
+		(shape bidirectional)
+		(at 149.86 245.11 0)
+		(effects
+			(font
+				(size 1.27 1.27)
+			)
+			(justify left)
+		)
+	)
 	(hierarchical_label "TP_INT"
 		(shape input)
@@
 	)
 	(hierarchical_label "FG_ALRT_N"
-		(shape input)
+		(shape bidirectional)
 		(at 149.86 233.68 0)
 		(effects

Commit message: sch update
Connections:
- net BLE.WAKE_MCU: now reaches U15.D23 (PC13)
- net BLE.MCU_RX: now reaches U15.R10 (PB11)
- net BLE.MCU_RTS: now reaches U15.R6 (PB14)
- net BLE.MCU_TX: now reaches U15.T13 (PB10)
- net BLE.WAKE_NRF: now reaches U15.T5 (PB12)
- net BLE.MCU_CTS: now reaches U15.T7 (PB13)
- net OSPI_CLK renamed OSPI.CLK
- net OSPI_IO0 renamed OSPI.IO0
- net OSPI_IO1 renamed OSPI.IO1
- net OSPI_IO2 renamed OSPI.IO2
- net OSPI_IO3 renamed OSPI.IO3
- net OSPI_NCS renamed OSPI.NCS
Other:
- note added: "BLE"
- note added: "PB10"
- note added: "PB11"
- note added: "PB12"
- note added: "PB13"
- note added: "PB14"
- note added: "PC13"

Commit message: sch update
Connections:
- net DSI_CK_N renamed DSI.CK_N
- net DSI_CK_P renamed DSI.CK_P
- net DSI_D0_N renamed DSI.D0_N
- net DSI_D0_P renamed DSI.D0_P
- net DSI_D1_N renamed DSI.D1_N
- net DSI_D1_P renamed DSI.D1_P
- net DSI_PWR_EN renamed DSI.PWR_EN
- net DSI_RESET renamed DSI.RESET
- net DSI_TE renamed DSI.TE
- net TP_INT renamed TP.INT
- net TP_RESET renamed TP.RESET
- net TP_SCL renamed TP.SCL
- net TP_SDA renamed TP.SDA
Changed lines of the file:
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@@
 		)
 	)
-	(label "DSI.CK_N"
+	(label "DSI_CK_N"
 		(at 217.17 67.31 0)
 		(effects
@@
 		)
 	)
-	(label "DSI.CK_N"
+	(label "DSI_CK_N"
 		(at 311.15 213.36 0)
 		(effects
@@
 		)
 	)
-	(label "DSI.TE"
+	(label "DSI_TE"
 		(at 95.25 115.57 0)
 		(effects
@@
 		)
 	)
-	(label "DSI.TE"
+	(label "DSI_TE"
 		(at 311.15 232.41 0)
 		(effects
@@
 		)
 	)
-	(label "DSI.D1_P"
+	(label "DSI_D1_P"
 		(at 217.17 80.01 0)
 		(effects
@@
 		)
 	)
-	(label "DSI.D0_N"
+	(label "DSI_D0_N"
 		(at 311.15 200.66 0)
 		(effects
@@
 		)
 	)
-	(label "DSI.D0_N"
+	(label "DSI_D0_N"
 		(at 217.17 72.39 0)
 		(effects
@@
 		)
 	)
-	(label "DSI.CK_P"
+	(label "DSI_CK_P"
 		(at 217.17 69.85 0)
 		(effects
@@
 		)
 	)
-	(label "DSI.D1_N"
+	(label "DSI_D1_N"
 		(at 217.17 77.47 0)
 		(effects
@@
 		)
 	)
-	(label "DSI.D1_P"
+	(label "DSI_D1_P"
 		(at 311.15 204.47 0)
 		(effects
@@
 		)
 	)
-	(label "DSI.CK_P"
+	(label "DSI_CK_P"
 		(at 311.15 210.82 0)
 		(effects
@@
 		)
 	)
-	(label "DSI.D0_P"
+	(label "DSI_D0_P"
 		(at 311.15 198.12 0)
 		(effects
@@
 		)
 	)
-	(label "DSI.RESET"
+	(label "DSI_RESET"
 		(at 311.15 238.76 0)
 		(effects
@@
 		)
 	)
-	(label "DSI.D0_P"
+	(label "DSI_D0_P"
 		(at 217.17 74.93 0)
 		(effects
@@
 		)
 	)
-	(label "DSI.RESET"
+	(label "DSI_RESET"
 		(at 278.13 124.46 0)
 		(effects
@@
 		)
 	)
-	(label "DSI.D1_N"
+	(label "DSI_D1_N"
 		(at 311.15 207.01 0)
 		(effects
@@
 		)
 	)
-	(hierarchical_label "TP_SCL"
+	(hierarchical_label "TP.SCL"
 		(shape output)
 		(at 325.12 224.79 0)
@@
 		)
 	)
-	(hierarchical_label "DSI_PWR_EN"
+	(hierarchical_label "DSI.PWR_EN"
 		(shape output)
 		(at 382.27 238.76 0)
@@
 		)
 	)
-	(hierarchical_label "TP_INT"
+	(hierarchical_label "TP.INT"
 		(shape input)
 		(at 382.27 234.95 0)
@@
 		)
 	)
-	(hierarchical_label "DSI_CK_P"
+	(hierarchical_label "DSI.CK_P"
 		(shape bidirectional)
 		(at 325.12 210.82 0)
@@
 		)
 	)
-	(hierarchical_label "DSI_D0_N"
+	(hierarchical_label "DSI.D0_N"
 		(shape bidirectional)
 		(at 325.12 200.66 0)
@@
 		)
 	)
-	(hierarchical_label "DSI_CK_N"
+	(hierarchical_label "DSI.CK_N"
 		(shape bidirectional)
 		(at 325.12 213.36 0)
@@
 		)
 	)
-	(hierarchical_label "DSI_D1_P"
+	(hierarchical_label "DSI.D1_P"
 		(shape bidirectional)
 		(at 325.12 204.47 0)
@@
 		)
 	)
-	(hierarchical_label "TP_SDA"
+	(hierarchical_label "TP.SDA"
 		(shape bidirectional)
 		(at 325.12 222.25 0)
@@
 		)
 	)
-	(hierarchical_label "DSI_D1_N"
+	(hierarchical_label "DSI.D1_N"
 		(shape bidirectional)
 		(at 325.12 207.01 0)
@@
 		)
 	)
-	(hierarchical_label "DSI_RESET"
+	(hierarchical_label "DSI.RESET"
 		(shape output)
 		(at 325.12 238.76 0)
@@
 		)
 	)
-	(hierarchical_label "DSI_TE"
+	(hierarchical_label "DSI.TE"
 		(shape input)
 		(at 325.12 232.41 0)
@@
 		)
 	)
-	(hierarchical_label "TP_RESET"
+	(hierarchical_label "TP.RESET"
 		(shape output)
 		(at 382.27 231.14 0)
@@
 		)
 	)
-	(hierarchical_label "DSI_D0_P"
+	(hierarchical_label "DSI.D0_P"
 		(shape bidirectional)
 		(at 325.12 198.12 0)

Commit message: sch update
Connections:
- net PWR.RIN_N: now reaches U15.A10 (PD1)
- net SWDIO: now reaches U15.B3 (PA13)
- net PWR.ALRT_N: now reaches U15.C12 (PD3)
- net SWCLK: now reaches U15.D11 (PA14)
- net PWR.CHG_EN_N: now reaches U15.D13 (PD2)
- net PWR.INT_N: now reaches U15.D15 (PD4)
- net PWR.EN_3V3: now reaches U15.F15 (PD0)
- net PWR_SCL renamed PWR.SCL
- net PWR_SDA renamed PWR.SDA
- net USB_DM renamed USB.DM
- net USB_DP renamed USB.DP
Other:
- note added: "PA13"
- note added: "PA14"
- note added: "PD0"
- note added: "PD1"
- note added: "PD2"
- note added: "PD3"
- note added: "PD4"

Commit message: sch update
Parts:
- added TP1, TP2, TP3, TP4: TestPoint, TestPoint:TestPoint_Pad_D1.0mm, symbol Connector:TestPoint
Connections:
- net GND: now also TP4.1
- net SWCLK: now also TP2.1
- net SWDIO: now also TP1.1
- net NRST: now reaches C48.1, U15.M21 (NRST)
- net NRST: now also TP3.1
- no-connect marks 0 -> 96
Other:
- note added: "SWD"
