File: hardware/schematic/v1.0/XWatch_Rev3.0/MCU_IO.kicad_sch (KiCad schematic)
At the start: 15 parts, among them U15 STM32U5A9BJY6QTR, X1 32.768KHZ, X2 16MHZ

Commit message: sch update
Connections:
- net ALS_INT_N renamed ALS.INT_N
- net BARO_INT renamed BARO.INT
- net HAPTIC_EN renamed HAPTIC.EN
- net IMU_INT1 renamed IMU.INT1
- net IMU_INT2 renamed IMU.INT2
- net MAG_DRDY renamed MAG.DRDY
- net PPG_INT_N renamed PPG.INT_N
- net SENSOR_SCL renamed SENSOR.SCL
- net SENSOR_SDA renamed SENSOR.SDA
Changed lines of the file:
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@@
 		)
 	)
-	(hierarchical_label "ALS_INT_N"
+	(hierarchical_label "ALS.INT_N"
 		(shape input)
 		(at 229.87 232.41 0)
@@
 		)
 	)
-	(hierarchical_label "HAPTIC_EN"
+	(hierarchical_label "HAPTIC.EN"
 		(shape output)
 		(at 229.87 247.65 0)
@@
 		)
 	)
-	(hierarchical_label "BARO_INT"
+	(hierarchical_label "BARO.INT"
 		(shape input)
 		(at 229.87 242.57 0)
@@
 		)
 	)
-	(hierarchical_label "SENSOR_SCL"
+	(hierarchical_label "SENSOR.SCL"
 		(shape output)
 		(at 229.87 227.33 0)
@@
 		)
 	)
-	(hierarchical_label "IMU_INT2"
+	(hierarchical_label "IMU.INT2"
 		(shape input)
 		(at 229.87 237.49 0)
@@
 		)
 	)
-	(hierarchical_label "PPG_INT_N"
+	(hierarchical_label "PPG.INT_N"
 		(shape input)
 		(at 229.87 245.11 0)
@@
 		)
 	)
-	(hierarchical_label "SENSOR_SDA"
+	(hierarchical_label "SENSOR.SDA"
 		(shape bidirectional)
 		(at 229.87 224.79 0)
@@
 		)
 	)
-	(hierarchical_label "MAG_DRDY"
+	(hierarchical_label "MAG.DRDY"
 		(shape input)
 		(at 229.87 240.03 0)
@@
 		)
 	)
-	(hierarchical_label "IMU_INT1"
+	(hierarchical_label "IMU.INT1"
 		(shape input)
 		(at 229.87 234.95 0)
