File: hardware/schematic/v1.0/XWatch_Rev3.0/PWR.kicad_sch (KiCad schematic)
At the start: 33 parts, among them U13 SK6018D4-33, U3 DA9168, U4 TPS62840DLCR, U5 MAX17048G_T10, U8 SM03B-SRSS-TB_LF_SN_P

Commit message: sch update
Parts:
- added CN1, CN2, CN3, CN4: SCTA1A0100, XWatch_Rev3.0:SCTA1A0100, symbol XWatch_Rev3.0:SCTA1A0100
Connections:
- net GND: now also CN4.1
- net VBUS: now also CN1.1
- new net USB_DM: CN3.1
- new net USB_DP: CN2.1

Commit message: sch update
Connections:
- net EN_3V3 renamed PWR.EN_3V3
- net FG_ALRT_N renamed PWR.ALRT_N
- net PWR_CHG_EN_N renamed PWR.CHG_EN_N
- net PWR_INT_N renamed PWR.INT_N
- net PWR_RIN_N renamed PWR.RIN_N
- net PWR_SCL renamed PWR.SCL
- net PWR_SDA renamed PWR.SDA
- net USB_DM renamed USB.DM
- net USB_DP renamed USB.DP
Other:
- moved on the sheet: C65
Changed lines of the file:
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@@
 	)
 	(junction
-		(at 237.49 54.61)
+		(at 242.57 54.61)
 		(diameter 0)
 		(color 0 0 0 0)
@@
 	(wire
 		(pts
-			(xy 237.49 54.61) (xy 240.03 54.61)
+			(xy 242.57 54.61) (xy 245.11 54.61)
 		)
 		(stroke
@@
 	(wire
 		(pts
-			(xy 237.49 64.77) (xy 237.49 66.04)
+			(xy 242.57 64.77) (xy 242.57 66.04)
 		)
 		(stroke
@@
 	(wire
 		(pts
-			(xy 237.49 54.61) (xy 237.49 57.15)
+			(xy 242.57 54.61) (xy 242.57 57.15)
 		)
 		(stroke
@@
 	(wire
 		(pts
-			(xy 218.44 54.61) (xy 237.49 54.61)
+			(xy 218.44 54.61) (xy 242.57 54.61)
 		)
 		(stroke
@@
 		)
 	)
-	(hierarchical_label "PWR_SCL"
+	(hierarchical_label "PWR.SCL"
 		(shape input)
 		(at 120.65 100.33 0)
@@
 		)
 	)
-	(hierarchical_label "PWR_INT_N"
+	(hierarchical_label "PWR.INT_N"
 		(shape output)
 		(at 120.65 107.95 0)
@@
 		)
 	)
-	(hierarchical_label "PWR_SDA"
+	(hierarchical_label "PWR.SDA"
 		(shape bidirectional)
 		(at 120.65 104.14 0)
@@
 		)
 	)
-	(hierarchical_label "USB_DM"
+	(hierarchical_label "USB.DM"
 		(shape bidirectional)
 		(at 101.6 170.18 180)
@@
 		)
 	)
-	(hierarchical_label "FG_ALRT_N"
+	(hierarchical_label "PWR.ALRT_N"
 		(shape output)
 		(at 241.3 149.86 180)
@@
 		)
 	)
-	(hierarchical_label "PWR_RIN_N"
-		(shape output)
+	(hierarchical_label "PWR.RIN_N"
+		(shape input)
 		(at 132.08 115.57 0)
 		(effects
@@
 		)
 	)
-	(hierarchical_label "PWR_CHG_EN_N"
+	(hierarchical_label "PWR.CHG_EN_N"
 		(shape input)
 		(at 132.08 119.38 0)
@@
 		)
 	)
-	(hierarchical_label "USB_DP"
+	(hierarchical_label "USB.DP"
 		(shape bidirectional)
 		(at 101.6 162.56 180)
@@
 		)
 	)
-	(hierarchical_label "PWR_SDA"
+	(hierarchical_label "PWR.SDA"
 		(shape bidirectional)
 		(at 217.17 92.71 0)
@@
 		)
 	)
-	(hierarchical_label "PWR_SDA"
+	(hierarchical_label "PWR.SDA"
 		(shape bidirectional)
 		(at 241.3 142.24 180)
@@
 		)
 	)
-	(hierarchical_label "FG_ALRT_N"
+	(hierarchical_label "PWR.ALRT_N"
 		(shape output)
 		(at 217.17 100.33 0)
@@
 		)
 	)
-	(hierarchical_label "PWR_INT_N"
+	(hierarchical_label "PWR.INT_N"
 		(shape output)
 		(at 241.3 146.05 180)
@@
 		)
 	)
-	(hierarchical_label "PWR_SCL"
+	(hierarchical_label "PWR.SCL"
 		(shape input)
 		(at 241.3 138.43 180)
@@
 		)
 	)
-	(hierarchical_label "PWR_SCL"
+	(hierarchical_label "PWR.SCL"
 		(shape input)
 		(at 217.17 95.25 0)
@@
 		)
 	)
-	(hierarchical_label "EN_3V3"
+	(hierarchical_label "PWR.EN_3V3"
 		(shape input)
 		(at 224.79 57.15 0)
@@
 	(symbol
 		(lib_id "XWatch_Rev3.0:GND")
-		(at 237.49 66.04 0)
+		(at 242.57 66.04 0)
 		(unit 1)
 		(body_style 1)
@@
 		(fields_autoplaced yes)
 		(property "Reference" "#PWR0196"
-			(at 237.49 72.39 0)
+			(at 242.57 72.39 0)
 			(hide yes)
 			(show_name no)
@@
 		)
 		(property "Value" "GND"
-			(at 237.4899 69.85 90)
+			(at 242.5699 69.85 90)
 			(hide yes)
 			(show_name no)
@@
 		)
 		(property "Footprint" ""
-			(at 237.49 66.04 0)
+			(at 242.57 66.04 0)
 			(hide yes)
 			(show_name no)
@@
 		)
 		(property "Datasheet" ""
-			(at 237.49 66.04 0)
+			(at 242.57 66.04 0)
 			(hide yes)
 			(show_name no)
@@
 		)
 		(property "Description" "Power symbol creates a global label with name \"GND\" , ground"
-			(at 237.49 66.04 0)
+			(at 242.57 66.04 0)
 			(hide yes)
 			(show_name no)
@@
 	(symbol
 		(lib_id "XWatch_Rev3.0:C")
-		(at 237.49 60.96 0)
+		(at 242.57 60.96 0)
 		(unit 1)
 		(body_style 1)
@@
 		(dnp no)
 		(property "Reference" "C65"
-			(at 238.252 58.674 0)
+			(at 243.332 58.674 0)
 			(show_name no)
 			(do_not_autoplace no)
@@
 		)
 		(property "Value" "1uF"
-			(at 238.252 63.5 0)
+			(at 243.332 63.5 0)
 			(show_name no)
 			(do_not_autoplace no)
@@
 		)
 		(property "Footprint" "XWatch_Rev3.0:GEN_C_0402"
-			(at 238.4552 64.77 0)
+			(at 243.5352 64.77 0)
 			(hide yes)
 			(show_name no)
@@
 		)
 		(property "Datasheet" ""
-			(at 237.49 60.96 0)
+			(at 242.57 60.96 0)
 			(hide yes)
 			(show_name no)
@@
 		)
 		(property "Description" "Unpolarized capacitor"
-			(at 237.49 60.96 0)
+			(at 242.57 60.96 0)
 			(hide yes)
 			(show_name no)
@@
 	(symbol
 		(lib_id "XWatch_Rev3.0:VSYS")
-		(at 240.03 54.61 0)
+		(at 245.11 54.61 0)
 		(unit 1)
 		(body_style 1)
@@
 		(fields_autoplaced yes)
 		(property "Reference" "#PWR011"
-			(at 240.03 58.42 0)
+			(at 245.11 58.42 0)
 			(hide yes)
 			(show_name no)
@@
 		)
 		(property "Value" "VSYS"
-			(at 240.03 49.53 0)
+			(at 245.11 49.53 0)
 			(show_name no)
 			(do_not_autoplace no)
@@
 		)
 		(property "Footprint" ""
-			(at 240.03 54.61 0)
+			(at 245.11 54.61 0)
 			(hide yes)
 			(show_name no)
@@
 		)
 		(property "Datasheet" ""
-			(at 240.03 54.61 0)
+			(at 245.11 54.61 0)
 			(hide yes)
 			(show_name no)
@@
 		)
 		(property "Description" "Power symbol creates a global label with name \"VSYS\""
-			(at 240.03 54.61 0)
+			(at 245.11 54.61 0)
 			(hide yes)
 			(show_name no)

Commit message: sch update
Changed lines of the file:
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@@
 		(color 0 0 0 0)
 	)
+	(junction
+		(at 95.25 152.2464)
+		(diameter 0)
+		(color 0 0 0 0)
+	)
 	(wire
 		(pts
@@
 	(wire
 		(pts
+			(xy 95.25 151.13) (xy 95.25 152.2464)
+		)
+		(stroke
+			(width 0)
+			(type default)
+		)
+	)
+	(wire
+		(pts
 			(xy 60.96 58.42) (xy 67.31 58.42)
 		)
@@
 	(wire
 		(pts
+			(xy 95.25 153.67) (xy 101.6 153.67)
+		)
+		(stroke
+			(width 0)
+			(type default)
+		)
+	)
+	(wire
+		(pts
 			(xy 46.99 58.42) (xy 60.96 58.42)
 		)
@@
 	(wire
 		(pts
+			(xy 95.25 152.2464) (xy 95.25 153.67)
+		)
+		(stroke
+			(width 0)
+			(type default)
+		)
+	)
+	(wire
+		(pts
 			(xy 156.21 139.7) (xy 158.75 139.7)
 		)
@@
 	(wire
 		(pts
-			(xy 93.98 153.67) (xy 101.6 153.67)
-		)
-		(stroke
-			(width 0)
-			(type default)
-		)
-	)
-	(wire
-		(pts
 			(xy 182.88 49.53) (xy 182.88 48.26)
 		)
@@
 	(symbol
 		(lib_id "XWatch_Rev3.0:VBUS")
-		(at 93.98 153.67 0)
+		(at 95.25 151.13 0)
 		(unit 1)
 		(body_style 1)
@@
 		(fields_autoplaced yes)
 		(property "Reference" "#PWR013"
-			(at 93.98 157.48 0)
+			(at 95.25 154.94 0)
 			(hide yes)
 			(show_name no)
@@
 		)
 		(property "Value" "VBUS"
-			(at 93.98 148.59 0)
+			(at 95.25 146.05 0)
 			(show_name no)
 			(do_not_autoplace no)
@@
 		)
 		(property "Footprint" ""
-			(at 93.98 153.67 0)
+			(at 95.25 151.13 0)
 			(hide yes)
 			(show_name no)
@@
 		)
 		(property "Datasheet" ""
-			(at 93.98 153.67 0)
+			(at 95.25 151.13 0)
 			(hide yes)
 			(show_name no)
@@
 		)
 		(property "Description" "Power symbol creates a global label with name \"VBUS\""
-			(at 93.98 153.67 0)
+			(at 95.25 151.13 0)
 			(hide yes)
 			(show_name no)
@@
 					(unit 1)
 				)
+			)
+		)
+	)
+	(symbol
+		(lib_id "XWatch_Rev3.0:PWR_FLAG")
+		(at 95.25 152.2464 90)
+		(unit 1)
+		(body_style 1)
+		(exclude_from_sim no)
+		(in_bom yes)
+		(on_board yes)
+		(in_pos_files yes)
+		(dnp no)
+		(property "Reference" "#FLG06"
+			(at 93.345 152.2464 0)
+			(hide yes)
+			(show_name no)
+			(do_not_autoplace no)
+			(effects
+				(font
+					(size 1.27 1.27)
+				)
+			)
+		)
+		(property "Value" "PWR_FLAG"
+			(at 92.456 152.2464 90)
+			(show_name no)
+			(do_not_autoplace no)
+			(effects
+				(font
+					(size 1.27 1.27)
+				)
+				(justify left)
+			)
+		)
+		(property "Footprint" ""
+			(at 95.25 152.2464 0)
+			(hide yes)
+			(show_name no)
+			(do_not_autoplace no)
+			(effects
+				(font
+					(size 1.27 1.27)
+				)
+			)
+		)
+		(property "Datasheet" ""
+			(at 95.25 152.2464 0)
+			(hide yes)
+			(show_name no)
+			(do_not_autoplace no)
+			(effects
+				(font
+					(size 1.27 1.27)
+				)
+			)
+		)
+		(property "Description" "Special symbol for telling ERC where power comes from"
+			(at 95.25 152.2464 0)
+			(hide yes)
+			(show_name no)
+			(do_not_autoplace no)
+			(effects
+				(font
+					(size 1.27 1.27)
+				)
+			)
+		)
+		(pin "1"
+		)
+		(instances
+			(project "XWatch_Rev3.0"
+				(path "/64425c00-526a-4829-b8a6-ed1dc1b19578/e10fc6fe-cee5-4ccf-ade7-f348522d306a"
+					(reference "#FLG06")
+					(unit 1)
+				)
