File: hardware/schematic/v1.0/XWatch_Rev3.0/DSI_LCD.kicad_sch (KiCad schematic)
At the start: 12 parts, among them U14 AXE530127-DO0143FMST02

Commit message: sch update
Connections:
- net DSI_CK_N renamed DSI.CK_N
- net DSI_CK_P renamed DSI.CK_P
- net DSI_D0_N renamed DSI.D0_N
- net DSI_D0_P renamed DSI.D0_P
- net DSI_PWR_EN renamed DSI.PWR_EN
- net DSI_RESET renamed DSI.RESET
- net DSI_TE renamed DSI.TE
- net TP_INT renamed TP.INT
- net TP_RESET renamed TP.RESET
- net TP_SCL renamed TP.SCL
- net TP_SDA renamed TP.SDA
Changed lines of the file:
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@@
 		)
 	)
-	(hierarchical_label "TP_RESET"
+	(hierarchical_label "TP.RESET"
 		(shape input)
 		(at 113.03 97.79 180)
@@
 		)
 	)
-	(hierarchical_label "DSI_RESET"
+	(hierarchical_label "DSI.RESET"
 		(shape input)
 		(at 156.21 109.22 0)
@@
 		)
 	)
-	(hierarchical_label "DSI_CK_P"
+	(hierarchical_label "DSI.CK_P"
 		(shape bidirectional)
 		(at 156.21 113.03 0)
@@
 		)
 	)
-	(hierarchical_label "TP_SCL"
+	(hierarchical_label "TP.SCL"
 		(shape input)
 		(at 113.03 74.93 180)
@@
 		)
 	)
-	(hierarchical_label "TP_SCL"
+	(hierarchical_label "TP.SCL"
 		(shape input)
 		(at 224.79 121.92 180)
@@
 		)
 	)
-	(hierarchical_label "DSI_CK_N"
+	(hierarchical_label "DSI.CK_N"
 		(shape bidirectional)
 		(at 156.21 105.41 0)
@@
 		)
 	)
-	(hierarchical_label "DSI_TE"
+	(hierarchical_label "DSI.TE"
 		(shape input)
 		(at 156.21 78.74 0)
@@
 		)
 	)
-	(hierarchical_label "TP_INT"
+	(hierarchical_label "TP.INT"
 		(shape output)
 		(at 224.79 124.46 180)
@@
 		)
 	)
-	(hierarchical_label "TP_SDA"
+	(hierarchical_label "TP.SDA"
 		(shape bidirectional)
 		(at 113.03 82.55 180)
@@
 		)
 	)
-	(hierarchical_label "DSI_PWR_EN"
+	(hierarchical_label "DSI.PWR_EN"
 		(shape input)
 		(at 156.21 101.6 0)
@@
 		)
 	)
-	(hierarchical_label "DSI_D0_P"
+	(hierarchical_label "DSI.D0_P"
 		(shape bidirectional)
 		(at 156.21 90.17 0)
@@
 		)
 	)
-	(hierarchical_label "TP_SDA"
+	(hierarchical_label "TP.SDA"
 		(shape bidirectional)
 		(at 224.79 119.38 180)
@@
 		)
 	)
-	(hierarchical_label "DSI_D0_N"
+	(hierarchical_label "DSI.D0_N"
 		(shape bidirectional)
 		(at 156.21 82.55 0)
@@
 		)
 	)
-	(hierarchical_label "TP_INT"
+	(hierarchical_label "TP.INT"
 		(shape output)
 		(at 113.03 90.17 180)

Commit message: sch update
Other:
- note added: "If IM1=GND,IM0=GND, CS=IOVCC, DO0143FMST02 set to MIPI-DSI interface"
- note added: "If IM1=IOVCC,IM0=GND, DO0143FMST02 set to QSPI interface"
Changed lines of the file:
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@@
+		)
+	)
+	(text "If IM1=GND,IM0=GND, CS=IOVCC, DO0143FMST02 set to MIPI-DSI interface"
+		(exclude_from_sim no)
+		(at 137.16 170.18 0)
+		(effects
+			(font
+				(size 1.27 1.27)
+			)
+		)
+	)
+	(text "If IM1=IOVCC,IM0=GND, DO0143FMST02 set to QSPI interface"
+		(exclude_from_sim no)
+		(at 137.16 165.1 0)
+		(effects
+			(font
+				(size 1.27 1.27)
+			)
 		)
 	)
