File: hardware/schematic/v1.0/XWatch_Rev3.0/BLE.kicad_sch (KiCad schematic)
At the start: 3 parts, among them IC1 nRF52833-QDAA-R

Commit message: sch update
Parts:
- added C71: 4.7uF, XWatch_Rev3.0:GEN_C_0402, symbol XWatch_Rev3.0:C
- added C72, C79: 100nF, XWatch_Rev3.0:GEN_C_0201, symbol XWatch_Rev3.0:C
- added C80, C81: 1uF, XWatch_Rev3.0:GEN_C_0402, symbol XWatch_Rev3.0:C
- added C82: 1pF, XWatch_Rev3.0:GEN_C_0201, symbol XWatch_Rev3.0:C
- added C83: 1.2pF, XWatch_Rev3.0:GEN_C_0201, symbol XWatch_Rev3.0:C
- added L4: 4.7nH, XWatch_Rev3.0:L_0201_0603Metric, symbol XWatch_Rev3.0:L
- added L5: 2.2nH, XWatch_Rev3.0:L_0201_0603Metric, symbol XWatch_Rev3.0:L
- added R26, R27: 100K, XWatch_Rev3.0:GEN_R_0201, symbol XWatch_Rev3.0:R
- added U16: R832000033-32MHZ, XWatch_Rev3.0:R832000033, symbol XWatch_Rev3.0:R832000033
Connections:
- net GND: now also IC1.41 (VSS_2), C71.2, C72.1, C79.1, C80.2, C81.2, C82.2, C83.2, R26.1, R27.1
- net BLE.MCU_CTS: now reaches IC1.14 (P0.15)
- net BLE.MCU_RTS: now reaches IC1.15 (P0.17)
- net nRESET: now reaches IC1.16 (P0.18/NRESET)
- net BLE.WAKE_MCU: now reaches IC1.17 (P0.20)
- net BLE.WAKE_MCU: now also R27.2
- net +1V8: now reaches IC1.18 (VDD_2)
- net +1V8: now also IC1.30 (VDD_3), IC1.40 (VDD_4), IC1.8 (VDD_1), IC1.9 (VDDH), C71.1, C72.2, C79.2, C80.1
- net SWDIO: now reaches IC1.19 (SWDIO)
- net SWDCLK: now reaches IC1.20 (SWDCLK)
- net at IC1.24 (ANT): now also C82.1, L4.1
- net at IC1.38 (DEC4): now also C81.1
- net BLE.MCU_RX: now reaches IC1.4 (P0.04/AIN2)
- net BLE.MCU_TX: now reaches IC1.5 (P0.05/AIN3)
- net BLE.WAKE_NRF: now reaches IC1.7 (P0.11)
- net BLE.WAKE_NRF: now also R26.2
- new net: C83.1, L4.2, L5.1
Other:
- note added: "CTS"
- note added: "RF_50R"
- note added: "RTS"
- note added: "RXD"
- note added: "TXD"

Commit message: sch update
Parts:
- added C84, C85: 12pF, XWatch_Rev3.0:GEN_C_0201, symbol XWatch_Rev3.0:C
- added C86, C87: 5.6pF, XWatch_Rev3.0:GEN_C_0201, symbol XWatch_Rev3.0:C
- added C88: 100pF, XWatch_Rev3.0:GEN_C_0201, symbol XWatch_Rev3.0:C
- added X3: 32.768KHZ, XWatch_Rev3.0:NX3215SA_32_768KHZ_EXS00A-MU00525, symbol XWatch_Rev3.0:NX3215SA_32_768KHZ_EXS00A-MU00525
Connections:
- net GND: now also U16.2 (GND), U16.4 (GND), C84.1, C85.2, C86.1, C87.1, C88.2
- net DEC6: now reaches C81.1, IC1.38 (DEC4)
- net DEC6: now also IC1.26 (DEC6)
- net at IC1.2 (P0.00/XL1): now also C86.2, X3.1
- net at IC1.27 (DEC3): now also C88.1
- net at IC1.28 (XC1): now also U16.3, C85.1
- net at IC1.29 (XC2): now also U16.1, C84.2
- net at IC1.3 (P0.01/XL2): now also C87.2, X3.2
- no-connect marks 11 -> 13
Other:
- moved on the sheet: R27, U16

Commit message: sch update
Parts:
- added CN5, CN6: SCTA1A0100, XWatch_Rev3.0:SCTA1A0100, symbol XWatch_Rev3.0:SCTA1A0100
- added R28: 100K, XWatch_Rev3.0:GEN_R_0201, symbol XWatch_Rev3.0:R
Connections:
- net +1V8: now also R28.2
- net GND: now also CN6.1
- net nRESET: now also R28.1
- net at L5.2: now also CN5.1

Commit message: sch update
Parts:
- added TP5, TP6, TP7, TP8: TestPoint, TestPoint:TestPoint_Pad_D1.0mm, symbol Connector:TestPoint
Connections:
- net GND: now also TP8.1
- net SWDCLK: now also TP6.1
- net SWDIO: now also TP5.1
- net nRESET: now also TP7.1
