File: hardware/schematic/v1.0/XWatch_Rev3.0/SENSOR.kicad_sch (KiCad schematic)
At the start: 26 parts, among them U10 OPT3001DNPR, U11 MAX30101EFD_T, U12 DRV2605LDGSR, U6 LSM6DSOXTR, U7 LIS2MDLTR, U9 LPS27HHWTR

Commit message: sch update
Connections:
- net DRV_REG: no longer names the net of C64.2, U12.1 (REG)
- net MAG_C1: no longer names the net of C52.1, U7.5 (C1)
Changed lines of the file:
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@@
-	)
-	(junction
-		(at 45.72 109.22)
-		(diameter 0)
-		(color 0 0 0 0)
-	)
-	(junction
-		(at 104.14 161.29)
-		(diameter 0)
-		(color 0 0 0 0)
 	)
 	(junction
@@
 	(wire
 		(pts
-			(xy 43.18 109.22) (xy 45.72 109.22)
-		)
-		(stroke
-			(width 0)
-			(type default)
-		)
-	)
-	(wire
-		(pts
 			(xy 232.41 128.27) (xy 232.41 130.81)
 		)
@@
 		(pts
 			(xy 140.97 171.45) (xy 140.97 172.72)
-		)
-		(stroke
-			(width 0)
-			(type default)
-		)
-	)
-	(wire
-		(pts
-			(xy 99.06 161.29) (xy 104.14 161.29)
 		)
 		(stroke
@@
 		)
 	)
-	(hierarchical_label "MAG_C1"
-		(shape output)
-		(at 43.18 109.22 180)
-		(effects
-			(font
-				(size 1.27 1.27)
-			)
-			(justify right)
-		)
-	)
 	(hierarchical_label "LRA_P"
 		(shape output)
@@
 		(effects
 			(font
-				(size 1.27 1.27)
-			)
-			(justify right)
-		)
-	)
-	(hierarchical_label "DRV_REG"
-		(shape input)
-		(at 99.06 161.29 180)
-		(effects
-			(font

Commit message: sch update
Connections:
- net ALS_INT_N renamed ALS.INT_N
- net BARO_INT renamed BARO.INT
- net HAPTIC_EN renamed HAPTIC.EN
- net IMU_INT1 renamed IMU.INT1
- net IMU_INT2 renamed IMU.INT2
- net LRA_N renamed LRA.N
- net LRA_P renamed LRA.P
- net MAG_DRDY renamed MAG.DRDY
- net PPG_INT_N renamed PPG.INT_N
- net SENSOR_SCL renamed SENSOR.SCL
- net SENSOR_SDA renamed SENSOR.SDA
Changed lines of the file:
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@@
 		)
 	)
-	(hierarchical_label "ALS_INT_N"
+	(hierarchical_label "ALS.INT_N"
 		(shape output)
 		(at 179.07 124.46 0)
@@
 		)
 	)
-	(hierarchical_label "LRA_P"
+	(hierarchical_label "LRA.P"
 		(shape output)
 		(at 137.16 168.91 0)
@@
 		)
 	)
-	(hierarchical_label "SENSOR_SCL"
+	(hierarchical_label "SENSOR.SCL"
 		(shape input)
 		(at 50.8 99.06 180)
@@
 		)
 	)
-	(hierarchical_label "SENSOR_SDA"
+	(hierarchical_label "SENSOR.SDA"
 		(shape bidirectional)
 		(at 217.17 143.51 180)
@@
 		)
 	)
-	(hierarchical_label "BARO_INT"
+	(hierarchical_label "BARO.INT"
 		(shape output)
 		(at 182.88 57.15 0)
@@
 		)
 	)
-	(hierarchical_label "SENSOR_SDA"
+	(hierarchical_label "SENSOR.SDA"
 		(shape bidirectional)
 		(at 91.44 46.99 0)
@@
 		)
 	)
-	(hierarchical_label "LRA_N"
+	(hierarchical_label "LRA.N"
 		(shape output)
 		(at 137.16 163.83 0)
@@
 		)
 	)
-	(hierarchical_label "SENSOR_SDA"
+	(hierarchical_label "SENSOR.SDA"
 		(shape bidirectional)
 		(at 50.8 106.68 180)
@@
 		)
 	)
-	(hierarchical_label "IMU_INT2"
+	(hierarchical_label "IMU.INT2"
 		(shape output)
 		(at 91.44 59.69 0)
@@
 		)
 	)
-	(hierarchical_label "SENSOR_SCL"
+	(hierarchical_label "SENSOR.SCL"
 		(shape input)
 		(at 217.17 146.05 180)
@@
 		)
 	)
-	(hierarchical_label "IMU_INT1"
+	(hierarchical_label "IMU.INT1"
 		(shape output)
 		(at 58.42 54.61 180)
@@
 		)
 	)
-	(hierarchical_label "SENSOR_SCL"
+	(hierarchical_label "SENSOR.SCL"
 		(shape input)
 		(at 106.68 163.83 180)
@@
 		)
 	)
-	(hierarchical_label "HAPTIC_EN"
+	(hierarchical_label "HAPTIC.EN"
 		(shape input)
 		(at 102.87 171.45 180)
@@
 		)
 	)
-	(hierarchical_label "SENSOR_SCL"
+	(hierarchical_label "SENSOR.SCL"
 		(shape input)
 		(at 173.99 105.41 0)
@@
 		)
 	)
-	(hierarchical_label "SENSOR_SDA"
+	(hierarchical_label "SENSOR.SDA"
 		(shape bidirectional)
 		(at 173.99 100.33 0)
@@
 		)
 	)
-	(hierarchical_label "MAG_DRDY"
+	(hierarchical_label "MAG.DRDY"
 		(shape output)
 		(at 114.3 111.76 0)
@@
 		)
 	)
-	(hierarchical_label "SENSOR_SCL"
+	(hierarchical_label "SENSOR.SCL"
 		(shape input)
 		(at 142.24 52.07 180)
@@
 		)
 	)
-	(hierarchical_label "SENSOR_SCL"
+	(hierarchical_label "SENSOR.SCL"
 		(shape input)
 		(at 212.09 71.12 180)
@@
 		)
 	)
-	(hierarchical_label "PPG_INT_N"
+	(hierarchical_label "PPG.INT_N"
 		(shape output)
 		(at 209.55 101.6 0)
@@
 		)
 	)
-	(hierarchical_label "SENSOR_SDA"
+	(hierarchical_label "SENSOR.SDA"
 		(shape bidirectional)
 		(at 142.24 57.15 180)
@@
 		)
 	)
-	(hierarchical_label "SENSOR_SDA"
+	(hierarchical_label "SENSOR.SDA"
 		(shape bidirectional)
 		(at 212.09 73.66 180)
@@
 		)
 	)
-	(hierarchical_label "SENSOR_SCL"
+	(hierarchical_label "SENSOR.SCL"
 		(shape input)
 		(at 91.44 49.53 0)
@@
 		)
 	)
-	(hierarchical_label "PPG_INT_N"
+	(hierarchical_label "PPG.INT_N"
 		(shape output)
 		(at 234.95 71.12 0)
@@
 		)
 	)
-	(hierarchical_label "ALS_INT_N"
+	(hierarchical_label "ALS.INT_N"
 		(shape output)
 		(at 173.99 102.87 0)
@@
 		)
 	)
-	(hierarchical_label "SENSOR_SDA"
+	(hierarchical_label "SENSOR.SDA"
 		(shape bidirectional)
 		(at 106.68 166.37 180)
